Commit message: material not working

File: march_ws/src/march_description/urdf/march.xacro (robot description, xacro)
@@ -2,87 +2,88 @@
 <!-- Revolute-Revolute Manipulator -->
 <robot name="march" xmlns:xacro="http://www.ros.org/wiki/xacro">
-  <!-- Constants for robot dimensions -->
-  <xacro:property name="PI" value="3.1415926535897931"/>
-  <xacro:property name="mass" value="1" /> <!-- arbitrary value for mass -->
-  <xacro:property name="width" value="0.1" /> <!-- Square dimensions (widthxwidth) of beams -->
-  <xacro:property name="height1" value="2" /> <!-- Link 1 -->
-  <xacro:property name="height2" value="1" /> <!-- Link 2 -->
-  <xacro:property name="height3" value="1" /> <!-- Link 3 -->
-  <xacro:property name="camera_link" value="0.05" /> <!-- Size of square 'camera' box -->
-  <xacro:property name="axel_offset" value="0.05" /> <!-- Space btw top of beam and the each joint -->
-  <!-- Import all Gazebo-customization elements, including Gazebo colors -->
-  <xacro:include filename="$(find march_description)/urdf/march.gazebo" />
-  <!-- Import Rviz colors -->
-  <xacro:include filename="$(find march_description)/urdf/materials.xacro" />
-  <!-- Used for fixing robot to Gazebo 'base_link' -->
-  <link name="world"/>
-  <joint name="fixed" type="fixed">
-    <parent link="world"/>
-    <child link="link1"/>
-  </joint>
-  <!-- Base Link -->
-  <link name="link1">
-    <collision>
-      <origin xyz="0 0 ${height1/2}" rpy="0 0 0"/>
-      <geometry>
-	<box size="${width} ${width} ${height1}"/>
-      </geometry>
-    </collision>
-    <visual>
-      <origin xyz="0 0 ${height1/2}" rpy="0 0 0"/>
-      <geometry>
-	<box size="${width} ${width} ${height1}"/>
-      </geometry>
-      <material name="blue"/>
-    </visual>
-    <inertial>
-      <origin xyz="0 0 ${height1/2}" rpy="0 0 0"/>
-      <mass value="${mass}"/>
-      <inertia
-	  ixx="${mass / 12.0 * (width*width + height1*height1)}" ixy="0.0" ixz="0.0"
-	  iyy="${mass / 12.0 * (height1*height1 + width*width)}" iyz="0.0"
-	  izz="${mass / 12.0 * (width*width + width*width)}"/>
-    </inertial>
-  </link>
-  <joint name="joint1" type="continuous">
-    <parent link="link1"/>
-    <child link="link2"/>
-    <origin xyz="0 ${width} ${height1 - axel_offset}" rpy="0 0 0"/>
-    <axis xyz="0 1 0"/>
-    <dynamics damping="0.7"/>
-  </joint>
-  <!-- Middle Link -->
-  <link name="link2">
-    <collision>
-      <origin xyz="0 0 ${height2/2 - axel_offset}" rpy="0 0 0"/>
-      <geometry>
-	<box size="${width} ${width} ${height2}"/>
-      </geometry>
-    </collision>
-    <visual>
-      <origin xyz="0 0 ${height2/2 - axel_offset}" rpy="0 0 0"/>
-      <geometry>
-	<box size="${width} ${width} ${height2}"/>
-      </geometry>
-      <material name="orange"/>
-    </visual>
-    <inertial>
-      <origin xyz="0 0 ${height2/2 - axel_offset}" rpy="0 0 0"/>
-      <mass value="${mass}"/>
-      <inertia
-	  ixx="${mass / 12.0 * (width*width + height2*height2)}" ixy="0.0" ixz="0.0"
-	  iyy="${mass / 12.0 * (height2*height2 + width*width)}" iyz="0.0"
-	  izz="${mass / 12.0 * (width*width + width*width)}"/>
-    </inertial>
-  </link>
-  <transmission name="tran1">
-    <type>transmission_interface/SimpleTransmission</type>
-    <joint name="joint1">
-      <hardwareInterface>hardware_interface/EffortJointInterface</hardwareInterface>
+    <!-- Constants for robot dimensions -->
+    <xacro:property name="PI" value="3.1415926535897931"/>
+    <xacro:property name="mass" value="1"/> <!-- arbitrary value for mass -->
+    <xacro:property name="width" value="0.1"/> <!-- Square dimensions (widthxwidth) of beams -->
+    <xacro:property name="height1" value="2"/> <!-- Link 1 -->
+    <xacro:property name="height2" value="1"/> <!-- Link 2 -->
+    <xacro:property name="height3" value="1"/> <!-- Link 3 -->
+    <xacro:property name="camera_link" value="0.05"/> <!-- Size of square 'camera' box -->
+    <xacro:property name="axel_offset" value="0.05"/> <!-- Space btw top of beam and the each joint -->
+    <!-- Import all Gazebo-customization elements, including Gazebo colors -->
+    <xacro:include filename="$(find march_description)/urdf/march.gazebo"/>
+    <!-- Import Rviz colors -->
+    <xacro:include filename="$(find march_description)/urdf/materials.xacro"/>
+    <!-- Used for fixing robot to Gazebo 'base_link' -->
+    <link name="world"/>
+    <joint name="fixed" type="fixed">
+        <parent link="world"/>
+        <child link="link1"/>
     </joint>
-    <actuator name="motor1">
-      <hardwareInterface>hardware_interface/EffortJointInterface</hardwareInterface>
-      <mechanicalReduction>1</mechanicalReduction>
-    </actuator>
-  </transmission>
+    <!-- Base Link -->
+    <link name="link1">
+        <collision>
+            <origin xyz="0 0 ${height1/2}" rpy="0 0 0"/>
+            <geometry>
+                <box size="${width} ${width} ${height1}"/>
+            </geometry>
+        </collision>
+        <visual>
+            <origin xyz="0 0 ${height1/2}" rpy="0 0 0"/>
+            <geometry>
+                <box size="${width} ${width} ${height1}"/>
+            </geometry>
+        </visual>
+        <inertial>
+            <origin xyz="0 0 ${height1/2}" rpy="0 0 0"/>
+            <mass value="${mass}"/>
+            <inertia
+                    ixx="${mass / 12.0 * (width*width + height1*height1)}" ixy="0.0" ixz="0.0"
+                    iyy="${mass / 12.0 * (height1*height1 + width*width)}" iyz="0.0"
+                    izz="${mass / 12.0 * (width*width + width*width)}"/>
+        </inertial>
+    </link>
+    <gazebo reference="link1">
+        <material>march_blue</material>
+    </gazebo>
+    <joint name="joint1" type="continuous">
+        <parent link="link1"/>
+        <child link="link2"/>
+        <origin xyz="0 ${width} ${height1 - axel_offset}" rpy="0 0 0"/>
+        <axis xyz="0 1 0"/>
+        <dynamics damping="0.7"/>
+    </joint>
+    <!-- Middle Link -->
+    <link name="link2">
+        <collision>
+            <origin xyz="0 0 ${height2/2 - axel_offset}" rpy="0 0 0"/>
+            <geometry>
+                <box size="${width} ${width} ${height2}"/>
+            </geometry>
+        </collision>
+        <visual>
+            <origin xyz="0 0 ${height2/2 - axel_offset}" rpy="0 0 0"/>
+            <geometry>
+                <box size="${width} ${width} ${height2}"/>
+            </geometry>
+        </visual>
+        <inertial>
+            <origin xyz="0 0 ${height2/2 - axel_offset}" rpy="0 0 0"/>
+            <mass value="${mass}"/>
+            <inertia
+                    ixx="${mass / 12.0 * (width*width + height2*height2)}" ixy="0.0" ixz="0.0"
+                    iyy="${mass / 12.0 * (height2*height2 + width*width)}" iyz="0.0"
+                    izz="${mass / 12.0 * (width*width + width*width)}"/>
+        </inertial>
+    </link>
+    <transmission name="tran1">
+        <type>transmission_interface/SimpleTransmission</type>
+        <joint name="joint1">
+            <hardwareInterface>hardware_interface/EffortJointInterface</hardwareInterface>
+        </joint>
+        <actuator name="motor1">
+            <hardwareInterface>hardware_interface/EffortJointInterface</hardwareInterface>
+            <mechanicalReduction>1</mechanicalReduction>
+        </actuator>
+    </transmission>
 </robot>

File: march_ws/src/march_description/urdf/materials.xacro (robot description, xacro)
@@ -4,5 +4,5 @@
     <color rgba="0.0 0.0 0.0 1.0"/>
   </material>
-  <material name="blue">
+  <material name="march_blue">
     <color rgba="${18/255} ${98/255} ${135/255} 1.0"/>
   </material>

Commit message: materials linked

File: march_ws/src/march_description/urdf/march.xacro (robot description, xacro)
@@ -13,6 +13,4 @@
     <!-- Import all Gazebo-customization elements, including Gazebo colors -->
     <xacro:include filename="$(find march_description)/urdf/march.gazebo"/>
-    <!-- Import Rviz colors -->
-    <xacro:include filename="$(find march_description)/urdf/materials.xacro"/>
     <!-- Used for fixing robot to Gazebo 'base_link' -->
     <link name="world"/>
@@ -44,7 +42,4 @@
         </inertial>
     </link>
-    <gazebo reference="link1">
-        <material>march_blue</material>
-    </gazebo>
     <joint name="joint1" type="continuous">
         <parent link="link1"/>

Commit message: Add rough draft of exoskeleton URDF

File: march_ws/src/march_description/urdf/march.xacro (robot description, xacro)
@@ -6,7 +6,20 @@
     <xacro:property name="mass" value="1"/> <!-- arbitrary value for mass -->
     <xacro:property name="width" value="0.1"/> <!-- Square dimensions (widthxwidth) of beams -->
-    <xacro:property name="height1" value="2"/> <!-- Link 1 -->
-    <xacro:property name="height2" value="1"/> <!-- Link 2 -->
-    <xacro:property name="height3" value="1"/> <!-- Link 3 -->
+    <xacro:property name="upper_leg_height" value="${0.37*3}"/>
+    <xacro:property name="lower_leg_height" value="${0.41*3}"/>
+    <xacro:property name="foot_height" value="${0.14*3}"/>
+    <xacro:property name="hip_height" value="1"/>
+    <xacro:property name="hip_rotation_lower_limit" value="${0*pi/180}"/>
+    <xacro:property name="hip_rotation_upper_limit" value="${30*pi/180}"/>
+    <xacro:property name="hip_effort_limit" value="100.0"/>
+    <xacro:property name="hip_velocity_limit" value="10.0"/>
+    <xacro:property name="knee_rotation_lower_limit" value="${-50*pi/180}"/>
+    <xacro:property name="knee_rotation_upper_limit" value="${0*pi/180}"/>
+    <xacro:property name="knee_effort_limit" value="100.0"/>
+    <xacro:property name="knee_velocity_limit" value="10.0"/>
+    <xacro:property name="ankle_rotation_lower_limit" value="${0*pi/180}"/>
+    <xacro:property name="ankle_rotation_upper_limit" value="${30*pi/180}"/>
+    <xacro:property name="ankle_effort_limit" value="100.0"/>
+    <xacro:property name="ankle_velocity_limit" value="10.0"/>
     <xacro:property name="camera_link" value="0.05"/> <!-- Size of square 'camera' box -->
     <xacro:property name="axel_offset" value="0.05"/> <!-- Space btw top of beam and the each joint -->
@@ -15,67 +28,225 @@
     <!-- Used for fixing robot to Gazebo 'base_link' -->
     <link name="world"/>
-    <joint name="fixed" type="fixed">
+    <joint name="hip" type="fixed">
         <parent link="world"/>
-        <child link="link1"/>
-    </joint>
-    <!-- Base Link -->
-    <link name="link1">
-        <collision>
-            <origin xyz="0 0 ${height1/2}" rpy="0 0 0"/>
-            <geometry>
-                <box size="${width} ${width} ${height1}"/>
-            </geometry>
-        </collision>
-        <visual>
-            <origin xyz="0 0 ${height1/2}" rpy="0 0 0"/>
-            <geometry>
-                <box size="${width} ${width} ${height1}"/>
-            </geometry>
-        </visual>
-        <inertial>
-            <origin xyz="0 0 ${height1/2}" rpy="0 0 0"/>
-            <mass value="${mass}"/>
-            <inertia
-                    ixx="${mass / 12.0 * (width*width + height1*height1)}" ixy="0.0" ixz="0.0"
-                    iyy="${mass / 12.0 * (height1*height1 + width*width)}" iyz="0.0"
-                    izz="${mass / 12.0 * (width*width + width*width)}"/>
-        </inertial>
-    </link>
-    <joint name="joint1" type="continuous">
-        <parent link="link1"/>
-        <child link="link2"/>
-        <origin xyz="0 ${width} ${height1 - axel_offset}" rpy="0 0 0"/>
-        <axis xyz="0 1 0"/>
-        <dynamics damping="0.7"/>
-    </joint>
-    <!-- Middle Link -->
-    <link name="link2">
-        <collision>
-            <origin xyz="0 0 ${height2/2 - axel_offset}" rpy="0 0 0"/>
-            <geometry>
-                <box size="${width} ${width} ${height2}"/>
-            </geometry>
-        </collision>
-        <visual>
-            <origin xyz="0 0 ${height2/2 - axel_offset}" rpy="0 0 0"/>
-            <geometry>
-                <box size="${width} ${width} ${height2}"/>
-            </geometry>
-        </visual>
-        <inertial>
-            <origin xyz="0 0 ${height2/2 - axel_offset}" rpy="0 0 0"/>
-            <mass value="${mass}"/>
-            <inertia
-                    ixx="${mass / 12.0 * (width*width + height2*height2)}" ixy="0.0" ixz="0.0"
-                    iyy="${mass / 12.0 * (height2*height2 + width*width)}" iyz="0.0"
-                    izz="${mass / 12.0 * (width*width + width*width)}"/>
-        </inertial>
-    </link>
-    <transmission name="tran1">
+        <child link="hip_bone"/>
+        <origin xyz="0 0 ${lower_leg_height+upper_leg_height}" rpy="0 0 0"/>
+    </joint>
+    <!--<joint name="right_hip" type="revolute">-->
+        <!--<parent link="hip"/>-->
+        <!--<child link="upper_leg_right"/>-->
+        <!--<origin xyz="0 0 ${lower_leg_height+upper_leg_height}" rpy="0 0 0"/>-->
+        <!--<axis xyz="0 1 0"/>-->
+        <!--<limit velocity="${hip_velocity_limit}" effort="${hip_effort_limit}" lower="${hip_rotation_lower_limit}" upper="${hip_rotation_upper_limit}"/>-->
+    <!--</joint>-->
+    <joint name="left_hip" type="revolute">
+        <parent link="hip_bone"/>
+        <child link="upper_leg_left"/>
+        <origin xyz="0 ${-hip_height/2} 0" rpy="0 0 0"/>
+        <axis xyz="0 1 0"/>
+        <limit velocity="${hip_velocity_limit}" effort="${hip_effort_limit}" lower="${hip_rotation_lower_limit}" upper="${hip_rotation_upper_limit}"/>
+    </joint>
+    <joint name="left_knee" type="revolute">
+        <parent link="upper_leg_left"/>
+        <child link="lower_leg_left"/>
+        <origin xyz="0 0 ${-upper_leg_height}" rpy="0 0 0"/>
+        <axis xyz="0 1 0"/>
+        <limit velocity="${knee_velocity_limit}" effort="${knee_effort_limit}" lower="${knee_rotation_lower_limit}" upper="${knee_rotation_upper_limit}"/>
+    </joint>
+    <joint name="left_ankle" type="revolute">
+        <parent link="lower_leg_left"/>
+        <child link="foot_left"/>
+        <origin xyz="0 0 ${-lower_leg_height}" rpy="0 0 0"/>
+        <axis xyz="0 1 0"/>
+        <limit velocity="${ankle_velocity_limit}" effort="${ankle_effort_limit}" lower="${ankle_rotation_lower_limit}" upper="${ankle_rotation_upper_limit}"/>
+    </joint>
+    <joint name="right_hip" type="revolute">
+        <parent link="hip_bone"/>
+        <child link="upper_leg_right"/>
+        <origin xyz="0 ${hip_height/2} 0" rpy="0 0 0"/>
+        <axis xyz="0 1 0"/>
+        <limit velocity="${hip_velocity_limit}" effort="${hip_effort_limit}" lower="${hip_rotation_lower_limit}" upper="${hip_rotation_upper_limit}"/>
+    </joint>
+    <joint name="right_knee" type="revolute">
+        <parent link="upper_leg_right"/>
+        <child link="lower_leg_right"/>
+        <origin xyz="0 0 ${-upper_leg_height}" rpy="0 0 0"/>
+        <axis xyz="0 1 0"/>
+        <limit velocity="${knee_velocity_limit}" effort="${knee_effort_limit}" lower="${knee_rotation_lower_limit}" upper="${knee_rotation_upper_limit}"/>
+    </joint>
+    <joint name="right_ankle" type="revolute">
+        <parent link="lower_leg_right"/>
+        <child link="foot_right"/>
+        <origin xyz="0 0 ${-lower_leg_height}" rpy="0 0 0"/>
+        <axis xyz="0 1 0"/>
+        <limit velocity="${ankle_velocity_limit}" effort="${ankle_effort_limit}" lower="${ankle_rotation_lower_limit}" upper="${ankle_rotation_upper_limit}"/>
+    </joint>
+    <!-- Hip-->
+    <link name="hip_bone">
+        <collision>
+            <origin xyz="0 0 0" rpy="0 0 0"/>
+            <geometry>
+                <box size="${width} ${width} ${hip_height}"/>
+            </geometry>
+        </collision>
+        <visual>
+            <origin xyz="0 0 0" rpy="0 0 0"/>
+            <geometry>
+                <box size="${width} ${hip_height} ${width}"/>
+            </geometry>
+        </visual>
+        <inertial>
+            <origin xyz="0 0 0" rpy="0 0 0"/>
+            <mass value="${mass}"/>
+            <inertia
+                    ixx="${mass / 12.0 * (width*width + lower_leg_height*lower_leg_height)}" ixy="0.0" ixz="0.0"
+                    iyy="${mass / 12.0 * (lower_leg_height*lower_leg_height + width*width)}" iyz="0.0"
+                    izz="${mass / 12.0 * (width*width + width*width)}"/>
+        </inertial>
+    </link>
+    <!-- Upper Leg Left-->
+    <link name="upper_leg_left">
+        <collision>
+            <origin xyz="0 0 ${-upper_leg_height/2}" rpy="0 0 0"/>
+            <geometry>
+                <box size="${width} ${width} ${upper_leg_height}"/>
+            </geometry>
+        </collision>
+        <visual>
+            <origin xyz="0 0 ${-upper_leg_height/2}" rpy="0 0 0"/>
+            <geometry>
+                <box size="${width} ${width} ${upper_leg_height}"/>
+            </geometry>
+        </visual>
+        <inertial>
+            <origin xyz="0 0 ${-upper_leg_height/2}" rpy="0 0 0"/>
+            <mass value="${mass}"/>
+            <inertia
+                    ixx="${mass / 12.0 * (width*width + upper_leg_height*upper_leg_height)}" ixy="0.0" ixz="0.0"
+                    iyy="${mass / 12.0 * (upper_leg_height*upper_leg_height + width*width)}" iyz="0.0"
+                    izz="${mass / 12.0 * (width*width + width*width)}"/>
+        </inertial>
+    </link>
+    <!-- Lower Leg Left -->
+    <link name="lower_leg_left">
+        <collision>
+            <origin xyz="0 0 ${-lower_leg_height/2}" rpy="0 0 0"/>
+            <geometry>
+                <box size="${width} ${width} ${lower_leg_height}"/>
+            </geometry>
+        </collision>
+        <visual>
+            <origin xyz="0 0 ${-lower_leg_height/2}" rpy="0 0 0"/>
+            <geometry>
+                <box size="${width} ${width} ${lower_leg_height}"/>
+            </geometry>
+        </visual>
+        <inertial>
+            <origin xyz="0 0 ${-lower_leg_height/2}" rpy="0 0 0"/>
+            <mass value="${mass}"/>
+            <inertia
+                    ixx="${mass / 12.0 * (width*width + lower_leg_height*lower_leg_height)}" ixy="0.0" ixz="0.0"
+                    iyy="${mass / 12.0 * (lower_leg_height*lower_leg_height + width*width)}" iyz="0.0"
+                    izz="${mass / 12.0 * (width*width + width*width)}"/>
+        </inertial>
+    </link>
+    <!-- Foot Left -->
+    <link name="foot_left">
+        <collision>
+            <origin xyz="${-foot_height/2} 0 0" rpy="0 0 0"/>
+            <geometry>
+                <box size="${width} ${foot_height} ${width}"/>
+            </geometry>
+        </collision>
+        <visual>
+            <origin xyz="${-foot_height/2} 0 0" rpy="0 0 0"/>
+            <geometry>
+                <box size="${foot_height} ${width} ${width}"/>
+            </geometry>
+        </visual>
+        <inertial>
+            <origin xyz="${-foot_height/2} 0 0" rpy="0 0 0"/>
+            <mass value="${mass}"/>
+            <inertia
+                    ixx="${mass / 12.0 * (width*width + lower_leg_height*lower_leg_height)}" ixy="0.0" ixz="0.0"
+                    iyy="${mass / 12.0 * (lower_leg_height*lower_leg_height + width*width)}" iyz="0.0"
+                    izz="${mass / 12.0 * (width*width + width*width)}"/>
+        </inertial>
+    </link>
+    <!-- Upper Leg Right-->
+    <link name="upper_leg_right">
+        <collision>
+            <origin xyz="0 0 ${-upper_leg_height/2}" rpy="0 0 0"/>
+            <geometry>
+                <box size="${width} ${width} ${upper_leg_height}"/>
+            </geometry>
+        </collision>
+        <visual>
+            <origin xyz="0 0 ${-upper_leg_height/2}" rpy="0 0 0"/>
+            <geometry>
+                <box size="${width} ${width} ${upper_leg_height}"/>
+            </geometry>
+        </visual>
+        <inertial>
+            <origin xyz="0 0 ${-upper_leg_height/2}" rpy="0 0 0"/>
+            <mass value="${mass}"/>
+            <inertia
+                    ixx="${mass / 12.0 * (width*width + upper_leg_height*upper_leg_height)}" ixy="0.0" ixz="0.0"
+                    iyy="${mass / 12.0 * (upper_leg_height*upper_leg_height + width*width)}" iyz="0.0"
+                    izz="${mass / 12.0 * (width*width + width*width)}"/>
+        </inertial>
+    </link>
+    <!-- Lower Leg Right -->
+    <link name="lower_leg_right">
+        <collision>
+            <origin xyz="0 0 ${-lower_leg_height/2}" rpy="0 0 0"/>
+            <geometry>
+                <box size="${width} ${width} ${lower_leg_height}"/>
+            </geometry>
+        </collision>
+        <visual>
+            <origin xyz="0 0 ${-lower_leg_height/2}" rpy="0 0 0"/>
+            <geometry>
+                <box size="${width} ${width} ${lower_leg_height}"/>
+            </geometry>
+        </visual>
+        <inertial>
+            <origin xyz="0 0 ${-lower_leg_height/2}" rpy="0 0 0"/>
+            <mass value="${mass}"/>
+            <inertia
+                    ixx="${mass / 12.0 * (width*width + lower_leg_height*lower_leg_height)}" ixy="0.0" ixz="0.0"
+                    iyy="${mass / 12.0 * (lower_leg_height*lower_leg_height + width*width)}" iyz="0.0"
+                    izz="${mass / 12.0 * (width*width + width*width)}"/>
+        </inertial>
+    </link>
+    <!-- Foot Right -->
+    <link name="foot_right">
+        <collision>
+            <origin xyz="${-foot_height/2} 0 0" rpy="0 0 0"/>
+            <geometry>
+                <box size="${width} ${foot_height} ${width}"/>
+            </geometry>
+        </collision>
+        <visual>
+            <origin xyz="${-foot_height/2} 0 0" rpy="0 0 0"/>
+            <geometry>
+                <box size="${foot_height} ${width} ${width}"/>
+            </geometry>
+        </visual>
+        <inertial>
+            <origin xyz="${-foot_height/2} 0 0" rpy="0 0 0"/>
+            <mass value="${mass}"/>
+            <inertia
+                    ixx="${mass / 12.0 * (width*width + lower_leg_height*lower_leg_height)}" ixy="0.0" ixz="0.0"
+                    iyy="${mass / 12.0 * (lower_leg_height*lower_leg_height + width*width)}" iyz="0.0"
+                    izz="${mass / 12.0 * (width*width + width*width)}"/>
+        </inertial>
+    </link>
+    <transmission name="left_hip">
         <type>transmission_interface/SimpleTransmission</type>
-        <joint name="joint1">
+        <joint name="left_hip">
             <hardwareInterface>hardware_interface/PositionJointInterface</hardwareInterface>
         </joint>
-        <actuator name="motor1">
+        <actuator name="left_hip_motor">
             <hardwareInterface>hardware_interface/PositionJointInterface</hardwareInterface>
             <mechanicalReduction>1</mechanicalReduction>
