Commit message: Control exoskeleton with ROS

File: march_ws/src/march_description/urdf/march.xacro (robot description, xacro)
@@ -33,11 +33,4 @@
         <origin xyz="0 0 ${lower_leg_height+upper_leg_height}" rpy="0 0 0"/>
     </joint>
-    <!--<joint name="right_hip" type="revolute">-->
-        <!--<parent link="hip"/>-->
-        <!--<child link="upper_leg_right"/>-->
-        <!--<origin xyz="0 0 ${lower_leg_height+upper_leg_height}" rpy="0 0 0"/>-->
-        <!--<axis xyz="0 1 0"/>-->
-        <!--<limit velocity="${hip_velocity_limit}" effort="${hip_effort_limit}" lower="${hip_rotation_lower_limit}" upper="${hip_rotation_upper_limit}"/>-->
-    <!--</joint>-->
     <joint name="left_hip" type="revolute">
         <parent link="hip_bone"/>
@@ -243,13 +236,13 @@
         </inertial>
     </link>
-    <transmission name="left_hip">
-        <type>transmission_interface/SimpleTransmission</type>
-        <joint name="left_hip">
-            <hardwareInterface>hardware_interface/PositionJointInterface</hardwareInterface>
-        </joint>
-        <actuator name="left_hip_motor">
-            <hardwareInterface>hardware_interface/PositionJointInterface</hardwareInterface>
-            <mechanicalReduction>1</mechanicalReduction>
-        </actuator>
-    </transmission>
+    <!--<transmission name="left_hip">-->
+        <!--<type>transmission_interface/SimpleTransmission</type>-->
+        <!--<joint name="left_hip">-->
+            <!--<hardwareInterface>hardware_interface/PositionJointInterface</hardwareInterface>-->
+        <!--</joint>-->
+        <!--<actuator name="left_hip_motor">-->
+            <!--<hardwareInterface>hardware_interface/PositionJointInterface</hardwareInterface>-->
+            <!--<mechanicalReduction>1</mechanicalReduction>-->
+        <!--</actuator>-->
+    <!--</transmission>-->
 </robot>

Commit message: Small example which loads a gaitfile and plays it in rviz

File: march_ws/src/march_description/urdf/march.xacro (robot description, xacro)
@@ -4,5 +4,5 @@
     <!-- Constants for robot dimensions -->
     <xacro:property name="PI" value="3.1415926535897931"/>
-    <xacro:property name="mass" value="1"/> <!-- arbitrary value for mass -->
+    <xacro:property name="mass" value="100"/> <!-- arbitrary value for mass -->
     <xacro:property name="width" value="0.1"/> <!-- Square dimensions (widthxwidth) of beams -->
     <xacro:property name="upper_leg_height" value="${0.37*3}"/>
@@ -10,16 +10,16 @@
     <xacro:property name="foot_height" value="${0.14*3}"/>
     <xacro:property name="hip_height" value="1"/>
-    <xacro:property name="hip_rotation_lower_limit" value="${0*pi/180}"/>
-    <xacro:property name="hip_rotation_upper_limit" value="${30*pi/180}"/>
-    <xacro:property name="hip_effort_limit" value="100.0"/>
-    <xacro:property name="hip_velocity_limit" value="10.0"/>
-    <xacro:property name="knee_rotation_lower_limit" value="${-50*pi/180}"/>
-    <xacro:property name="knee_rotation_upper_limit" value="${0*pi/180}"/>
-    <xacro:property name="knee_effort_limit" value="100.0"/>
-    <xacro:property name="knee_velocity_limit" value="10.0"/>
-    <xacro:property name="ankle_rotation_lower_limit" value="${0*pi/180}"/>
-    <xacro:property name="ankle_rotation_upper_limit" value="${30*pi/180}"/>
-    <xacro:property name="ankle_effort_limit" value="100.0"/>
-    <xacro:property name="ankle_velocity_limit" value="10.0"/>
+    <xacro:property name="hip_rotation_lower_limit" value="${-100*pi/180}"/>
+    <xacro:property name="hip_rotation_upper_limit" value="${90*pi/180}"/>
+    <xacro:property name="hip_effort_limit" value="1000.0"/>
+    <xacro:property name="hip_velocity_limit" value="1000.0"/>
+    <xacro:property name="knee_rotation_lower_limit" value="${-90*pi/180}"/>
+    <xacro:property name="knee_rotation_upper_limit" value="${90*pi/180}"/>
+    <xacro:property name="knee_effort_limit" value="1000.0"/>
+    <xacro:property name="knee_velocity_limit" value="1000.0"/>
+    <xacro:property name="ankle_rotation_lower_limit" value="${-50*pi/180}"/>
+    <xacro:property name="ankle_rotation_upper_limit" value="${90*pi/180}"/>
+    <xacro:property name="ankle_effort_limit" value="1000.0"/>
+    <xacro:property name="ankle_velocity_limit" value="1000.0"/>
     <xacro:property name="camera_link" value="0.05"/> <!-- Size of square 'camera' box -->
     <xacro:property name="axel_offset" value="0.05"/> <!-- Space btw top of beam and the each joint -->
@@ -44,5 +44,5 @@
         <child link="lower_leg_left"/>
         <origin xyz="0 0 ${-upper_leg_height}" rpy="0 0 0"/>
-        <axis xyz="0 1 0"/>
+        <axis xyz="0 -1 0"/>
         <limit velocity="${knee_velocity_limit}" effort="${knee_effort_limit}" lower="${knee_rotation_lower_limit}" upper="${knee_rotation_upper_limit}"/>
     </joint>
@@ -65,5 +65,5 @@
         <child link="lower_leg_right"/>
         <origin xyz="0 0 ${-upper_leg_height}" rpy="0 0 0"/>
-        <axis xyz="0 1 0"/>
+        <axis xyz="0 -1 0"/>
         <limit velocity="${knee_velocity_limit}" effort="${knee_effort_limit}" lower="${knee_rotation_lower_limit}" upper="${knee_rotation_upper_limit}"/>
     </joint>
@@ -236,13 +236,63 @@
         </inertial>
     </link>
-    <!--<transmission name="left_hip">-->
-        <!--<type>transmission_interface/SimpleTransmission</type>-->
-        <!--<joint name="left_hip">-->
-            <!--<hardwareInterface>hardware_interface/PositionJointInterface</hardwareInterface>-->
-        <!--</joint>-->
-        <!--<actuator name="left_hip_motor">-->
-            <!--<hardwareInterface>hardware_interface/PositionJointInterface</hardwareInterface>-->
-            <!--<mechanicalReduction>1</mechanicalReduction>-->
-        <!--</actuator>-->
-    <!--</transmission>-->
+    <transmission name="left_hip">
+        <type>transmission_interface/SimpleTransmission</type>
+        <joint name="left_hip">
+            <hardwareInterface>hardware_interface/PositionJointInterface</hardwareInterface>
+        </joint>
+        <actuator name="left_hip_motor">
+            <hardwareInterface>hardware_interface/PositionJointInterface</hardwareInterface>
+            <mechanicalReduction>1</mechanicalReduction>
+        </actuator>
+    </transmission>
+    <transmission name="left_knee">
+        <type>transmission_interface/SimpleTransmission</type>
+        <joint name="left_knee">
+            <hardwareInterface>hardware_interface/PositionJointInterface</hardwareInterface>
+        </joint>
+        <actuator name="left_knee_motor">
+            <hardwareInterface>hardware_interface/PositionJointInterface</hardwareInterface>
+            <mechanicalReduction>1</mechanicalReduction>
+        </actuator>
+    </transmission>
+    <transmission name="left_ankle">
+        <type>transmission_interface/SimpleTransmission</type>
+        <joint name="left_ankle">
+            <hardwareInterface>hardware_interface/PositionJointInterface</hardwareInterface>
+        </joint>
+        <actuator name="left_ankle_motor">
+            <hardwareInterface>hardware_interface/PositionJointInterface</hardwareInterface>
+            <mechanicalReduction>1</mechanicalReduction>
+        </actuator>
+    </transmission>
+    <transmission name="right_hip">
+        <type>transmission_interface/SimpleTransmission</type>
+        <joint name="right_hip">
+            <hardwareInterface>hardware_interface/PositionJointInterface</hardwareInterface>
+        </joint>
+        <actuator name="right_hip_motor">
+            <hardwareInterface>hardware_interface/PositionJointInterface</hardwareInterface>
+            <mechanicalReduction>1</mechanicalReduction>
+        </actuator>
+    </transmission>
+    <transmission name="right_knee">
+        <type>transmission_interface/SimpleTransmission</type>
+        <joint name="right_knee">
+            <hardwareInterface>hardware_interface/PositionJointInterface</hardwareInterface>
+        </joint>
+        <actuator name="right_knee_motor">
+            <hardwareInterface>hardware_interface/PositionJointInterface</hardwareInterface>
+            <mechanicalReduction>1</mechanicalReduction>
+        </actuator>
+    </transmission>
+    <transmission name="right_ankle">
+        <type>transmission_interface/SimpleTransmission</type>
+        <joint name="right_ankle">
+            <hardwareInterface>hardware_interface/PositionJointInterface</hardwareInterface>
+        </joint>
+        <actuator name="right_ankle_motor">
+            <hardwareInterface>hardware_interface/PositionJointInterface</hardwareInterface>
+            <mechanicalReduction>1</mechanicalReduction>
+        </actuator>
+    </transmission>
 </robot>

Commit message: Start gazebo not paused

File: march_ws/src/march_description/urdf/march.xacro (robot description, xacro)
@@ -28,5 +28,5 @@
     <!-- Used for fixing robot to Gazebo 'base_link' -->
     <link name="world"/>
-    <joint name="hip" type="fixed">
+    <joint name="hip" type="floating">
         <parent link="world"/>
         <child link="hip_bone"/>

Commit message: Effort control instead of postion control

File: march_ws/src/march_description/urdf/march.xacro (robot description, xacro)
@@ -4,5 +4,5 @@
     <!-- Constants for robot dimensions -->
     <xacro:property name="PI" value="3.1415926535897931"/>
-    <xacro:property name="mass" value="100"/> <!-- arbitrary value for mass -->
+    <xacro:property name="mass" value="1"/> <!-- arbitrary value for mass -->
     <xacro:property name="width" value="0.1"/> <!-- Square dimensions (widthxwidth) of beams -->
     <xacro:property name="upper_leg_height" value="${0.37*3}"/>
@@ -19,5 +19,5 @@
     <xacro:property name="knee_velocity_limit" value="1000.0"/>
     <xacro:property name="ankle_rotation_lower_limit" value="${-50*pi/180}"/>
-    <xacro:property name="ankle_rotation_upper_limit" value="${90*pi/180}"/>
+    <xacro:property name="ankle_rotation_upper_limit" value="${30*pi/180}"/>
     <xacro:property name="ankle_effort_limit" value="1000.0"/>
     <xacro:property name="ankle_velocity_limit" value="1000.0"/>
@@ -239,8 +239,8 @@
         <type>transmission_interface/SimpleTransmission</type>
         <joint name="left_hip">
-            <hardwareInterface>hardware_interface/PositionJointInterface</hardwareInterface>
+            <hardwareInterface>hardware_interface/EffortJointInterface</hardwareInterface>
         </joint>
         <actuator name="left_hip_motor">
-            <hardwareInterface>hardware_interface/PositionJointInterface</hardwareInterface>
+            <hardwareInterface>hardware_interface/EffortJointInterface</hardwareInterface>
             <mechanicalReduction>1</mechanicalReduction>
         </actuator>
@@ -249,8 +249,8 @@
         <type>transmission_interface/SimpleTransmission</type>
         <joint name="left_knee">
-            <hardwareInterface>hardware_interface/PositionJointInterface</hardwareInterface>
+            <hardwareInterface>hardware_interface/EffortJointInterface</hardwareInterface>
         </joint>
         <actuator name="left_knee_motor">
-            <hardwareInterface>hardware_interface/PositionJointInterface</hardwareInterface>
+            <hardwareInterface>hardware_interface/EffortJointInterface</hardwareInterface>
             <mechanicalReduction>1</mechanicalReduction>
         </actuator>
@@ -259,8 +259,8 @@
         <type>transmission_interface/SimpleTransmission</type>
         <joint name="left_ankle">
-            <hardwareInterface>hardware_interface/PositionJointInterface</hardwareInterface>
+            <hardwareInterface>hardware_interface/EffortJointInterface</hardwareInterface>
         </joint>
         <actuator name="left_ankle_motor">
-            <hardwareInterface>hardware_interface/PositionJointInterface</hardwareInterface>
+            <hardwareInterface>hardware_interface/EffortJointInterface</hardwareInterface>
             <mechanicalReduction>1</mechanicalReduction>
         </actuator>
@@ -269,8 +269,8 @@
         <type>transmission_interface/SimpleTransmission</type>
         <joint name="right_hip">
-            <hardwareInterface>hardware_interface/PositionJointInterface</hardwareInterface>
+            <hardwareInterface>hardware_interface/EffortJointInterface</hardwareInterface>
         </joint>
         <actuator name="right_hip_motor">
-            <hardwareInterface>hardware_interface/PositionJointInterface</hardwareInterface>
+            <hardwareInterface>hardware_interface/EffortJointInterface</hardwareInterface>
             <mechanicalReduction>1</mechanicalReduction>
         </actuator>
@@ -279,8 +279,8 @@
         <type>transmission_interface/SimpleTransmission</type>
         <joint name="right_knee">
-            <hardwareInterface>hardware_interface/PositionJointInterface</hardwareInterface>
+            <hardwareInterface>hardware_interface/EffortJointInterface</hardwareInterface>
         </joint>
         <actuator name="right_knee_motor">
-            <hardwareInterface>hardware_interface/PositionJointInterface</hardwareInterface>
+            <hardwareInterface>hardware_interface/EffortJointInterface</hardwareInterface>
             <mechanicalReduction>1</mechanicalReduction>
         </actuator>
@@ -289,8 +289,8 @@
         <type>transmission_interface/SimpleTransmission</type>
         <joint name="right_ankle">
-            <hardwareInterface>hardware_interface/PositionJointInterface</hardwareInterface>
+            <hardwareInterface>hardware_interface/EffortJointInterface</hardwareInterface>
         </joint>
         <actuator name="right_ankle_motor">
-            <hardwareInterface>hardware_interface/PositionJointInterface</hardwareInterface>
+            <hardwareInterface>hardware_interface/EffortJointInterface</hardwareInterface>
             <mechanicalReduction>1</mechanicalReduction>
         </actuator>

Commit message: Move ros control to march_control package

File: march_ws/src/march_description/urdf/march.xacro (robot description, xacro)
@@ -22,4 +22,5 @@
     <xacro:property name="ankle_effort_limit" value="1000.0"/>
     <xacro:property name="ankle_velocity_limit" value="1000.0"/>
+    <xacro:property name="hover_height" value="0.3"/>
     <xacro:property name="camera_link" value="0.05"/> <!-- Size of square 'camera' box -->
     <xacro:property name="axel_offset" value="0.05"/> <!-- Space btw top of beam and the each joint -->
@@ -28,8 +29,8 @@
     <!-- Used for fixing robot to Gazebo 'base_link' -->
     <link name="world"/>
-    <joint name="hip" type="floating">
+    <joint name="hip" type="fixed">
         <parent link="world"/>
         <child link="hip_bone"/>
-        <origin xyz="0 0 ${lower_leg_height+upper_leg_height}" rpy="0 0 0"/>
+        <origin xyz="0 0 ${lower_leg_height+upper_leg_height+hover_height}" rpy="0 0 0"/>
     </joint>
     <joint name="left_hip" type="revolute">
@@ -236,4 +237,5 @@
         </inertial>
     </link>
+    <!-- ROS Control plugin for Gazebo -->
     <transmission name="left_hip">
         <type>transmission_interface/SimpleTransmission</type>

Commit message: Update size of the exoskeleton URDF

File: march_ws/src/march_description/urdf/march.xacro (robot description, xacro)
@@ -5,9 +5,9 @@
     <xacro:property name="PI" value="3.1415926535897931"/>
     <xacro:property name="mass" value="1"/> <!-- arbitrary value for mass -->
-    <xacro:property name="width" value="0.1"/> <!-- Square dimensions (widthxwidth) of beams -->
-    <xacro:property name="upper_leg_height" value="${0.37*3}"/>
-    <xacro:property name="lower_leg_height" value="${0.41*3}"/>
-    <xacro:property name="foot_height" value="${0.14*3}"/>
-    <xacro:property name="hip_height" value="1"/>
+    <xacro:property name="width" value="0.05"/> <!-- Square dimensions (widthxwidth) of beams -->
+    <xacro:property name="upper_leg_height" value="${0.37*1}"/>
+    <xacro:property name="lower_leg_height" value="${0.41*1}"/>
+    <xacro:property name="foot_height" value="${0.14*1}"/>
+    <xacro:property name="hip_height" value="0.3"/>
     <xacro:property name="hip_rotation_lower_limit" value="${-100*pi/180}"/>
     <xacro:property name="hip_rotation_upper_limit" value="${90*pi/180}"/>
