Commit message: Add stl files to the URDF

File: march_description/urdf/march-iii.xacro (robot description, xacro)
@@ -127,5 +127,5 @@
         <parent link="ankle_plate_right"/>
         <child link="foot_right"/>
-        <origin xyz="0 0 ${-ankle_pslate_height}" rpy="0 0 0"/>
+        <origin xyz="0 0 ${-ankle_plate_height}" rpy="0 0 0"/>
     </joint>
     <!-- give colors to some links in gazebo -->
@@ -142,7 +142,8 @@
     <link name="hip_base">
         <visual>
-            <origin xyz="0 0 0" rpy="0 0 0"/>
-            <geometry>
-                <box size="${width} ${hip_base_height} ${width}"/>
+            <origin xyz="0 0 0" rpy="0 0 ${-pi/2}"/>
+            <geometry>
+<!--                <box size="${width} ${hip_base_height} ${width}"/>-->
+                <mesh filename="package://march_description/urdf/stl-files/HipBase.stl" scale="1.15 1.15 1.15"/>
             </geometry>
         </visual>
@@ -159,7 +160,8 @@
     <link name="hip_aa_frame_left_side">
         <visual>
-            <origin xyz="0 ${-hip_aa_frame_height/2} 0" rpy="0 0 0"/>
-            <geometry>
-                <box size="${width} ${hip_aa_frame_height} ${width}"/>
+            <origin xyz="0 0 0" rpy="0 0 ${-pi/2}"/>
+            <geometry>
+<!--                <box size="${width} ${hip_aa_frame_height} ${width}"/>-->
+                <mesh filename="package://march_description/urdf/stl-files/HipLeft.stl" scale="1.15 1.15 1.15"/>
             </geometry>
         </visual>
@@ -174,10 +176,10 @@
     </link>
     <link name="hip_aa_frame_left_front">
-        <visual>
-            <origin xyz="${-hip_aa_frame_width/2} 0 0" rpy="0 0 0"/>
-            <geometry>
-                <box size="${hip_aa_frame_width} ${width} ${width}"/>
-            </geometry>
-        </visual>
+<!--        <visual>-->
+<!--            <origin xyz="${-hip_aa_frame_width/2} 0 0" rpy="0 0 0"/>-->
+<!--            <geometry>-->
+<!--                <box size="${hip_aa_frame_width} ${width} ${width}"/>-->
+<!--            </geometry>-->
+<!--        </visual>-->
         <inertial>
             <origin xyz="${-hip_aa_frame_width/2} 0 0" rpy="0 0 0"/>
@@ -192,8 +194,8 @@
     <link name="upper_leg_left">
         <visual>
-            <origin xyz="0 0 ${-0.9*upper_leg_height}" rpy="0 0 1.8"/>
+            <origin xyz="0 0 0" rpy="0 0 ${-pi/2}"/>
             <geometry>
                 <!--                <box size="${width} ${width} ${upper_leg_height}"/>-->
-                <mesh filename="package://march_description/urdf/stl-files/UpperLegRight1.stl" scale="1.2 1.2 1.2"/>
+                <mesh filename="package://march_description/urdf/stl-files/UpperLegLeft.stl" scale="1.15 1.15 1.15"/>
                 <!--                TODO: both upper legs are the same. So one of them has to be replaced.-->
             </geometry>
@@ -217,8 +219,8 @@
     <link name="lower_leg_left">
         <visual>
-            <origin xyz="0 0 ${-lower_leg_height/2}" rpy="0 0 0"/>
-            <geometry>
-                <box size="${width} ${width} ${lower_leg_height}"/>
-                <!--                <mesh filename="package://march_description/urdf/stl-files/LowerLeg.stl" scale="1.2 1.2 1.2"/>-->
+            <origin xyz="0 0 0" rpy="0 0 ${-pi/2}"/>
+            <geometry>
+<!--                <box size="${width} ${width} ${lower_leg_height}"/>-->
+                <mesh filename="package://march_description/urdf/stl-files/LowerLegLeft.stl" scale="1.15 1.15 1.15"/>
             </geometry>
         </visual>
@@ -235,8 +237,8 @@
     <link name="ankle_plate_left">
         <visual>
-            <origin xyz="0 0 ${-ankle_plate_height/2}" rpy="0 0 0"/>
-            <geometry>
-                <box size="${width} ${width} ${ankle_plate_height}"/>
-                <!--                <mesh filename="package://march_description/urdf/stl-files/LowerLeg.stl" scale="1.2 1.2 1.2"/>-->
+            <origin xyz="0 0 0" rpy="0 0 ${-pi/2}"/>
+            <geometry>
+<!--                <box size="${width} ${width} ${ankle_plate_height}"/>-->
+                <mesh filename="package://march_description/urdf/stl-files/FootLeft.stl" scale="1.15 1.15 1.15"/>
             </geometry>
         </visual>
@@ -252,10 +254,10 @@
     <!-- Foot Left -->
     <link name="foot_left">
-        <visual>
-            <origin xyz="${-foot_height/2} 0 0" rpy="0 0 0"/>
-            <geometry>
-                <box size="${foot_height} ${width} ${width}"/>
-            </geometry>
-        </visual>
+<!--        <visual>-->
+<!--            <origin xyz="${-foot_height/2} 0 0" rpy="0 0 0"/>-->
+<!--            <geometry>-->
+<!--                <box size="${foot_height} ${width} ${width}"/>-->
+<!--            </geometry>-->
+<!--        </visual>-->
         <inertial>
             <origin xyz="${-foot_height/2} 0 0" rpy="0 0 0"/>
@@ -276,11 +278,12 @@
     <link name="hip_aa_frame_right_side">
         <visual>
+            <origin xyz="0 0 0" rpy="0 0 ${-pi/2}"/>
+            <geometry>
+<!--                <box size="${width} ${hip_aa_frame_height} ${width}"/>-->
+                <mesh filename="package://march_description/urdf/stl-files/HipRight.stl" scale="1.15 1.15 1.15"/>
+            </geometry>
+        </visual>
+        <inertial>
             <origin xyz="0 ${hip_aa_frame_height/2} 0" rpy="0 0 0"/>
-            <geometry>
-                <box size="${width} ${hip_aa_frame_height} ${width}"/>
-            </geometry>
-        </visual>
-        <inertial>
-            <origin xyz="0 ${hip_aa_frame_height/2} 0" rpy="0 0 0"/>
             <mass value="${mass}"/>
             <inertia
@@ -291,10 +294,10 @@
     </link>
     <link name="hip_aa_frame_right_front">
-        <visual>
-            <origin xyz="${-hip_aa_frame_width/2} 0 0" rpy="0 0 0"/>
-            <geometry>
-                <box size="${hip_aa_frame_width} ${width} ${width}"/>
-            </geometry>
-        </visual>
+<!--        <visual>-->
+<!--            <origin xyz="${-hip_aa_frame_width/2} 0 0" rpy="0 0 0"/>-->
+<!--            <geometry>-->
+<!--                <box size="${hip_aa_frame_width} ${width} ${width}"/>-->
+<!--            </geometry>-->
+<!--        </visual>-->
         <inertial>
             <origin xyz="${-hip_aa_frame_width/2} 0 0" rpy="0 0 0"/>
@@ -309,8 +312,8 @@
     <link name="upper_leg_right">
         <visual>
-            <origin xyz="0 0 ${-0.9*upper_leg_height}" rpy="0 0 -1.8"/>
+            <origin xyz="0 0 0" rpy="0 0 ${-pi/2}"/>
             <geometry>
                 <!--                <box size="${width} ${width} ${upper_leg_height}"/>-->
-                <mesh filename="package://march_description/urdf/stl-files/UpperLegRight1.stl" scale="1.2 1.2 1.2"/>
+                <mesh filename="package://march_description/urdf/stl-files/UpperLegRight.stl" scale="1.15 1.15 1.15"/>
             </geometry>
         </visual>
@@ -333,7 +336,8 @@
     <link name="lower_leg_right">
         <visual>
-            <origin xyz="0 0 ${-lower_leg_height/2}" rpy="0 0 0"/>
-            <geometry>
-                <box size="${width} ${width} ${lower_leg_height}"/>
+            <origin xyz="0 0 0" rpy="0 0 ${-pi/2}"/>
+            <geometry>
+<!--                <box size="${width} ${width} ${lower_leg_height}"/>-->
+                <mesh filename="package://march_description/urdf/stl-files/LowerLegRight.stl" scale="1.15 1.15 1.15"/>
             </geometry>
         </visual>
@@ -350,8 +354,8 @@
     <link name="ankle_plate_right">
         <visual>
-            <origin xyz="0 0 ${-ankle_plate_height/2}" rpy="0 0 0"/>
-            <geometry>
-                <box size="${width} ${width} ${ankle_plate_height}"/>
-                <!--                <mesh filename="package://march_description/urdf/stl-files/LowerLeg.stl" scale="1.2 1.2 1.2"/>-->
+            <origin xyz="0 0 0" rpy="0 0 ${-pi/2}"/>
+            <geometry>
+<!--                <box size="${width} ${width} ${ankle_plate_height}"/>-->
+                <mesh filename="package://march_description/urdf/stl-files/FootRight.stl" scale="1.15 1.15 1.15"/>
             </geometry>
         </visual>
@@ -367,10 +371,10 @@
     <!-- Foot Right -->
     <link name="foot_right">
-        <visual>
-            <origin xyz="${-foot_height/2} 0 0" rpy="0 0 0"/>
-            <geometry>
-                <box size="${foot_height} ${width} ${width}"/>
-            </geometry>
-        </visual>
+<!--        <visual>-->
+<!--            <origin xyz="${-foot_height/2} 0 0" rpy="0 0 0"/>-->
+<!--            <geometry>-->
+<!--                <box size="${foot_height} ${width} ${width}"/>-->
+<!--            </geometry>-->
+<!--        </visual>-->
         <inertial>
             <origin xyz="${-foot_height/2} 0 0" rpy="0 0 0"/>
