Commit message: add correct name for joint lin vs rot in xacro

File: march_description/urdf/test-joint-lin.xacro (robot description, xacro)
@@ -31,5 +31,5 @@
         <origin xyz="0 0 ${hover_height}" rpy="0 0 0"/>
     </joint>
-    <joint name="test_joint" type="revolute">
+    <joint name="test_joint_lin" type="revolute">
         <parent link="joint_base"/>
         <child link="bar"/>

File: march_description/urdf/test-joint-rot.xacro (robot description, xacro)
@@ -31,5 +31,5 @@
         <origin xyz="0 0 ${hover_height}" rpy="0 0 0"/>
     </joint>
-    <joint name="test_joint" type="revolute">
+    <joint name="test_joint_rot" type="revolute">
         <parent link="joint_base"/>
         <child link="bar"/>
