Commit message: set joint limits in test-joint.xacro

File: march_description/urdf/test-joint.xacro (robot description, xacro)
@@ -13,8 +13,10 @@
     <xacro:property name="bar_mass" value="1.080"/>
     <xacro:property name="bar_width" value="0.05"/>
-    <xacro:property name="joint_lower_limit" value="${-15*pi/180}"/> <!-- rad -->
-    <xacro:property name="joint_upper_limit" value="${105*pi/180}"/> <!-- rad -->
-    <xacro:property name="joint_effort_limit" value="1000.0"/> <!-- Rad -->
-    <xacro:property name="joint_velocity_limit" value="1000.0"/> <!-- rad/s -->
+    <xacro:property name="join_buffer" value="${5*pi/180}"/> <!-- rad -->
+    <xacro:property name="joint_lower_limit" value="-0.04"/> <!-- rad -->
+    <xacro:property name="joint_upper_limit" value="1.75"/> <!-- rad -->
+    <xacro:property name="joint_effort_limit" value="1000.0"/>
+    <xacro:property name="joint_velocity_limit" value="0.2"/> <!-- rad/s -->
+    <xacro:property name="joint_lower_limit" value="${-15*pi/180}"/>
     <xacro:property name="hover_height" value="0.5"/>
     <!-- Import all Gazebo-customization elements, including Gazebo colors -->
@@ -36,4 +38,5 @@
         <axis xyz="0 1 0"/>
         <limit velocity="${joint_velocity_limit}" effort="${joint_effort_limit}" lower="${joint_lower_limit}" upper="${joint_upper_limit}"/>
+        <safety_controller soft_lower_limit="${joint_lower_limit + join_buffer}" soft_upper_limit="${joint_upper_limit - join_buffer}" k_position="100" k_velocity="10" />
     </joint>
     <!-- give colors to some links in gazebo -->

Commit message: remove double attribute

File: march_description/urdf/test-joint.xacro (robot description, xacro)
@@ -18,5 +18,4 @@
     <xacro:property name="joint_effort_limit" value="1000.0"/>
     <xacro:property name="joint_velocity_limit" value="0.2"/> <!-- rad/s -->
-    <xacro:property name="joint_lower_limit" value="${-15*pi/180}"/>
     <xacro:property name="hover_height" value="0.5"/>
     <!-- Import all Gazebo-customization elements, including Gazebo colors -->

Commit message: Correct a typo and increase the velocity limit and decrease the k position value

File: march_description/urdf/test-joint.xacro (robot description, xacro)
@@ -13,9 +13,9 @@
     <xacro:property name="bar_mass" value="1.080"/>
     <xacro:property name="bar_width" value="0.05"/>
-    <xacro:property name="join_buffer" value="${5*pi/180}"/> <!-- rad -->
+    <xacro:property name="joint_buffer" value="${5*pi/180}"/> <!-- rad -->
     <xacro:property name="joint_lower_limit" value="-0.04"/> <!-- rad -->
     <xacro:property name="joint_upper_limit" value="1.75"/> <!-- rad -->
     <xacro:property name="joint_effort_limit" value="1000.0"/>
-    <xacro:property name="joint_velocity_limit" value="0.2"/> <!-- rad/s -->
+    <xacro:property name="joint_velocity_limit" value="1.5"/> <!-- rad/s -->
     <xacro:property name="hover_height" value="0.5"/>
     <!-- Import all Gazebo-customization elements, including Gazebo colors -->
@@ -37,5 +37,5 @@
         <axis xyz="0 1 0"/>
         <limit velocity="${joint_velocity_limit}" effort="${joint_effort_limit}" lower="${joint_lower_limit}" upper="${joint_upper_limit}"/>
-        <safety_controller soft_lower_limit="${joint_lower_limit + join_buffer}" soft_upper_limit="${joint_upper_limit - join_buffer}" k_position="100" k_velocity="10" />
+        <safety_controller soft_lower_limit="${joint_lower_limit + joint_buffer}" soft_upper_limit="${joint_upper_limit - joint_buffer}" k_position="10" k_velocity="10" />
     </joint>
     <!-- give colors to some links in gazebo -->

Commit message: fix limits of test joint (adjusted for limit switches)

File: march_description/urdf/test-joint.xacro (robot description, xacro)
@@ -13,7 +13,7 @@
     <xacro:property name="bar_mass" value="1.080"/>
     <xacro:property name="bar_width" value="0.05"/>
-    <xacro:property name="joint_buffer" value="${5*pi/180}"/> <!-- rad -->
-    <xacro:property name="joint_lower_limit" value="-0.04"/> <!-- rad -->
-    <xacro:property name="joint_upper_limit" value="1.75"/> <!-- rad -->
+    <xacro:property name="joint_buffer" value="${3*pi/180}"/> <!-- rad -->
+    <xacro:property name="joint_lower_limit" value="-0.5673"/> <!-- rad -->
+    <xacro:property name="joint_upper_limit" value="0.3549"/> <!-- rad -->
     <xacro:property name="joint_effort_limit" value="1000.0"/>
     <xacro:property name="joint_velocity_limit" value="1.5"/> <!-- rad/s -->

Commit message: Implement effortsoftlimitsinterface after computing the command, adjust k_velocity, adjust p value

File: march_description/urdf/test-joint.xacro (robot description, xacro)
@@ -15,7 +15,7 @@
     <xacro:property name="joint_buffer" value="${3*pi/180}"/> <!-- rad -->
     <xacro:property name="joint_lower_limit" value="-0.5673"/> <!-- rad -->
-    <xacro:property name="joint_upper_limit" value="0.3549"/> <!-- rad -->
-    <xacro:property name="joint_effort_limit" value="1000.0"/>
-    <xacro:property name="joint_velocity_limit" value="1.5"/> <!-- rad/s -->
+    <xacro:property name="joint_upper_limit" value="0"/> <!-- rad -->
+    <xacro:property name="joint_effort_limit" value="8000.0"/>
+    <xacro:property name="joint_velocity_limit" value="0.5"/> <!-- rad/s -->
     <xacro:property name="hover_height" value="0.5"/>
     <!-- Import all Gazebo-customization elements, including Gazebo colors -->
@@ -36,6 +36,6 @@
         <origin xyz="0 ${-joint_base_width} 0" rpy="0 0 0"/>
         <axis xyz="0 1 0"/>
-        <limit velocity="${joint_velocity_limit}" effort="${joint_effort_limit}" lower="${joint_lower_limit}" upper="${joint_upper_limit}"/>
-        <safety_controller soft_lower_limit="${joint_lower_limit + joint_buffer}" soft_upper_limit="${joint_upper_limit - joint_buffer}" k_position="10" k_velocity="10" />
+        <limit velocity="${joint_velocity_limit}" effort="${joint_effort_limit}" lower="${joint_lower_limit - joint_buffer*2}" upper="${joint_upper_limit + joint_buffer*2}"/>
+        <safety_controller soft_lower_limit="${joint_lower_limit + joint_buffer}" soft_upper_limit="${joint_upper_limit - joint_buffer}" k_position="5" k_velocity="20000" />
     </joint>
     <!-- give colors to some links in gazebo -->

Commit message: Change joint upper limit back to the normal limit

File: march_description/urdf/test-joint.xacro (robot description, xacro)
@@ -15,5 +15,5 @@
     <xacro:property name="joint_buffer" value="${3*pi/180}"/> <!-- rad -->
     <xacro:property name="joint_lower_limit" value="-0.5673"/> <!-- rad -->
-    <xacro:property name="joint_upper_limit" value="0"/> <!-- rad -->
+    <xacro:property name="joint_upper_limit" value="0.3549"/> <!-- rad -->
     <xacro:property name="joint_effort_limit" value="8000.0"/>
     <xacro:property name="joint_velocity_limit" value="0.5"/> <!-- rad/s -->

Commit message: Adjust effort limit for test joint

File: march_description/urdf/test-joint.xacro (robot description, xacro)
@@ -16,5 +16,5 @@
     <xacro:property name="joint_lower_limit" value="-0.5673"/> <!-- rad -->
     <xacro:property name="joint_upper_limit" value="0.3549"/> <!-- rad -->
-    <xacro:property name="joint_effort_limit" value="8000.0"/>
+    <xacro:property name="joint_effort_limit" value="21840"/> <!-- IU = 20 A -->
     <xacro:property name="joint_velocity_limit" value="0.5"/> <!-- rad/s -->
     <xacro:property name="hover_height" value="0.5"/>

Commit message: Update march_description/urdf/test-joint.xacro
Co-Authored-By: sopje <44405009+sopje@users.noreply.github.com>

File: march_description/urdf/test-joint.xacro (robot description, xacro)
@@ -17,5 +17,5 @@
     <xacro:property name="joint_upper_limit" value="0.3549"/> <!-- rad -->
     <xacro:property name="joint_effort_limit" value="21840"/> <!-- IU = 20 A -->
-    <xacro:property name="joint_velocity_limit" value="0.5"/> <!-- rad/s -->
+    <xacro:property name="joint_velocity_limit" value="2.0"/> <!-- rad/s -->
     <xacro:property name="hover_height" value="0.5"/>
     <!-- Import all Gazebo-customization elements, including Gazebo colors -->
