Commit message: add fully written linear and rotational and replace testsetup naming by testjoint

File: march_description/urdf/test-joint-linear.xacro (robot description, xacro)
@@ -14,8 +14,8 @@
     <xacro:property name="bar_width" value="0.05"/>
     <xacro:property name="joint_buffer" value="${3*pi/180}"/> <!-- rad -->
-    <xacro:property name="joint_lower_limit" value="-0.5673"/> <!-- rad -->
-    <xacro:property name="joint_upper_limit" value="0.3549"/> <!-- rad -->
-    <xacro:property name="joint_effort_limit" value="1000.0"/>
-    <xacro:property name="joint_velocity_limit" value="1.5"/> <!-- rad/s -->
+    <xacro:property name="joint_lower_limit" value="${-8.5*pi/180}"/> <!-- rad -->
+    <xacro:property name="joint_upper_limit" value="${8.5*pi/180}"/> <!-- rad -->
+    <xacro:property name="joint_effort_limit" value="10927.0"/>
+    <xacro:property name="joint_velocity_limit" value="1.0"/> <!-- rad/s -->
     <xacro:property name="hover_height" value="0.5"/>
     <!-- Import all Gazebo-customization elements, including Gazebo colors -->
@@ -31,5 +31,5 @@
         <origin xyz="0 0 ${hover_height}" rpy="0 0 0"/>
     </joint>
-    <joint name="test_joint_rot" type="revolute">
+    <joint name="linear_joint" type="revolute">
         <parent link="joint_base"/>
         <child link="bar"/>
@@ -58,5 +58,5 @@
                     iyy="${joint_base_mass / 12.0 * (2*(joint_base_width*joint_base_width))}" iyz="0.0"
                     izz="${joint_base_mass / 12.0 * (2*(joint_base_width*joint_base_width))}"/>
-                                                <!--(joint_base_width*joint_base_width + joint_base_width*joint_base_width)-->
+            <!--(joint_base_width*joint_base_width + joint_base_width*joint_base_width)-->
         </inertial>
     </link>
@@ -81,5 +81,5 @@
     <transmission name="test_joint">
         <type>transmission_interface/SimpleTransmission</type>
-        <joint name="test_joint">
+        <joint name="linear_joint">
             <hardwareInterface>hardware_interface/EffortJointInterface</hardwareInterface>
         </joint>

File: march_description/urdf/test-joint-rotational.xacro (robot description, xacro)
@@ -14,8 +14,8 @@
     <xacro:property name="bar_width" value="0.05"/>
     <xacro:property name="joint_buffer" value="${3*pi/180}"/> <!-- rad -->
-    <xacro:property name="joint_lower_limit" value="${-8.5*pi/180}"/> <!-- rad -->
-    <xacro:property name="joint_upper_limit" value="${8.5*pi/180}"/> <!-- rad -->
-    <xacro:property name="joint_effort_limit" value="10927.0"/>
-    <xacro:property name="joint_velocity_limit" value="1.0"/> <!-- rad/s -->
+    <xacro:property name="joint_lower_limit" value="-0.5673"/> <!-- rad -->
+    <xacro:property name="joint_upper_limit" value="0.3549"/> <!-- rad -->
+    <xacro:property name="joint_effort_limit" value="1000.0"/>
+    <xacro:property name="joint_velocity_limit" value="1.5"/> <!-- rad/s -->
     <xacro:property name="hover_height" value="0.5"/>
     <!-- Import all Gazebo-customization elements, including Gazebo colors -->
@@ -31,5 +31,5 @@
         <origin xyz="0 0 ${hover_height}" rpy="0 0 0"/>
     </joint>
-    <joint name="test_joint_lin" type="revolute">
+    <joint name="rotational_joint" type="revolute">
         <parent link="joint_base"/>
         <child link="bar"/>
@@ -58,5 +58,5 @@
                     iyy="${joint_base_mass / 12.0 * (2*(joint_base_width*joint_base_width))}" iyz="0.0"
                     izz="${joint_base_mass / 12.0 * (2*(joint_base_width*joint_base_width))}"/>
-            <!--(joint_base_width*joint_base_width + joint_base_width*joint_base_width)-->
+                                                <!--(joint_base_width*joint_base_width + joint_base_width*joint_base_width)-->
         </inertial>
     </link>
@@ -81,5 +81,5 @@
     <transmission name="test_joint">
         <type>transmission_interface/SimpleTransmission</type>
-        <joint name="test_joint">
+        <joint name="rotational_joint">
             <hardwareInterface>hardware_interface/EffortJointInterface</hardwareInterface>
         </joint>
