Commit message: Change name urdf, remove comments, add collision

File: march_description/urdf/march-iv.xacro (robot description, xacro)
@@ -144,5 +144,4 @@
             <origin xyz="0 0 0" rpy="0 0 ${-pi/2}"/>
             <geometry>
-<!--                <box size="${width} ${hip_base_height} ${width}"/>-->
                 <mesh filename="package://march_description/urdf/stl-files/HipBase.stl" scale="1.15 1.15 1.15"/>
             </geometry>
@@ -156,4 +155,10 @@
                     izz="${mass / 12.0 * (width*width + width*width)}"/>
         </inertial>
+        <collision>
+            <origin xyz="0 0 0" rpy="0 0 0"/>
+            <geometry>
+                <box size="${width} ${hip_base_height} ${width}"/>
+            </geometry>
+        </collision>
     </link>
     <!-- Left Moving Hip-->
@@ -162,24 +167,23 @@
             <origin xyz="0 0 0" rpy="0 0 ${-pi/2}"/>
             <geometry>
-<!--                <box size="${width} ${hip_aa_frame_height} ${width}"/>-->
                 <mesh filename="package://march_description/urdf/stl-files/HipLeft.stl" scale="1.15 1.15 1.15"/>
             </geometry>
         </visual>
         <inertial>
-            <origin xyz="0 ${hip_aa_frame_height/2} 0" rpy="0 0 0"/>
-            <mass value="${mass}"/>
-            <inertia
-                    ixx="${mass / 12.0 * (width*width + lower_leg_height*lower_leg_height)}" ixy="0.0" ixz="0.0"
-                    iyy="${mass / 12.0 * (lower_leg_height*lower_leg_height + width*width)}" iyz="0.0"
-                    izz="${mass / 12.0 * (width*width + width*width)}"/>
-        </inertial>
+            <origin xyz="0 ${-hip_aa_frame_height/2} 0" rpy="0 0 0"/>
+            <mass value="${mass}"/>
+            <inertia
+                    ixx="${mass / 12.0 * (width*width + lower_leg_height*lower_leg_height)}" ixy="0.0" ixz="0.0"
+                    iyy="${mass / 12.0 * (lower_leg_height*lower_leg_height + width*width)}" iyz="0.0"
+                    izz="${mass / 12.0 * (width*width + width*width)}"/>
+        </inertial>
+        <collision>
+            <origin xyz="0 ${-hip_aa_frame_height/2} 0" rpy="0 0 0"/>
+            <geometry>
+                <box size="${width} ${hip_aa_frame_height} ${width}"/>
+            </geometry>
+        </collision>
     </link>
     <link name="hip_aa_frame_left_front">
-<!--        <visual>-->
-<!--            <origin xyz="${-hip_aa_frame_width/2} 0 0" rpy="0 0 0"/>-->
-<!--            <geometry>-->
-<!--                <box size="${hip_aa_frame_width} ${width} ${width}"/>-->
-<!--            </geometry>-->
-<!--        </visual>-->
         <inertial>
             <origin xyz="${-hip_aa_frame_width/2} 0 0" rpy="0 0 0"/>
@@ -190,4 +194,10 @@
                     izz="${mass / 12.0 * (width*width + width*width)}"/>
         </inertial>
+        <collision>
+            <origin xyz="${-hip_aa_frame_width/2} 0 0" rpy="0 0 0"/>
+            <geometry>
+                <box size="${hip_aa_frame_width} ${width} ${width}"/>
+            </geometry>
+        </collision>
     </link>
     <!-- Upper Leg Left-->
@@ -196,15 +206,7 @@
             <origin xyz="0 0 0" rpy="0 0 ${-pi/2}"/>
             <geometry>
-                <!--                <box size="${width} ${width} ${upper_leg_height}"/>-->
                 <mesh filename="package://march_description/urdf/stl-files/UpperLegLeft.stl" scale="1.15 1.15 1.15"/>
-                <!--                TODO: both upper legs are the same. So one of them has to be replaced.-->
-            </geometry>
-        </visual>
-        <collision>
-            <origin xyz="0 0 ${-upper_leg_height/2}" rpy="0 0 0"/>
-            <geometry>
-                <box size="${width} ${width} ${upper_leg_height}"/>
-            </geometry>
-        </collision>
+            </geometry>
+        </visual>
         <inertial>
             <origin xyz="0 0 ${-upper_leg_height/2}" rpy="0 0 0"/>
@@ -215,4 +217,10 @@
                     izz="${mass / 12.0 * (width*width + width*width)}"/>
         </inertial>
+        <collision>
+            <origin xyz="0 0 ${-upper_leg_height/2}" rpy="0 0 0"/>
+            <geometry>
+                <box size="${width} ${width} ${upper_leg_height}"/>
+            </geometry>
+        </collision>
     </link>
     <!-- Lower Leg Left -->
@@ -221,5 +229,4 @@
             <origin xyz="0 0 0" rpy="0 0 ${-pi/2}"/>
             <geometry>
-<!--                <box size="${width} ${width} ${lower_leg_height}"/>-->
                 <mesh filename="package://march_description/urdf/stl-files/LowerLegLeft.stl" scale="1.15 1.15 1.15"/>
             </geometry>
@@ -233,4 +240,10 @@
                     izz="${mass / 12.0 * (width*width + width*width)}"/>
         </inertial>
+        <collision>
+            <origin xyz="0 0 ${-lower_leg_height/2}" rpy="0 0 0"/>
+            <geometry>
+                <box size="${width} ${width} ${lower_leg_height}"/>
+            </geometry>
+        </collision>
     </link>
     <!-- Lower Leg Left -->
@@ -239,5 +252,4 @@
             <origin xyz="0 0 0" rpy="0 0 ${-pi/2}"/>
             <geometry>
-<!--                <box size="${width} ${width} ${ankle_plate_height}"/>-->
                 <mesh filename="package://march_description/urdf/stl-files/FootLeft.stl" scale="1.15 1.15 1.15"/>
             </geometry>
@@ -251,13 +263,13 @@
                     izz="${mass / 12.0 * (width*width + width*width)}"/>
         </inertial>
+        <collision>
+            <origin xyz="0 0 ${-ankle_plate_height/2}" rpy="0 0 0"/>
+            <geometry>
+                <box size="${width} ${width} ${ankle_plate_height}"/>
+            </geometry>
+        </collision>
     </link>
     <!-- Foot Left -->
     <link name="foot_left">
-<!--        <visual>-->
-<!--            <origin xyz="${-foot_height/2} 0 0" rpy="0 0 0"/>-->
-<!--            <geometry>-->
-<!--                <box size="${foot_height} ${width} ${width}"/>-->
-<!--            </geometry>-->
-<!--        </visual>-->
         <inertial>
             <origin xyz="${-foot_height/2} 0 0" rpy="0 0 0"/>
@@ -270,4 +282,5 @@
         </inertial>
         <collision>
+            <origin xyz="${-foot_height/2} 0 0" rpy="0 0 0"/>
             <geometry>
                 <box size="${foot_height} ${width} ${width}"/>
@@ -280,5 +293,4 @@
             <origin xyz="0 0 0" rpy="0 0 ${-pi/2}"/>
             <geometry>
-<!--                <box size="${width} ${hip_aa_frame_height} ${width}"/>-->
                 <mesh filename="package://march_description/urdf/stl-files/HipRight.stl" scale="1.15 1.15 1.15"/>
             </geometry>
@@ -292,12 +304,12 @@
                     izz="${mass / 12.0 * (width*width + width*width)}"/>
         </inertial>
+        <collision>
+            <origin xyz="0 ${hip_aa_frame_height/2} 0" rpy="0 0 0"/>
+            <geometry>
+                <box size="${width} ${hip_aa_frame_height} ${width}"/>
+            </geometry>
+        </collision>
     </link>
     <link name="hip_aa_frame_right_front">
-<!--        <visual>-->
-<!--            <origin xyz="${-hip_aa_frame_width/2} 0 0" rpy="0 0 0"/>-->
-<!--            <geometry>-->
-<!--                <box size="${hip_aa_frame_width} ${width} ${width}"/>-->
-<!--            </geometry>-->
-<!--        </visual>-->
         <inertial>
             <origin xyz="${-hip_aa_frame_width/2} 0 0" rpy="0 0 0"/>
@@ -308,4 +320,10 @@
                     izz="${mass / 12.0 * (width*width + width*width)}"/>
         </inertial>
+        <collision>
+            <origin xyz="${-hip_aa_frame_width/2} 0 0" rpy="0 0 0"/>
+            <geometry>
+                <box size="${hip_aa_frame_width} ${width} ${width}"/>
+            </geometry>
+        </collision>
     </link>
     <!-- Upper Leg Right-->
@@ -314,14 +332,7 @@
             <origin xyz="0 0 0" rpy="0 0 ${-pi/2}"/>
             <geometry>
-                <!--                <box size="${width} ${width} ${upper_leg_height}"/>-->
                 <mesh filename="package://march_description/urdf/stl-files/UpperLegRight.stl" scale="1.15 1.15 1.15"/>
             </geometry>
         </visual>
-        <collision>
-            <origin xyz="0 0 ${-upper_leg_height/2}" rpy="0 0 0"/>
-            <geometry>
-                <box size="${width} ${width} ${upper_leg_height}"/>
-            </geometry>
-        </collision>
         <inertial>
             <origin xyz="0 0 ${-upper_leg_height/2}" rpy="0 0 0"/>
@@ -332,4 +343,10 @@
                     izz="${mass / 12.0 * (width*width + width*width)}"/>
         </inertial>
+        <collision>
+            <origin xyz="0 0 ${-upper_leg_height/2}" rpy="0 0 0"/>
+            <geometry>
+                <box size="${width} ${width} ${upper_leg_height}"/>
+            </geometry>
+        </collision>
     </link>
     <!-- Lower Leg Right -->
@@ -338,5 +355,4 @@
             <origin xyz="0 0 0" rpy="0 0 ${-pi/2}"/>
             <geometry>
-<!--                <box size="${width} ${width} ${lower_leg_height}"/>-->
                 <mesh filename="package://march_description/urdf/stl-files/LowerLegRight.stl" scale="1.15 1.15 1.15"/>
             </geometry>
@@ -350,4 +366,10 @@
                     izz="${mass / 12.0 * (width*width + width*width)}"/>
         </inertial>
+        <collision>
+            <origin xyz="0 0 ${-lower_leg_height/2}" rpy="0 0 0"/>
+            <geometry>
+                <box size="${width} ${width} ${lower_leg_height}"/>
+            </geometry>
+        </collision>
     </link>
     <!-- Lower Leg Right -->
@@ -356,5 +378,4 @@
             <origin xyz="0 0 0" rpy="0 0 ${-pi/2}"/>
             <geometry>
-<!--                <box size="${width} ${width} ${ankle_plate_height}"/>-->
                 <mesh filename="package://march_description/urdf/stl-files/FootRight.stl" scale="1.15 1.15 1.15"/>
             </geometry>
@@ -368,13 +389,13 @@
                     izz="${mass / 12.0 * (width*width + width*width)}"/>
         </inertial>
+        <collision>
+            <origin xyz="0 0 ${-ankle_plate_height/2}" rpy="0 0 0"/>
+            <geometry>
+                <box size="${width} ${width} ${ankle_plate_height}"/>
+            </geometry>
+        </collision>
     </link>
     <!-- Foot Right -->
     <link name="foot_right">
-<!--        <visual>-->
-<!--            <origin xyz="${-foot_height/2} 0 0" rpy="0 0 0"/>-->
-<!--            <geometry>-->
-<!--                <box size="${foot_height} ${width} ${width}"/>-->
-<!--            </geometry>-->
-<!--        </visual>-->
         <inertial>
             <origin xyz="${-foot_height/2} 0 0" rpy="0 0 0"/>
@@ -387,4 +408,5 @@
         </inertial>
         <collision>
+            <origin xyz="${-foot_height/2} 0 0" rpy="0 0 0"/>
             <geometry>
                 <box size="${foot_height} ${width} ${width}"/>

Commit message: Change colour

File: march_description/urdf/march-iv.xacro (robot description, xacro)
@@ -43,4 +43,7 @@
     <!-- Import all Gazebo-customization elements, including Gazebo colors -->
     <xacro:include filename="$(find march_description)/urdf/march.gazebo"/>
+    <material name="blue">
+        <color rgba="0 0 0.6 1"/>
+    </material>
     <plugin name="gazebo_ros_control" filename="libgazebo_ros_control.so">
         <robotNamespace>/march</robotNamespace>
@@ -73,5 +76,5 @@
     </joint>
     <joint name="left_knee" type="revolute">
-        <parent link="upper_leg_left"/>
+        <parent link= "upper_leg_left"/>
         <child link="lower_leg_left"/>
         <origin xyz="0 0 ${-upper_leg_height}" rpy="0 0 0"/>
@@ -146,4 +149,5 @@
                 <mesh filename="package://march_description/urdf/stl-files/HipBase.stl" scale="1.15 1.15 1.15"/>
             </geometry>
+            <material name="blue"/>
         </visual>
         <inertial>
@@ -169,4 +173,5 @@
                 <mesh filename="package://march_description/urdf/stl-files/HipLeft.stl" scale="1.15 1.15 1.15"/>
             </geometry>
+            <material name="blue"/>
         </visual>
         <inertial>
@@ -208,4 +213,5 @@
                 <mesh filename="package://march_description/urdf/stl-files/UpperLegLeft.stl" scale="1.15 1.15 1.15"/>
             </geometry>
+            <material name="blue"/>
         </visual>
         <inertial>
@@ -231,4 +237,5 @@
                 <mesh filename="package://march_description/urdf/stl-files/LowerLegLeft.stl" scale="1.15 1.15 1.15"/>
             </geometry>
+            <material name="blue"/>
         </visual>
         <inertial>
@@ -254,4 +261,5 @@
                 <mesh filename="package://march_description/urdf/stl-files/FootLeft.stl" scale="1.15 1.15 1.15"/>
             </geometry>
+            <material name="blue"/>
         </visual>
         <inertial>
@@ -295,4 +303,5 @@
                 <mesh filename="package://march_description/urdf/stl-files/HipRight.stl" scale="1.15 1.15 1.15"/>
             </geometry>
+            <material name="blue"/>
         </visual>
         <inertial>
@@ -334,4 +343,5 @@
                 <mesh filename="package://march_description/urdf/stl-files/UpperLegRight.stl" scale="1.15 1.15 1.15"/>
             </geometry>
+            <material name="blue"/>
         </visual>
         <inertial>
@@ -357,4 +367,5 @@
                 <mesh filename="package://march_description/urdf/stl-files/LowerLegRight.stl" scale="1.15 1.15 1.15"/>
             </geometry>
+            <material name="blue"/>
         </visual>
         <inertial>
@@ -380,4 +391,5 @@
                 <mesh filename="package://march_description/urdf/stl-files/FootRight.stl" scale="1.15 1.15 1.15"/>
             </geometry>
+            <material name="blue"/>
         </visual>
         <inertial>

Commit message: Add todo

File: march_description/urdf/march-iv.xacro (robot description, xacro)
@@ -8,6 +8,6 @@
     <xacro:property name="parent_name" value="world"/>
     <!-- Constants for robot dimensions -->
-    <xacro:property name="PI" value="3.1415926535897931"/>
     <xacro:property name="mass" value="1"/> <!-- arbitrary value for mass -->
+    <!-- TODO @Jitske: add accurate masses and inertia for all links -->
     <xacro:property name="width" value="0.05"/> <!-- Square dimensions (widthxwidth) of beams -->
     <xacro:property name="upper_leg_height" value="${0.385}"/>

Commit message: Adjust the origin of the feet

File: march_description/urdf/march-iv.xacro (robot description, xacro)
@@ -15,5 +15,6 @@
     <xacro:property name="lower_leg_height" value="${0.385}"/>
     <xacro:property name="lower_leg_mass" value="1.133"/>
-    <xacro:property name="foot_height" value="${0.184}"/>
+    <xacro:property name="foot_height_forward" value="${0.184}"/>
+    <xacro:property name="foot_height_backward" value="${0.059}"/>
     <xacro:property name="foot_mass" value="0.393"/>
     <xacro:property name="ankle_plate_height" value="0.07"/>
@@ -281,6 +282,5 @@
     <link name="foot_left">
         <inertial>
-            <origin xyz="${-foot_height/2} 0 0" rpy="0 0 0"/>
-            <!--            TODO: adjust the origin so the foot also sticks out a little bit to the back-->
+            <origin xyz="${(-foot_height_forward+foot_height_backward)/2} 0 0" rpy="0 0 0"/>
             <mass value="${foot_mass}"/>
             <inertia
@@ -290,7 +290,7 @@
         </inertial>
         <collision>
-            <origin xyz="${-foot_height/2} 0 0" rpy="0 0 0"/>
-            <geometry>
-                <box size="${foot_height} ${width} ${width}"/>
+            <origin xyz="${(-foot_height_forward+foot_height_backward)/2} 0 0" rpy="0 0 0"/>
+            <geometry>
+                <box size="${foot_height_forward+foot_height_backward} ${width} ${width}"/>
             </geometry>
         </collision>
@@ -411,16 +411,15 @@
     <link name="foot_right">
         <inertial>
-            <origin xyz="${-foot_height/2} 0 0" rpy="0 0 0"/>
-            <!--            TODO: adjust the origin so the foot also sticks out a little bit to the back-->
-            <mass value="${mass}"/>
-            <inertia
-                    ixx="${mass / 12.0 * (width*width + lower_leg_height*lower_leg_height)}" ixy="0.0" ixz="0.0"
-                    iyy="${mass / 12.0 * (lower_leg_height*lower_leg_height + width*width)}" iyz="0.0"
-                    izz="${mass / 12.0 * (width*width + width*width)}"/>
-        </inertial>
-        <collision>
-            <origin xyz="${-foot_height/2} 0 0" rpy="0 0 0"/>
-            <geometry>
-                <box size="${foot_height} ${width} ${width}"/>
+            <origin xyz="${(-foot_height_forward+foot_height_backward)/2} 0 0" rpy="0 0 0"/>
+            <mass value="${mass}"/>
+            <inertia
+                    ixx="${mass / 12.0 * (width*width + lower_leg_height*lower_leg_height)}" ixy="0.0" ixz="0.0"
+                    iyy="${mass / 12.0 * (lower_leg_height*lower_leg_height + width*width)}" iyz="0.0"
+                    izz="${mass / 12.0 * (width*width + width*width)}"/>
+        </inertial>
+        <collision>
+            <origin xyz="${(-foot_height_forward+foot_height_backward)/2} 0 0" rpy="0 0 0"/>
+            <geometry>
+                <box size="${foot_height_forward+foot_height_backward} ${width} ${width}"/>
             </geometry>
         </collision>

Commit message: Change mechanical reduction into the true transmission for HFE/KFE

File: march_description/urdf/march-iv.xacro (robot description, xacro)
@@ -443,66 +443,66 @@
         <actuator name="left_hip_fe_motor">
             <hardwareInterface>hardware_interface/EffortJointInterface</hardwareInterface>
+            <mechanicalReduction>101</mechanicalReduction>
+        </actuator>
+    </transmission>
+    <transmission name="left_knee">
+        <type>transmission_interface/SimpleTransmission</type>
+        <joint name="left_knee">
+            <hardwareInterface>hardware_interface/EffortJointInterface</hardwareInterface>
+        </joint>
+        <actuator name="left_knee_motor">
+            <hardwareInterface>hardware_interface/EffortJointInterface</hardwareInterface>
+            <mechanicalReduction>101</mechanicalReduction>
+        </actuator>
+    </transmission>
+    <transmission name="left_ankle">
+        <type>transmission_interface/SimpleTransmission</type>
+        <joint name="left_ankle">
+            <hardwareInterface>hardware_interface/EffortJointInterface</hardwareInterface>
+        </joint>
+        <actuator name="left_ankle_motor">
+            <hardwareInterface>hardware_interface/EffortJointInterface</hardwareInterface>
             <mechanicalReduction>1</mechanicalReduction>
         </actuator>
     </transmission>
-    <transmission name="left_knee">
-        <type>transmission_interface/SimpleTransmission</type>
-        <joint name="left_knee">
-            <hardwareInterface>hardware_interface/EffortJointInterface</hardwareInterface>
-        </joint>
-        <actuator name="left_knee_motor">
+    <transmission name="right_hip_aa">
+        <type>transmission_interface/SimpleTransmission</type>
+        <joint name="right_hip_aa">
+            <hardwareInterface>hardware_interface/EffortJointInterface</hardwareInterface>
+        </joint>
+        <actuator name="right_hip_aa_motor">
             <hardwareInterface>hardware_interface/EffortJointInterface</hardwareInterface>
             <mechanicalReduction>1</mechanicalReduction>
         </actuator>
     </transmission>
-    <transmission name="left_ankle">
-        <type>transmission_interface/SimpleTransmission</type>
-        <joint name="left_ankle">
-            <hardwareInterface>hardware_interface/EffortJointInterface</hardwareInterface>
-        </joint>
-        <actuator name="left_ankle_motor">
+    <transmission name="right_hip_fe">
+        <type>transmission_interface/SimpleTransmission</type>
+        <joint name="right_hip_fe">
+            <hardwareInterface>hardware_interface/EffortJointInterface</hardwareInterface>
+        </joint>
+        <actuator name="right_hip_fe_motor">
+            <hardwareInterface>hardware_interface/EffortJointInterface</hardwareInterface>
+            <mechanicalReduction>101</mechanicalReduction>
+        </actuator>
+    </transmission>
+    <transmission name="right_knee">
+        <type>transmission_interface/SimpleTransmission</type>
+        <joint name="right_knee">
+            <hardwareInterface>hardware_interface/EffortJointInterface</hardwareInterface>
+        </joint>
+        <actuator name="right_knee_motor">
+            <hardwareInterface>hardware_interface/EffortJointInterface</hardwareInterface>
+            <mechanicalReduction>101</mechanicalReduction>
+        </actuator>
+    </transmission>
+    <transmission name="right_ankle">
+        <type>transmission_interface/SimpleTransmission</type>
+        <joint name="right_ankle">
+            <hardwareInterface>hardware_interface/EffortJointInterface</hardwareInterface>
+        </joint>
+        <actuator name="right_ankle_motor">
             <hardwareInterface>hardware_interface/EffortJointInterface</hardwareInterface>
             <mechanicalReduction>1</mechanicalReduction>
         </actuator>
     </transmission>
-    <transmission name="right_hip_aa">
-        <type>transmission_interface/SimpleTransmission</type>
-        <joint name="right_hip_aa">
-            <hardwareInterface>hardware_interface/EffortJointInterface</hardwareInterface>
-        </joint>
-        <actuator name="right_hip_aa_motor">
-            <hardwareInterface>hardware_interface/EffortJointInterface</hardwareInterface>
-            <mechanicalReduction>1</mechanicalReduction>
-        </actuator>
-    </transmission>
-    <transmission name="right_hip_fe">
-        <type>transmission_interface/SimpleTransmission</type>
-        <joint name="right_hip_fe">
-            <hardwareInterface>hardware_interface/EffortJointInterface</hardwareInterface>
-        </joint>
-        <actuator name="right_hip_fe_motor">
-            <hardwareInterface>hardware_interface/EffortJointInterface</hardwareInterface>
-            <mechanicalReduction>1</mechanicalReduction>
-        </actuator>
-    </transmission>
-    <transmission name="right_knee">
-        <type>transmission_interface/SimpleTransmission</type>
-        <joint name="right_knee">
-            <hardwareInterface>hardware_interface/EffortJointInterface</hardwareInterface>
-        </joint>
-        <actuator name="right_knee_motor">
-            <hardwareInterface>hardware_interface/EffortJointInterface</hardwareInterface>
-            <mechanicalReduction>1</mechanicalReduction>
-        </actuator>
-    </transmission>
-    <transmission name="right_ankle">
-        <type>transmission_interface/SimpleTransmission</type>
-        <joint name="right_ankle">
-            <hardwareInterface>hardware_interface/EffortJointInterface</hardwareInterface>
-        </joint>
-        <actuator name="right_ankle_motor">
-            <hardwareInterface>hardware_interface/EffortJointInterface</hardwareInterface>
-            <mechanicalReduction>1</mechanicalReduction>
-        </actuator>
-    </transmission>
 </robot>
