Commit message: Invert the limits

File: march_description/urdf/march-iv.xacro (robot description, xacro)
@@ -8,6 +8,6 @@
     <xacro:property name="parent_name" value="world"/>
     <!-- Constants for robot dimensions -->
+    <!-- TODO @Jitske: add accurate masses and inertia for all links -->
     <xacro:property name="mass" value="1"/> <!-- arbitrary value for mass -->
-    <!-- TODO @Jitske: add accurate masses and inertia for all links -->
     <xacro:property name="width" value="0.05"/> <!-- Square dimensions (widthxwidth) of beams -->
     <xacro:property name="upper_leg_height" value="${0.385}"/>
@@ -27,6 +27,6 @@
     <xacro:property name="hip_fe_effort_limit" value="10927.0"/> <!-- IU -->
     <xacro:property name="hip_fe_velocity_limit" value="48.0"/> <!-- rad/s -->
-    <xacro:property name="hip_aa_rotation_lower_limit" value="${20*pi/180}"/> <!-- rad -->
-    <xacro:property name="hip_aa_rotation_upper_limit" value="${-30*pi/180}"/> <!-- rad -->
+    <xacro:property name="hip_aa_rotation_lower_limit" value="${-30*pi/180}"/> <!-- rad -->
+    <xacro:property name="hip_aa_rotation_upper_limit" value="${20*pi/180}"/> <!-- rad -->
     <xacro:property name="hip_aa_effort_limit" value="10927.0"/> <!-- IU -->
     <xacro:property name="hip_aa_velocity_limit" value="15.0"/> <!-- rad/s -->

Commit message: Adjustments on the range of motion

File: march_description/urdf/march-iv.xacro (robot description, xacro)
@@ -23,10 +23,10 @@
     <xacro:property name="hip_aa_frame_height" value="0.130"/>
     <xacro:property name="hip_aa_frame_width" value="0.1395"/>
-    <xacro:property name="hip_fe_rotation_lower_limit" value="${-15*pi/180}"/> <!-- rad -->
-    <xacro:property name="hip_fe_rotation_upper_limit" value="${105*pi/180}"/> <!-- rad -->
+    <xacro:property name="hip_fe_rotation_lower_limit" value="${-20*pi/180}"/> <!-- rad -->
+    <xacro:property name="hip_fe_rotation_upper_limit" value="${100*pi/180}"/> <!-- rad -->
     <xacro:property name="hip_fe_effort_limit" value="10927.0"/> <!-- IU -->
     <xacro:property name="hip_fe_velocity_limit" value="48.0"/> <!-- rad/s -->
-    <xacro:property name="hip_aa_rotation_lower_limit" value="${-30*pi/180}"/> <!-- rad -->
-    <xacro:property name="hip_aa_rotation_upper_limit" value="${20*pi/180}"/> <!-- rad -->
+    <xacro:property name="hip_aa_rotation_lower_limit" value="${-20*pi/180}"/> <!-- rad -->
+    <xacro:property name="hip_aa_rotation_upper_limit" value="${15*pi/180}"/> <!-- rad -->
     <xacro:property name="hip_aa_effort_limit" value="10927.0"/> <!-- IU -->
     <xacro:property name="hip_aa_velocity_limit" value="15.0"/> <!-- rad/s -->
@@ -36,5 +36,5 @@
     <xacro:property name="knee_velocity_limit" value="48.0"/>
     <xacro:property name="ankle_rotation_lower_limit" value="${-15*pi/180}"/>
-    <xacro:property name="ankle_rotation_upper_limit" value="${30*pi/180}"/>
+    <xacro:property name="ankle_rotation_upper_limit" value="${25*pi/180}"/>
     <xacro:property name="ankle_effort_limit" value="10927.0"/>
     <xacro:property name="ankle_velocity_limit" value="15.0"/>

Commit message: Align hip_aa on the correct axis

File: march_description/urdf/march-iv.xacro (robot description, xacro)
@@ -61,5 +61,5 @@
         <child link="hip_aa_frame_left_side"/>
         <origin xyz="0 ${-hip_base_height/2} 0" rpy="0 0 0"/>
-        <axis xyz="1 0 0"/>
+        <axis xyz="-1 0 0"/>
         <limit velocity="${hip_aa_velocity_limit}" effort="${hip_aa_effort_limit}" lower="${hip_aa_rotation_lower_limit}" upper="${hip_aa_rotation_upper_limit}"/>
     </joint>
@@ -100,5 +100,5 @@
         <origin xyz="0 ${hip_base_height/2} 0" rpy="0 0 0"/>
         <axis xyz="1 0 0"/>
-        <limit velocity="${hip_aa_velocity_limit}" effort="${hip_aa_effort_limit}" lower="${-hip_aa_rotation_lower_limit}" upper="${-hip_aa_rotation_upper_limit}"/>
+        <limit velocity="${hip_aa_velocity_limit}" effort="${hip_aa_effort_limit}" lower="${hip_aa_rotation_lower_limit}" upper="${hip_aa_rotation_upper_limit}"/>
     </joint>
     <joint name="right_hip_angle" type="fixed">

Commit message: Update march-iv.xacro

File: march_description/urdf/march-iv.xacro (robot description, xacro)
@@ -27,20 +27,20 @@
     <xacro:property name="hip_fe_soft_buffer" value="${5*pi/180}"/> <!-- rad -->
     <xacro:property name="hip_fe_effort_limit" value="10927.0"/> <!-- IU -->
-    <xacro:property name="hip_fe_velocity_limit" value="4.80"/> <!-- rad/s -->
+    <xacro:property name="hip_fe_velocity_limit" value="1.0"/> <!-- rad/s -->
     <xacro:property name="hip_aa_rotation_lower_limit" value="${-20*pi/180}"/> <!-- rad -->
     <xacro:property name="hip_aa_rotation_upper_limit" value="${15*pi/180}"/> <!-- rad -->
     <xacro:property name="hip_aa_soft_buffer" value="${5*pi/180}"/> <!-- rad -->
     <xacro:property name="hip_aa_effort_limit" value="10927.0"/> <!-- IU -->
-    <xacro:property name="hip_aa_velocity_limit" value="1.50"/> <!-- rad/s -->
+    <xacro:property name="hip_aa_velocity_limit" value="1.0"/> <!-- rad/s -->
     <xacro:property name="knee_rotation_lower_limit" value="${-5*pi/180}"/>
     <xacro:property name="knee_rotation_upper_limit" value="${115*pi/180}"/>
     <xacro:property name="knee_soft_buffer" value="${5*pi/180}"/> <!-- rad -->
     <xacro:property name="knee_effort_limit" value="10927.0"/>
-    <xacro:property name="knee_velocity_limit" value="4.8"/>
+    <xacro:property name="knee_velocity_limit" value="1.0"/>
     <xacro:property name="ankle_rotation_lower_limit" value="${-15*pi/180}"/>
     <xacro:property name="ankle_rotation_upper_limit" value="${25*pi/180}"/>
     <xacro:property name="ankle_soft_buffer" value="${5*pi/180}"/> <!-- rad -->
     <xacro:property name="ankle_effort_limit" value="10927.0"/>
-    <xacro:property name="ankle_velocity_limit" value="1.5"/>
+    <xacro:property name="ankle_velocity_limit" value="1.0"/>
     <xacro:property name="hover_height" value="0.3"/>
     <xacro:property name="camera_link" value="0.05"/> <!-- Size of square 'camera' box -->

Commit message: Change knee soft buffer from 5 to 4 degrees

File: march_description/urdf/march-iv.xacro (robot description, xacro)
@@ -35,5 +35,5 @@
     <xacro:property name="knee_rotation_lower_limit" value="${-5*pi/180}"/>
     <xacro:property name="knee_rotation_upper_limit" value="${115*pi/180}"/>
-    <xacro:property name="knee_soft_buffer" value="${5*pi/180}"/> <!-- rad -->
+    <xacro:property name="knee_soft_buffer" value="${4*pi/180}"/> <!-- rad -->
     <xacro:property name="knee_effort_limit" value="10927.0"/>
     <xacro:property name="knee_velocity_limit" value="1.0"/>

Commit message: Update march_description/urdf/march-iv.xacro

File: march_description/urdf/march-iv.xacro (robot description, xacro)
@@ -35,5 +35,5 @@
     <xacro:property name="knee_rotation_lower_limit" value="${-5*pi/180}"/>
     <xacro:property name="knee_rotation_upper_limit" value="${115*pi/180}"/>
-    <xacro:property name="knee_soft_buffer" value="${4*pi/180}"/> <!-- rad -->
+    <xacro:property name="knee_soft_buffer" value="${4.5*pi/180}"/> <!-- rad -->
     <xacro:property name="knee_effort_limit" value="10927.0"/>
     <xacro:property name="knee_velocity_limit" value="1.0"/>

Commit message: Adjusted the soft buffers

File: march_description/urdf/march-iv.xacro (robot description, xacro)
@@ -25,5 +25,5 @@
     <xacro:property name="hip_fe_rotation_lower_limit" value="${-20*pi/180}"/> <!-- rad -->
     <xacro:property name="hip_fe_rotation_upper_limit" value="${100*pi/180}"/> <!-- rad -->
-    <xacro:property name="hip_fe_soft_buffer" value="${5*pi/180}"/> <!-- rad -->
+    <xacro:property name="hip_fe_soft_buffer" value="${3*pi/180}"/> <!-- rad -->
     <xacro:property name="hip_fe_effort_limit" value="10927.0"/> <!-- IU -->
     <xacro:property name="hip_fe_velocity_limit" value="1.0"/> <!-- rad/s -->
@@ -35,10 +35,12 @@
     <xacro:property name="knee_rotation_lower_limit" value="${-5*pi/180}"/>
     <xacro:property name="knee_rotation_upper_limit" value="${115*pi/180}"/>
-    <xacro:property name="knee_soft_buffer" value="${4.5*pi/180}"/> <!-- rad -->
+    <xacro:property name="knee_extension_soft_buffer" value="${4.5*pi/180}"/> <!-- rad -->
+    <xacro:property name="knee_flexion_soft_buffer" value="${3*pi/180}"/> <!-- rad -->
     <xacro:property name="knee_effort_limit" value="10927.0"/>
     <xacro:property name="knee_velocity_limit" value="1.0"/>
     <xacro:property name="ankle_rotation_lower_limit" value="${-15*pi/180}"/>
     <xacro:property name="ankle_rotation_upper_limit" value="${25*pi/180}"/>
-    <xacro:property name="ankle_soft_buffer" value="${5*pi/180}"/> <!-- rad -->
+    <xacro:property name="ankle_dorsalflexion_soft_buffer" value="${5*pi/180}"/> <!-- rad -->
+    <xacro:property name="ankle_plantarflexion_soft_buffer" value="${3*pi/180}"/> <!-- rad -->
     <xacro:property name="ankle_effort_limit" value="10927.0"/>
     <xacro:property name="ankle_velocity_limit" value="1.0"/>
@@ -88,5 +90,5 @@
         <axis xyz="0 -1 0"/>
         <limit velocity="${knee_velocity_limit}" effort="${knee_effort_limit}" lower="${knee_rotation_lower_limit}" upper="${knee_rotation_upper_limit}"/>
-        <safety_controller soft_lower_limit="${knee_rotation_lower_limit + knee_soft_buffer}" soft_upper_limit="${knee_rotation_upper_limit - knee_soft_buffer}" k_position="5" k_velocity="5" />
+        <safety_controller soft_lower_limit="${knee_rotation_lower_limit + knee_extension_soft_buffer}" soft_upper_limit="${knee_rotation_upper_limit - knee_flexion_soft_buffer}" k_position="5" k_velocity="5" />
     </joint>
     <joint name="left_ankle" type="revolute">
@@ -96,5 +98,5 @@
         <axis xyz="0 1 0"/>
         <limit velocity="${ankle_velocity_limit}" effort="${ankle_effort_limit}" lower="${ankle_rotation_lower_limit}" upper="${ankle_rotation_upper_limit}"/>
-        <safety_controller soft_lower_limit="${ankle_rotation_lower_limit + ankle_soft_buffer}" soft_upper_limit="${ankle_rotation_upper_limit - ankle_soft_buffer}" k_position="5" k_velocity="5" />
+        <safety_controller soft_lower_limit="${ankle_rotation_lower_limit + ankle_dorsalflexion_soft_buffer}" soft_upper_limit="${ankle_rotation_upper_limit - ankle_plantarflexion_soft_buffer}" k_position="5" k_velocity="5" />
     </joint>
     <joint name="left_foot_angle" type="fixed">
@@ -130,5 +132,5 @@
         <axis xyz="0 -1 0"/>
         <limit velocity="${knee_velocity_limit}" effort="${knee_effort_limit}" lower="${knee_rotation_lower_limit}" upper="${knee_rotation_upper_limit}"/>
-        <safety_controller soft_lower_limit="${knee_rotation_lower_limit + knee_soft_buffer}" soft_upper_limit="${knee_rotation_upper_limit - knee_soft_buffer}" k_position="5" k_velocity="5" />
+        <safety_controller soft_lower_limit="${knee_rotation_lower_limit + knee_extension_soft_buffer}" soft_upper_limit="${knee_rotation_upper_limit - knee_flexion_soft_buffer}" k_position="5" k_velocity="5" />
     </joint>
     <joint name="right_ankle" type="revolute">
@@ -138,5 +140,5 @@
         <axis xyz="0 1 0"/>
         <limit velocity="${ankle_velocity_limit}" effort="${ankle_effort_limit}" lower="${ankle_rotation_lower_limit}" upper="${ankle_rotation_upper_limit}"/>
-        <safety_controller soft_lower_limit="${ankle_rotation_lower_limit + ankle_soft_buffer}" soft_upper_limit="${ankle_rotation_upper_limit - ankle_soft_buffer}" k_position="5" k_velocity="5" />
+        <safety_controller soft_lower_limit="${ankle_rotation_lower_limit + ankle_dorsalflexion_soft_buffer}" soft_upper_limit="${ankle_rotation_upper_limit - ankle_plantarflexion_soft_buffer}" k_position="5" k_velocity="5" />
     </joint>
     <joint name="right_foot_angle" type="fixed">

Commit message: Update march-iv.xacro

File: march_description/urdf/march-iv.xacro (robot description, xacro)
@@ -27,7 +27,7 @@
     <xacro:property name="hip_fe_soft_buffer" value="${3*pi/180}"/> <!-- rad -->
     <xacro:property name="hip_fe_effort_limit" value="10927.0"/> <!-- IU -->
-    <xacro:property name="hip_fe_velocity_limit" value="1.0"/> <!-- rad/s -->
-    <xacro:property name="hip_aa_rotation_lower_limit" value="${-20*pi/180}"/> <!-- rad -->
-    <xacro:property name="hip_aa_rotation_upper_limit" value="${15*pi/180}"/> <!-- rad -->
+    <xacro:property name="hip_fe_velocity_limit" value="1.7"/> <!-- rad/s -->
+    <xacro:property name="hip_aa_rotation_lower_limit" value="${-18*pi/180}"/> <!-- rad -->
+    <xacro:property name="hip_aa_rotation_upper_limit" value="${17*pi/180}"/> <!-- rad -->
     <xacro:property name="hip_aa_soft_buffer" value="${5*pi/180}"/> <!-- rad -->
     <xacro:property name="hip_aa_effort_limit" value="10927.0"/> <!-- IU -->
@@ -38,7 +38,7 @@
     <xacro:property name="knee_flexion_soft_buffer" value="${3*pi/180}"/> <!-- rad -->
     <xacro:property name="knee_effort_limit" value="10927.0"/>
-    <xacro:property name="knee_velocity_limit" value="1.0"/>
-    <xacro:property name="ankle_rotation_lower_limit" value="${-15*pi/180}"/>
-    <xacro:property name="ankle_rotation_upper_limit" value="${25*pi/180}"/>
+    <xacro:property name="knee_velocity_limit" value="1.7"/>
+    <xacro:property name="ankle_rotation_lower_limit" value="${-25*pi/180}"/>
+    <xacro:property name="ankle_rotation_upper_limit" value="${15*pi/180}"/>
     <xacro:property name="ankle_dorsalflexion_soft_buffer" value="${5*pi/180}"/> <!-- rad -->
     <xacro:property name="ankle_plantarflexion_soft_buffer" value="${3*pi/180}"/> <!-- rad -->
@@ -99,5 +99,5 @@
         <axis xyz="0 1 0"/>
         <limit velocity="${ankle_velocity_limit}" effort="${ankle_effort_limit}" lower="${ankle_rotation_lower_limit}" upper="${ankle_rotation_upper_limit}"/>
-        <safety_controller soft_lower_limit="${ankle_rotation_lower_limit + ankle_dorsalflexion_soft_buffer}" soft_upper_limit="${ankle_rotation_upper_limit - ankle_plantarflexion_soft_buffer}" k_position="5" k_velocity="5" />
+        <safety_controller soft_lower_limit="${ankle_rotation_lower_limit + ankle_plantarflexion_soft_buffer}" soft_upper_limit="${ankle_rotation_upper_limit - ankle_dorsalflexion_soft_buffer}" k_position="5" k_velocity="5" />
     </joint>
     <joint name="left_foot_angle" type="fixed">
@@ -141,5 +141,5 @@
         <axis xyz="0 1 0"/>
         <limit velocity="${ankle_velocity_limit}" effort="${ankle_effort_limit}" lower="${ankle_rotation_lower_limit}" upper="${ankle_rotation_upper_limit}"/>
-        <safety_controller soft_lower_limit="${ankle_rotation_lower_limit + ankle_dorsalflexion_soft_buffer}" soft_upper_limit="${ankle_rotation_upper_limit - ankle_plantarflexion_soft_buffer}" k_position="5" k_velocity="5" />
+        <safety_controller soft_lower_limit="${ankle_rotation_lower_limit + ankle_plantarflexion_soft_buffer}" soft_upper_limit="${ankle_rotation_upper_limit - ankle_dorsalflexion_soft_buffer}" k_position="5" k_velocity="5" />
     </joint>
     <joint name="right_foot_angle" type="fixed">

Commit message: Adjust k_velocity and effort limits to work with torque mode

File: march_description/urdf/march-iv.xacro (robot description, xacro)
@@ -26,10 +26,10 @@
     <xacro:property name="hip_fe_rotation_upper_limit" value="${100*pi/180}"/> <!-- rad -->
     <xacro:property name="hip_fe_soft_buffer" value="${3*pi/180}"/> <!-- rad -->
-    <xacro:property name="hip_fe_effort_limit" value="10927.0"/> <!-- IU -->
+    <xacro:property name="hip_fe_effort_limit" value="8000.0"/> <!-- IU -->
     <xacro:property name="hip_fe_velocity_limit" value="1.7"/> <!-- rad/s -->
     <xacro:property name="hip_aa_rotation_lower_limit" value="${-18*pi/180}"/> <!-- rad -->
     <xacro:property name="hip_aa_rotation_upper_limit" value="${17*pi/180}"/> <!-- rad -->
     <xacro:property name="hip_aa_soft_buffer" value="${5*pi/180}"/> <!-- rad -->
-    <xacro:property name="hip_aa_effort_limit" value="10927.0"/> <!-- IU -->
+    <xacro:property name="hip_aa_effort_limit" value="8000.0"/> <!-- IU -->
     <xacro:property name="hip_aa_velocity_limit" value="1.0"/> <!-- rad/s -->
     <xacro:property name="knee_rotation_lower_limit" value="${-5*pi/180}"/>
@@ -37,5 +37,5 @@
     <xacro:property name="knee_extension_soft_buffer" value="${4.5*pi/180}"/> <!-- rad -->
     <xacro:property name="knee_flexion_soft_buffer" value="${3*pi/180}"/> <!-- rad -->
-    <xacro:property name="knee_effort_limit" value="10927.0"/>
+    <xacro:property name="knee_effort_limit" value="8000.0"/>
     <xacro:property name="knee_velocity_limit" value="1.7"/>
     <xacro:property name="ankle_rotation_lower_limit" value="${-25*pi/180}"/>
@@ -43,5 +43,5 @@
     <xacro:property name="ankle_dorsalflexion_soft_buffer" value="${5*pi/180}"/> <!-- rad -->
     <xacro:property name="ankle_plantarflexion_soft_buffer" value="${3*pi/180}"/> <!-- rad -->
-    <xacro:property name="ankle_effort_limit" value="10927.0"/>
+    <xacro:property name="ankle_effort_limit" value="8000.0"/>
     <xacro:property name="ankle_velocity_limit" value="1.0"/>
     <xacro:property name="hover_height" value="0.3"/>
@@ -70,5 +70,5 @@
 <!-- TODO: @JitskedeVries  Improve k values-->
         <limit velocity="${hip_aa_velocity_limit}" effort="${hip_aa_effort_limit}" lower="${hip_aa_rotation_lower_limit}" upper="${hip_aa_rotation_upper_limit}"/>
-        <safety_controller soft_lower_limit="${hip_aa_rotation_lower_limit + hip_aa_soft_buffer}" soft_upper_limit="${hip_aa_rotation_upper_limit - hip_aa_soft_buffer}" k_position="5" k_velocity="5" />
+        <safety_controller soft_lower_limit="${hip_aa_rotation_lower_limit + hip_aa_soft_buffer}" soft_upper_limit="${hip_aa_rotation_upper_limit - hip_aa_soft_buffer}" k_position="5" k_velocity="20000" />
     </joint>
     <joint name="left_hip_angle" type="fixed">
@@ -83,5 +83,5 @@
         <axis xyz="0 1 0"/>
         <limit velocity="${hip_fe_velocity_limit}" effort="${hip_fe_effort_limit}" lower="${hip_fe_rotation_lower_limit}" upper="${hip_fe_rotation_upper_limit}"/>
-        <safety_controller soft_lower_limit="${hip_fe_rotation_lower_limit + hip_fe_soft_buffer}" soft_upper_limit="${hip_fe_rotation_upper_limit - hip_fe_soft_buffer}" k_position="5" k_velocity="5" />
+        <safety_controller soft_lower_limit="${hip_fe_rotation_lower_limit + hip_fe_soft_buffer}" soft_upper_limit="${hip_fe_rotation_upper_limit - hip_fe_soft_buffer}" k_position="5" k_velocity="20000" />
     </joint>
     <joint name="left_knee" type="revolute">
@@ -91,5 +91,5 @@
         <axis xyz="0 -1 0"/>
         <limit velocity="${knee_velocity_limit}" effort="${knee_effort_limit}" lower="${knee_rotation_lower_limit}" upper="${knee_rotation_upper_limit}"/>
-        <safety_controller soft_lower_limit="${knee_rotation_lower_limit + knee_extension_soft_buffer}" soft_upper_limit="${knee_rotation_upper_limit - knee_flexion_soft_buffer}" k_position="5" k_velocity="5" />
+        <safety_controller soft_lower_limit="${knee_rotation_lower_limit + knee_extension_soft_buffer}" soft_upper_limit="${knee_rotation_upper_limit - knee_flexion_soft_buffer}" k_position="5" k_velocity="20000" />
     </joint>
     <joint name="left_ankle" type="revolute">
@@ -99,5 +99,5 @@
         <axis xyz="0 1 0"/>
         <limit velocity="${ankle_velocity_limit}" effort="${ankle_effort_limit}" lower="${ankle_rotation_lower_limit}" upper="${ankle_rotation_upper_limit}"/>
-        <safety_controller soft_lower_limit="${ankle_rotation_lower_limit + ankle_plantarflexion_soft_buffer}" soft_upper_limit="${ankle_rotation_upper_limit - ankle_dorsalflexion_soft_buffer}" k_position="5" k_velocity="5" />
+        <safety_controller soft_lower_limit="${ankle_rotation_lower_limit + ankle_plantarflexion_soft_buffer}" soft_upper_limit="${ankle_rotation_upper_limit - ankle_dorsalflexion_soft_buffer}" k_position="5" k_velocity="20000" />
     </joint>
     <joint name="left_foot_angle" type="fixed">
@@ -112,5 +112,5 @@
         <axis xyz="1 0 0"/>
         <limit velocity="${hip_aa_velocity_limit}" effort="${hip_aa_effort_limit}" lower="${hip_aa_rotation_lower_limit}" upper="${hip_aa_rotation_upper_limit}"/>
-        <safety_controller soft_lower_limit="${hip_aa_rotation_lower_limit + hip_aa_soft_buffer}" soft_upper_limit="${hip_aa_rotation_upper_limit - hip_aa_soft_buffer}" k_position="5" k_velocity="5" />
+        <safety_controller soft_lower_limit="${hip_aa_rotation_lower_limit + hip_aa_soft_buffer}" soft_upper_limit="${hip_aa_rotation_upper_limit - hip_aa_soft_buffer}" k_position="5" k_velocity="20000" />
     </joint>
     <joint name="right_hip_angle" type="fixed">
@@ -125,5 +125,5 @@
         <axis xyz="0 1 0"/>
         <limit velocity="${hip_fe_velocity_limit}" effort="${hip_fe_effort_limit}" lower="${hip_fe_rotation_lower_limit}" upper="${hip_fe_rotation_upper_limit}"/>
-        <safety_controller soft_lower_limit="${hip_fe_rotation_lower_limit + hip_fe_soft_buffer}" soft_upper_limit="${hip_fe_rotation_upper_limit - hip_fe_soft_buffer}" k_position="5" k_velocity="5" />
+        <safety_controller soft_lower_limit="${hip_fe_rotation_lower_limit + hip_fe_soft_buffer}" soft_upper_limit="${hip_fe_rotation_upper_limit - hip_fe_soft_buffer}" k_position="5" k_velocity="20000" />
     </joint>
     <joint name="right_knee" type="revolute">
@@ -133,5 +133,5 @@
         <axis xyz="0 -1 0"/>
         <limit velocity="${knee_velocity_limit}" effort="${knee_effort_limit}" lower="${knee_rotation_lower_limit}" upper="${knee_rotation_upper_limit}"/>
-        <safety_controller soft_lower_limit="${knee_rotation_lower_limit + knee_extension_soft_buffer}" soft_upper_limit="${knee_rotation_upper_limit - knee_flexion_soft_buffer}" k_position="5" k_velocity="5" />
+        <safety_controller soft_lower_limit="${knee_rotation_lower_limit + knee_extension_soft_buffer}" soft_upper_limit="${knee_rotation_upper_limit - knee_flexion_soft_buffer}" k_position="5" k_velocity="20000" />
     </joint>
     <joint name="right_ankle" type="revolute">
@@ -141,5 +141,5 @@
         <axis xyz="0 1 0"/>
         <limit velocity="${ankle_velocity_limit}" effort="${ankle_effort_limit}" lower="${ankle_rotation_lower_limit}" upper="${ankle_rotation_upper_limit}"/>
-        <safety_controller soft_lower_limit="${ankle_rotation_lower_limit + ankle_plantarflexion_soft_buffer}" soft_upper_limit="${ankle_rotation_upper_limit - ankle_dorsalflexion_soft_buffer}" k_position="5" k_velocity="5" />
+        <safety_controller soft_lower_limit="${ankle_rotation_lower_limit + ankle_plantarflexion_soft_buffer}" soft_upper_limit="${ankle_rotation_upper_limit - ankle_dorsalflexion_soft_buffer}" k_position="5" k_velocity="20000" />
     </joint>
     <joint name="right_foot_angle" type="fixed">
