Commit message: Adjust effort limits

File: march_description/urdf/march-iv.xacro (robot description, xacro)
@@ -26,10 +26,10 @@
     <xacro:property name="hip_fe_rotation_upper_limit" value="${100*pi/180}"/> <!-- rad -->
     <xacro:property name="hip_fe_soft_buffer" value="${3*pi/180}"/> <!-- rad -->
-    <xacro:property name="hip_fe_effort_limit" value="8000.0"/> <!-- IU -->
-    <xacro:property name="hip_fe_velocity_limit" value="1.7"/> <!-- rad/s -->
+    <xacro:property name="hip_fe_effort_limit" value="21840"/> <!-- IU = 20 A -->
+    <xacro:property name="hip_fe_velocity_limit" value="2.0"/> <!-- rad/s -->
     <xacro:property name="hip_aa_rotation_lower_limit" value="${-18*pi/180}"/> <!-- rad -->
     <xacro:property name="hip_aa_rotation_upper_limit" value="${17*pi/180}"/> <!-- rad -->
     <xacro:property name="hip_aa_soft_buffer" value="${5*pi/180}"/> <!-- rad -->
-    <xacro:property name="hip_aa_effort_limit" value="8000.0"/> <!-- IU -->
+    <xacro:property name="hip_aa_effort_limit" value="21840"/> <!-- IU = 20 A -->
     <xacro:property name="hip_aa_velocity_limit" value="1.0"/> <!-- rad/s -->
     <xacro:property name="knee_rotation_lower_limit" value="${-5*pi/180}"/>
@@ -37,11 +37,11 @@
     <xacro:property name="knee_extension_soft_buffer" value="${4.5*pi/180}"/> <!-- rad -->
     <xacro:property name="knee_flexion_soft_buffer" value="${3*pi/180}"/> <!-- rad -->
-    <xacro:property name="knee_effort_limit" value="8000.0"/>
-    <xacro:property name="knee_velocity_limit" value="1.7"/>
+    <xacro:property name="knee_effort_limit" value="21840"/> <!-- IU = 20 A -->
+    <xacro:property name="knee_velocity_limit" value="2.0"/>
     <xacro:property name="ankle_rotation_lower_limit" value="${-25*pi/180}"/>
     <xacro:property name="ankle_rotation_upper_limit" value="${15*pi/180}"/>
     <xacro:property name="ankle_dorsalflexion_soft_buffer" value="${5*pi/180}"/> <!-- rad -->
     <xacro:property name="ankle_plantarflexion_soft_buffer" value="${3*pi/180}"/> <!-- rad -->
-    <xacro:property name="ankle_effort_limit" value="8000.0"/>
+    <xacro:property name="ankle_effort_limit" value="21840"/> <!-- IU = 20 A -->
     <xacro:property name="ankle_velocity_limit" value="1.0"/>
     <xacro:property name="hover_height" value="0.3"/>

Commit message: add k_velocity_value parameter to xacro which can be changed by launch file

File: march_description/urdf/march-iv.xacro (robot description, xacro)
@@ -48,4 +48,6 @@
     <xacro:property name="camera_link" value="0.05"/> <!-- Size of square 'camera' box -->
     <xacro:property name="axel_offset" value="0.05"/> <!-- Space btw top of beam and the each joint -->
+    <xacro:arg name="k_velocity_value" default="20000.0" />
+    <xacro:property name="k_velocity_value" value="$(arg k_velocity_value)" />
     <!-- Import all Gazebo-customization elements, including Gazebo colors -->
     <xacro:include filename="$(find march_description)/urdf/march.gazebo"/>
@@ -70,5 +72,5 @@
 <!-- TODO: @JitskedeVries  Improve k values-->
         <limit velocity="${hip_aa_velocity_limit}" effort="${hip_aa_effort_limit}" lower="${hip_aa_rotation_lower_limit}" upper="${hip_aa_rotation_upper_limit}"/>
-        <safety_controller soft_lower_limit="${hip_aa_rotation_lower_limit + hip_aa_soft_buffer}" soft_upper_limit="${hip_aa_rotation_upper_limit - hip_aa_soft_buffer}" k_position="5" k_velocity="20000" />
+        <safety_controller soft_lower_limit="${hip_aa_rotation_lower_limit + hip_aa_soft_buffer}" soft_upper_limit="${hip_aa_rotation_upper_limit - hip_aa_soft_buffer}" k_position="5" k_velocity="${k_velocity_value}" />
     </joint>
     <joint name="left_hip_angle" type="fixed">
@@ -83,5 +85,5 @@
         <axis xyz="0 1 0"/>
         <limit velocity="${hip_fe_velocity_limit}" effort="${hip_fe_effort_limit}" lower="${hip_fe_rotation_lower_limit}" upper="${hip_fe_rotation_upper_limit}"/>
-        <safety_controller soft_lower_limit="${hip_fe_rotation_lower_limit + hip_fe_soft_buffer}" soft_upper_limit="${hip_fe_rotation_upper_limit - hip_fe_soft_buffer}" k_position="5" k_velocity="20000" />
+        <safety_controller soft_lower_limit="${hip_fe_rotation_lower_limit + hip_fe_soft_buffer}" soft_upper_limit="${hip_fe_rotation_upper_limit - hip_fe_soft_buffer}" k_position="5" k_velocity="${k_velocity_value}" />
     </joint>
     <joint name="left_knee" type="revolute">
@@ -91,5 +93,5 @@
         <axis xyz="0 -1 0"/>
         <limit velocity="${knee_velocity_limit}" effort="${knee_effort_limit}" lower="${knee_rotation_lower_limit}" upper="${knee_rotation_upper_limit}"/>
-        <safety_controller soft_lower_limit="${knee_rotation_lower_limit + knee_extension_soft_buffer}" soft_upper_limit="${knee_rotation_upper_limit - knee_flexion_soft_buffer}" k_position="5" k_velocity="20000" />
+        <safety_controller soft_lower_limit="${knee_rotation_lower_limit + knee_extension_soft_buffer}" soft_upper_limit="${knee_rotation_upper_limit - knee_flexion_soft_buffer}" k_position="5" k_velocity="${k_velocity_value}" />
     </joint>
     <joint name="left_ankle" type="revolute">
@@ -99,5 +101,5 @@
         <axis xyz="0 1 0"/>
         <limit velocity="${ankle_velocity_limit}" effort="${ankle_effort_limit}" lower="${ankle_rotation_lower_limit}" upper="${ankle_rotation_upper_limit}"/>
-        <safety_controller soft_lower_limit="${ankle_rotation_lower_limit + ankle_plantarflexion_soft_buffer}" soft_upper_limit="${ankle_rotation_upper_limit - ankle_dorsalflexion_soft_buffer}" k_position="5" k_velocity="20000" />
+        <safety_controller soft_lower_limit="${ankle_rotation_lower_limit + ankle_plantarflexion_soft_buffer}" soft_upper_limit="${ankle_rotation_upper_limit - ankle_dorsalflexion_soft_buffer}" k_position="5" k_velocity="${k_velocity_value}" />
     </joint>
     <joint name="left_foot_angle" type="fixed">
@@ -112,5 +114,5 @@
         <axis xyz="1 0 0"/>
         <limit velocity="${hip_aa_velocity_limit}" effort="${hip_aa_effort_limit}" lower="${hip_aa_rotation_lower_limit}" upper="${hip_aa_rotation_upper_limit}"/>
-        <safety_controller soft_lower_limit="${hip_aa_rotation_lower_limit + hip_aa_soft_buffer}" soft_upper_limit="${hip_aa_rotation_upper_limit - hip_aa_soft_buffer}" k_position="5" k_velocity="20000" />
+        <safety_controller soft_lower_limit="${hip_aa_rotation_lower_limit + hip_aa_soft_buffer}" soft_upper_limit="${hip_aa_rotation_upper_limit - hip_aa_soft_buffer}" k_position="5" k_velocity="${k_velocity_value}" />
     </joint>
     <joint name="right_hip_angle" type="fixed">
@@ -125,5 +127,5 @@
         <axis xyz="0 1 0"/>
         <limit velocity="${hip_fe_velocity_limit}" effort="${hip_fe_effort_limit}" lower="${hip_fe_rotation_lower_limit}" upper="${hip_fe_rotation_upper_limit}"/>
-        <safety_controller soft_lower_limit="${hip_fe_rotation_lower_limit + hip_fe_soft_buffer}" soft_upper_limit="${hip_fe_rotation_upper_limit - hip_fe_soft_buffer}" k_position="5" k_velocity="20000" />
+        <safety_controller soft_lower_limit="${hip_fe_rotation_lower_limit + hip_fe_soft_buffer}" soft_upper_limit="${hip_fe_rotation_upper_limit - hip_fe_soft_buffer}" k_position="5" k_velocity="${k_velocity_value}" />
     </joint>
     <joint name="right_knee" type="revolute">
@@ -133,5 +135,5 @@
         <axis xyz="0 -1 0"/>
         <limit velocity="${knee_velocity_limit}" effort="${knee_effort_limit}" lower="${knee_rotation_lower_limit}" upper="${knee_rotation_upper_limit}"/>
-        <safety_controller soft_lower_limit="${knee_rotation_lower_limit + knee_extension_soft_buffer}" soft_upper_limit="${knee_rotation_upper_limit - knee_flexion_soft_buffer}" k_position="5" k_velocity="20000" />
+        <safety_controller soft_lower_limit="${knee_rotation_lower_limit + knee_extension_soft_buffer}" soft_upper_limit="${knee_rotation_upper_limit - knee_flexion_soft_buffer}" k_position="5" k_velocity="${k_velocity_value}" />
     </joint>
     <joint name="right_ankle" type="revolute">
@@ -141,5 +143,5 @@
         <axis xyz="0 1 0"/>
         <limit velocity="${ankle_velocity_limit}" effort="${ankle_effort_limit}" lower="${ankle_rotation_lower_limit}" upper="${ankle_rotation_upper_limit}"/>
-        <safety_controller soft_lower_limit="${ankle_rotation_lower_limit + ankle_plantarflexion_soft_buffer}" soft_upper_limit="${ankle_rotation_upper_limit - ankle_dorsalflexion_soft_buffer}" k_position="5" k_velocity="20000" />
+        <safety_controller soft_lower_limit="${ankle_rotation_lower_limit + ankle_plantarflexion_soft_buffer}" soft_upper_limit="${ankle_rotation_upper_limit - ankle_dorsalflexion_soft_buffer}" k_position="5" k_velocity="${k_velocity_value}" />
     </joint>
     <joint name="right_foot_angle" type="fixed">

Commit message: add max_effort_value argument to xacro

File: march_description/urdf/march-iv.xacro (robot description, xacro)
@@ -7,4 +7,8 @@
     <!--Important note: when changing value make sure rviz fixed frame is set to the same value (moveit.rviz)-->
     <xacro:property name="parent_name" value="world"/>
+    <xacro:arg name="max_effort_value" default="21840.0" />
+    <xacro:property name="max_effort_value" value="$(arg max_effort_value)" />
+    <xacro:arg name="k_velocity_value" default="20000.0" />
+    <xacro:property name="k_velocity_value" value="$(arg k_velocity_value)" />
     <!-- Constants for robot dimensions -->
     <!-- TODO @Jitske: add accurate masses and inertia for all links -->
@@ -26,10 +30,10 @@
     <xacro:property name="hip_fe_rotation_upper_limit" value="${100*pi/180}"/> <!-- rad -->
     <xacro:property name="hip_fe_soft_buffer" value="${3*pi/180}"/> <!-- rad -->
-    <xacro:property name="hip_fe_effort_limit" value="21840"/> <!-- IU = 20 A -->
+    <xacro:property name="hip_fe_effort_limit" value="${max_effort_value}"/> <!-- IU = 20 A -->
     <xacro:property name="hip_fe_velocity_limit" value="2.0"/> <!-- rad/s -->
     <xacro:property name="hip_aa_rotation_lower_limit" value="${-18*pi/180}"/> <!-- rad -->
     <xacro:property name="hip_aa_rotation_upper_limit" value="${17*pi/180}"/> <!-- rad -->
     <xacro:property name="hip_aa_soft_buffer" value="${5*pi/180}"/> <!-- rad -->
-    <xacro:property name="hip_aa_effort_limit" value="21840"/> <!-- IU = 20 A -->
+    <xacro:property name="hip_aa_effort_limit" value="${max_effort_value}"/> <!-- IU = 20 A -->
     <xacro:property name="hip_aa_velocity_limit" value="1.0"/> <!-- rad/s -->
     <xacro:property name="knee_rotation_lower_limit" value="${-5*pi/180}"/>
@@ -37,5 +41,5 @@
     <xacro:property name="knee_extension_soft_buffer" value="${4.5*pi/180}"/> <!-- rad -->
     <xacro:property name="knee_flexion_soft_buffer" value="${3*pi/180}"/> <!-- rad -->
-    <xacro:property name="knee_effort_limit" value="21840"/> <!-- IU = 20 A -->
+    <xacro:property name="knee_effort_limit" value="${max_effort_value}"/> <!-- IU = 20 A -->
     <xacro:property name="knee_velocity_limit" value="2.0"/>
     <xacro:property name="ankle_rotation_lower_limit" value="${-25*pi/180}"/>
@@ -43,11 +47,9 @@
     <xacro:property name="ankle_dorsalflexion_soft_buffer" value="${5*pi/180}"/> <!-- rad -->
     <xacro:property name="ankle_plantarflexion_soft_buffer" value="${3*pi/180}"/> <!-- rad -->
-    <xacro:property name="ankle_effort_limit" value="21840"/> <!-- IU = 20 A -->
+    <xacro:property name="ankle_effort_limit" value="${max_effort_value}"/> <!-- IU = 20 A -->
     <xacro:property name="ankle_velocity_limit" value="1.0"/>
     <xacro:property name="hover_height" value="0.3"/>
     <xacro:property name="camera_link" value="0.05"/> <!-- Size of square 'camera' box -->
     <xacro:property name="axel_offset" value="0.05"/> <!-- Space btw top of beam and the each joint -->
-    <xacro:arg name="k_velocity_value" default="20000.0" />
-    <xacro:property name="k_velocity_value" value="$(arg k_velocity_value)" />
     <!-- Import all Gazebo-customization elements, including Gazebo colors -->
     <xacro:include filename="$(find march_description)/urdf/march.gazebo"/>

Commit message: Increase knee velocity limit
Set knee velocity limit at 2.5 rad/s

File: march_description/urdf/march-iv.xacro (robot description, xacro)
@@ -42,5 +42,5 @@
     <xacro:property name="knee_flexion_soft_buffer" value="${3*pi/180}"/> <!-- rad -->
     <xacro:property name="knee_effort_limit" value="${max_effort_value}"/> <!-- IU = 20 A -->
-    <xacro:property name="knee_velocity_limit" value="2.0"/>
+    <xacro:property name="knee_velocity_limit" value="2.5"/>
     <xacro:property name="ankle_rotation_lower_limit" value="${-25*pi/180}"/>
     <xacro:property name="ankle_rotation_upper_limit" value="${15*pi/180}"/>

Commit message: Increase the effort limit

File: march_description/urdf/march-iv.xacro (robot description, xacro)
@@ -7,5 +7,7 @@
     <!--Important note: when changing value make sure rviz fixed frame is set to the same value (moveit.rviz)-->
     <xacro:property name="parent_name" value="world"/>
-    <xacro:arg name="max_effort_value" default="21840.0" />
+    <xacro:arg name="max_effort_rotary" default="26000.0" />
+    <!--    Rotary effort limit could be increased to 30905.66 IU = 25 A -->
+    <xacro:arg name="max_effort_linear" default="22932.0" />  <!-- = 28 A -->
     <xacro:property name="max_effort_value" value="$(arg max_effort_value)" />
     <xacro:arg name="k_velocity_value" default="20000.0" />
@@ -30,10 +32,10 @@
     <xacro:property name="hip_fe_rotation_upper_limit" value="${100*pi/180}"/> <!-- rad -->
     <xacro:property name="hip_fe_soft_buffer" value="${3*pi/180}"/> <!-- rad -->
-    <xacro:property name="hip_fe_effort_limit" value="${max_effort_value}"/> <!-- IU = 20 A -->
+    <xacro:property name="hip_fe_effort_limit" value="${max_effort_rotary}"/> <!-- IU = 20 A -->
     <xacro:property name="hip_fe_velocity_limit" value="2.0"/> <!-- rad/s -->
     <xacro:property name="hip_aa_rotation_lower_limit" value="${-18*pi/180}"/> <!-- rad -->
     <xacro:property name="hip_aa_rotation_upper_limit" value="${17*pi/180}"/> <!-- rad -->
     <xacro:property name="hip_aa_soft_buffer" value="${3.5*pi/180}"/> <!-- rad -->
-    <xacro:property name="hip_aa_effort_limit" value="${max_effort_value}"/> <!-- IU = 20 A -->
+    <xacro:property name="hip_aa_effort_limit" value="${max_effort_linear}"/> <!-- IU = 20 A -->
     <xacro:property name="hip_aa_velocity_limit" value="1.0"/> <!-- rad/s -->
     <xacro:property name="knee_rotation_lower_limit" value="${-5*pi/180}"/>
@@ -41,5 +43,5 @@
     <xacro:property name="knee_extension_soft_buffer" value="${3.5*pi/180}"/> <!-- rad -->
     <xacro:property name="knee_flexion_soft_buffer" value="${3*pi/180}"/> <!-- rad -->
-    <xacro:property name="knee_effort_limit" value="${max_effort_value}"/> <!-- IU = 20 A -->
+    <xacro:property name="knee_effort_limit" value="${max_effort_rotary}"/> <!-- IU = 20 A -->
     <xacro:property name="knee_velocity_limit" value="2.5"/>
     <xacro:property name="ankle_rotation_lower_limit" value="${-25*pi/180}"/>
@@ -47,5 +49,5 @@
     <xacro:property name="ankle_dorsalflexion_soft_buffer" value="${5*pi/180}"/> <!-- rad -->
     <xacro:property name="ankle_plantarflexion_soft_buffer" value="${3*pi/180}"/> <!-- rad -->
-    <xacro:property name="ankle_effort_limit" value="${max_effort_value}"/> <!-- IU = 20 A -->
+    <xacro:property name="ankle_effort_limit" value="${max_effort_linear}"/> <!-- IU = 20 A -->
     <xacro:property name="ankle_velocity_limit" value="1.0"/>
     <xacro:property name="hover_height" value="0.3"/>
