Commit message: PM-8 Add correct masses of the parts.

File: march_description/urdf/march-iv.xacro (robot description, xacro)
@@ -12,19 +12,30 @@
     <xacro:property name="k_velocity_value" value="$(arg k_velocity_value)" />
     <!-- Constants for robot dimensions -->
-    <!-- TODO @Jitske: add accurate masses and inertia for all links -->
-    <xacro:property name="mass" value="1"/> <!-- arbitrary value for mass -->
+    <!-- Masses determined in https://confluence.projectmarch.nl:8443/display/41TECH/Weights+of+the+Exoskeleton -->
     <xacro:property name="width" value="0.05"/> <!-- Square dimensions (widthxwidth) of beams -->
     <xacro:property name="upper_leg_height" value="${0.385}"/>
-    <xacro:property name="upper_leg_mass" value="1.080"/>
+    <xacro:property name="upper_leg_mass" value="7.238"/>
+    <!-- mass = KFE joint + HFE joint + Upper leg -->
     <xacro:property name="lower_leg_height" value="${0.385}"/>
-    <xacro:property name="lower_leg_mass" value="1.133"/>
+    <xacro:property name="lower_leg_mass" value="2.944"/>
+    <!-- mass = Ankle actuator + Lower leg -->
     <xacro:property name="foot_height_forward" value="${0.184}"/>
     <xacro:property name="foot_height_backward" value="${0.059}"/>
-    <xacro:property name="foot_mass" value="0.393"/>
+    <xacro:property name="foot_mass" value="0.847"/>
+    <!-- mass = Passive ankle + foot -->
+    <xacro:property name="ankle_mass" value="0"/>
+    <!-- ankle mass has been included in the foot mass -->
     <xacro:property name="ankle_plate_height" value="0.07"/>
     <xacro:property name="hip_height" value="0.420"/>
     <xacro:property name="hip_base_height" value="0.160"/>
+    <xacro:property name="hip_base_mass" value="6.089"/>
+    <!-- mass = Hip base + HAA actuators -->
     <xacro:property name="hip_aa_frame_height" value="0.130"/>
     <xacro:property name="hip_aa_frame_width" value="0.1395"/>
+    <xacro:property name="hip_aa_mass" value="1.407"/>
+    <!-- mass = Moving hip -->
+    <xacro:property name="hip_aa_mass_front" value="0"/>
+    <!-- hip_aa_mass_front has been included in the hip_aa_mass -->
+    <!-- Joint properties -->
     <xacro:property name="hip_fe_rotation_lower_limit" value="${-20*pi/180}"/> <!-- rad -->
     <xacro:property name="hip_fe_rotation_upper_limit" value="${100*pi/180}"/> <!-- rad -->
@@ -62,4 +73,5 @@
     <!-- Used for fixing robot to Gazebo 'base_link' -->
     <link name="${parent_name}"/>
+    <!-- Joints -->
     <joint name="hip" type="fixed">
         <parent link="${parent_name}"/>
@@ -72,5 +84,4 @@
         <origin xyz="0 ${-hip_base_height/2} 0" rpy="0 0 0"/>
         <axis xyz="-1 0 0"/>
-<!-- TODO: @JitskedeVries  Improve k values-->
         <limit velocity="${hip_aa_velocity_limit}" effort="${hip_aa_effort_limit}" lower="${hip_aa_rotation_lower_limit}" upper="${hip_aa_rotation_upper_limit}"/>
         <safety_controller soft_lower_limit="${hip_aa_rotation_lower_limit + hip_aa_soft_buffer}" soft_upper_limit="${hip_aa_rotation_upper_limit - hip_aa_soft_buffer}" k_position="5" k_velocity="${k_velocity_value}" />
@@ -162,4 +173,5 @@
         <material>Gazebo/Blue</material>
     </gazebo>
+    <!-- Parts -->
     <!-- Hip-->
     <link name="hip_base">
@@ -173,9 +185,9 @@
         <inertial>
             <origin xyz="0 0 0" rpy="0 0 0"/>
-            <mass value="${mass}"/>
-            <inertia
-                    ixx="${mass / 12.0 * (width*width + lower_leg_height*lower_leg_height)}" ixy="0.0" ixz="0.0"
-                    iyy="${mass / 12.0 * (lower_leg_height*lower_leg_height + width*width)}" iyz="0.0"
-                    izz="${mass / 12.0 * (width*width + width*width)}"/>
+            <mass value="${hip_base_mass}"/>
+            <inertia
+                    ixx="${hip_base_mass / 12.0 * (width*width + lower_leg_height*lower_leg_height)}" ixy="0.0" ixz="0.0"
+                    iyy="${hip_base_mass / 12.0 * (lower_leg_height*lower_leg_height + width*width)}" iyz="0.0"
+                    izz="${hip_base_mass / 12.0 * (width*width + width*width)}"/>
         </inertial>
         <collision>
@@ -197,9 +209,9 @@
         <inertial>
             <origin xyz="0 ${-hip_aa_frame_height/2} 0" rpy="0 0 0"/>
-            <mass value="${mass}"/>
-            <inertia
-                    ixx="${mass / 12.0 * (width*width + lower_leg_height*lower_leg_height)}" ixy="0.0" ixz="0.0"
-                    iyy="${mass / 12.0 * (lower_leg_height*lower_leg_height + width*width)}" iyz="0.0"
-                    izz="${mass / 12.0 * (width*width + width*width)}"/>
+            <mass value="${hip_aa_mass}"/>
+            <inertia
+                    ixx="${hip_aa_mass / 12.0 * (width*width + lower_leg_height*lower_leg_height)}" ixy="0.0" ixz="0.0"
+                    iyy="${hip_aa_mass / 12.0 * (lower_leg_height*lower_leg_height + width*width)}" iyz="0.0"
+                    izz="${hip_aa_mass / 12.0 * (width*width + width*width)}"/>
         </inertial>
         <collision>
@@ -213,9 +225,9 @@
         <inertial>
             <origin xyz="${-hip_aa_frame_width/2} 0 0" rpy="0 0 0"/>
-            <mass value="${mass}"/>
-            <inertia
-                    ixx="${mass / 12.0 * (width*width + lower_leg_height*lower_leg_height)}" ixy="0.0" ixz="0.0"
-                    iyy="${mass / 12.0 * (lower_leg_height*lower_leg_height + width*width)}" iyz="0.0"
-                    izz="${mass / 12.0 * (width*width + width*width)}"/>
+            <mass value="${hip_aa_mass_front}"/>
+            <inertia
+                    ixx="${hip_aa_mass_front / 12.0 * (width*width + lower_leg_height*lower_leg_height)}" ixy="0.0" ixz="0.0"
+                    iyy="${hip_aa_mass_front / 12.0 * (lower_leg_height*lower_leg_height + width*width)}" iyz="0.0"
+                    izz="${hip_aa_mass_front / 12.0 * (width*width + width*width)}"/>
         </inertial>
         <collision>
@@ -239,7 +251,7 @@
             <mass value="${upper_leg_mass}"/>
             <inertia
-                    ixx="${mass / 12.0 * (width*width + upper_leg_height*upper_leg_height)}" ixy="0.0" ixz="0.0"
-                    iyy="${mass / 12.0 * (upper_leg_height*upper_leg_height + width*width)}" iyz="0.0"
-                    izz="${mass / 12.0 * (width*width + width*width)}"/>
+                    ixx="${upper_leg_mass / 12.0 * (width*width + upper_leg_height*upper_leg_height)}" ixy="0.0" ixz="0.0"
+                    iyy="${upper_leg_mass / 12.0 * (upper_leg_height*upper_leg_height + width*width)}" iyz="0.0"
+                    izz="${upper_leg_mass / 12.0 * (width*width + width*width)}"/>
         </inertial>
         <collision>
@@ -263,7 +275,7 @@
             <mass value="${lower_leg_mass}"/>
             <inertia
-                    ixx="${mass / 12.0 * (width*width + lower_leg_height*lower_leg_height)}" ixy="0.0" ixz="0.0"
-                    iyy="${mass / 12.0 * (lower_leg_height*lower_leg_height + width*width)}" iyz="0.0"
-                    izz="${mass / 12.0 * (width*width + width*width)}"/>
+                    ixx="${lower_leg_mass / 12.0 * (width*width + lower_leg_height*lower_leg_height)}" ixy="0.0" ixz="0.0"
+                    iyy="${lower_leg_mass / 12.0 * (lower_leg_height*lower_leg_height + width*width)}" iyz="0.0"
+                    izz="${lower_leg_mass / 12.0 * (width*width + width*width)}"/>
         </inertial>
         <collision>
@@ -274,5 +286,5 @@
         </collision>
     </link>
-    <!-- Lower Leg Left -->
+    <!-- Ankle plate Left -->
     <link name="ankle_plate_left">
         <visual>
@@ -285,9 +297,9 @@
         <inertial>
             <origin xyz="0 0 ${-ankle_plate_height/2}" rpy="0 0 0"/>
-            <mass value="${mass}"/>
-            <inertia
-                    ixx="${mass / 12.0 * (width*width + lower_leg_height*lower_leg_height)}" ixy="0.0" ixz="0.0"
-                    iyy="${mass / 12.0 * (lower_leg_height*lower_leg_height + width*width)}" iyz="0.0"
-                    izz="${mass / 12.0 * (width*width + width*width)}"/>
+            <mass value="${foot_mass}"/>
+            <inertia
+                    ixx="${ankle_mass / 12.0 * (width*width + lower_leg_height*lower_leg_height)}" ixy="0.0" ixz="0.0"
+                    iyy="${ankle_mass / 12.0 * (lower_leg_height*lower_leg_height + width*width)}" iyz="0.0"
+                    izz="${ankle_mass / 12.0 * (width*width + width*width)}"/>
         </inertial>
         <collision>
@@ -304,7 +316,7 @@
             <mass value="${foot_mass}"/>
             <inertia
-                    ixx="${mass / 12.0 * (width*width + lower_leg_height*lower_leg_height)}" ixy="0.0" ixz="0.0"
-                    iyy="${mass / 12.0 * (lower_leg_height*lower_leg_height + width*width)}" iyz="0.0"
-                    izz="${mass / 12.0 * (width*width + width*width)}"/>
+                    ixx="${foot_mass / 12.0 * (width*width + lower_leg_height*lower_leg_height)}" ixy="0.0" ixz="0.0"
+                    iyy="${foot_mass / 12.0 * (lower_leg_height*lower_leg_height + width*width)}" iyz="0.0"
+                    izz="${foot_mass / 12.0 * (width*width + width*width)}"/>
         </inertial>
         <collision>
@@ -326,9 +338,9 @@
         <inertial>
             <origin xyz="0 ${hip_aa_frame_height/2} 0" rpy="0 0 0"/>
-            <mass value="${mass}"/>
-            <inertia
-                    ixx="${mass / 12.0 * (width*width + lower_leg_height*lower_leg_height)}" ixy="0.0" ixz="0.0"
-                    iyy="${mass / 12.0 * (lower_leg_height*lower_leg_height + width*width)}" iyz="0.0"
-                    izz="${mass / 12.0 * (width*width + width*width)}"/>
+            <mass value="${hip_aa_mass}"/>
+            <inertia
+                    ixx="${hip_aa_mass / 12.0 * (width*width + lower_leg_height*lower_leg_height)}" ixy="0.0" ixz="0.0"
+                    iyy="${hip_aa_mass / 12.0 * (lower_leg_height*lower_leg_height + width*width)}" iyz="0.0"
+                    izz="${hip_aa_mass / 12.0 * (width*width + width*width)}"/>
         </inertial>
         <collision>
@@ -342,9 +354,9 @@
         <inertial>
             <origin xyz="${-hip_aa_frame_width/2} 0 0" rpy="0 0 0"/>
-            <mass value="${mass}"/>
-            <inertia
-                    ixx="${mass / 12.0 * (width*width + lower_leg_height*lower_leg_height)}" ixy="0.0" ixz="0.0"
-                    iyy="${mass / 12.0 * (lower_leg_height*lower_leg_height + width*width)}" iyz="0.0"
-                    izz="${mass / 12.0 * (width*width + width*width)}"/>
+            <mass value="${hip_aa_mass_front}"/>
+            <inertia
+                    ixx="${hip_aa_mass_front / 12.0 * (width*width + lower_leg_height*lower_leg_height)}" ixy="0.0" ixz="0.0"
+                    iyy="${hip_aa_mass_front / 12.0 * (lower_leg_height*lower_leg_height + width*width)}" iyz="0.0"
+                    izz="${hip_aa_mass_front / 12.0 * (width*width + width*width)}"/>
         </inertial>
         <collision>
@@ -368,7 +380,7 @@
             <mass value="${upper_leg_mass}"/>
             <inertia
-                    ixx="${mass / 12.0 * (width*width + upper_leg_height*upper_leg_height)}" ixy="0.0" ixz="0.0"
-                    iyy="${mass / 12.0 * (upper_leg_height*upper_leg_height + width*width)}" iyz="0.0"
-                    izz="${mass / 12.0 * (width*width + width*width)}"/>
+                    ixx="${upper_leg_mass / 12.0 * (width*width + upper_leg_height*upper_leg_height)}" ixy="0.0" ixz="0.0"
+                    iyy="${upper_leg_mass / 12.0 * (upper_leg_height*upper_leg_height + width*width)}" iyz="0.0"
+                    izz="${upper_leg_mass / 12.0 * (width*width + width*width)}"/>
         </inertial>
         <collision>
@@ -392,7 +404,7 @@
             <mass value="${lower_leg_mass}"/>
             <inertia
-                    ixx="${mass / 12.0 * (width*width + lower_leg_height*lower_leg_height)}" ixy="0.0" ixz="0.0"
-                    iyy="${mass / 12.0 * (lower_leg_height*lower_leg_height + width*width)}" iyz="0.0"
-                    izz="${mass / 12.0 * (width*width + width*width)}"/>
+                    ixx="${lower_leg_mass / 12.0 * (width*width + lower_leg_height*lower_leg_height)}" ixy="0.0" ixz="0.0"
+                    iyy="${lower_leg_mass / 12.0 * (lower_leg_height*lower_leg_height + width*width)}" iyz="0.0"
+                    izz="${lower_leg_mass / 12.0 * (width*width + width*width)}"/>
         </inertial>
         <collision>
@@ -403,5 +415,5 @@
         </collision>
     </link>
-    <!-- Lower Leg Right -->
+    <!-- Ankle Plate Right -->
     <link name="ankle_plate_right">
         <visual>
@@ -414,9 +426,9 @@
         <inertial>
             <origin xyz="0 0 ${-ankle_plate_height/2}" rpy="0 0 0"/>
-            <mass value="${mass}"/>
-            <inertia
-                    ixx="${mass / 12.0 * (width*width + lower_leg_height*lower_leg_height)}" ixy="0.0" ixz="0.0"
-                    iyy="${mass / 12.0 * (lower_leg_height*lower_leg_height + width*width)}" iyz="0.0"
-                    izz="${mass / 12.0 * (width*width + width*width)}"/>
+            <mass value="${ankle_mass}"/>
+            <inertia
+                    ixx="${ankle_mass / 12.0 * (width*width + lower_leg_height*lower_leg_height)}" ixy="0.0" ixz="0.0"
+                    iyy="${ankle_mass / 12.0 * (lower_leg_height*lower_leg_height + width*width)}" iyz="0.0"
+                    izz="${ankle_mass / 12.0 * (width*width + width*width)}"/>
         </inertial>
         <collision>
@@ -431,9 +443,9 @@
         <inertial>
             <origin xyz="${(-foot_height_forward+foot_height_backward)/2} 0 0" rpy="0 0 0"/>
-            <mass value="${mass}"/>
-            <inertia
-                    ixx="${mass / 12.0 * (width*width + lower_leg_height*lower_leg_height)}" ixy="0.0" ixz="0.0"
-                    iyy="${mass / 12.0 * (lower_leg_height*lower_leg_height + width*width)}" iyz="0.0"
-                    izz="${mass / 12.0 * (width*width + width*width)}"/>
+            <mass value="${foot_mass}"/>
+            <inertia
+                    ixx="${foot_mass / 12.0 * (width*width + lower_leg_height*lower_leg_height)}" ixy="0.0" ixz="0.0"
+                    iyy="${foot_mass / 12.0 * (lower_leg_height*lower_leg_height + width*width)}" iyz="0.0"
+                    izz="${foot_mass / 12.0 * (width*width + width*width)}"/>
         </inertial>
         <collision>

Commit message: Fix two errors and a typo in the urdf.

File: march_description/urdf/march-iv.xacro (robot description, xacro)
@@ -9,5 +9,6 @@
     <xacro:arg name="max_effort_rotary" default="20475" /> <!-- = 25 A -->
     <xacro:arg name="max_effort_linear" default="22932.0" />  <!-- = 28 A -->
-    <xacro:property name="max_effort_value" value="$(arg max_effort_value)" />
+    <xacro:property name="max_effort_rotary" value="$(arg max_effort_rotary)" />
+    <xacro:property name="max_effort_linear" value="$(arg max_effort_linear)" />
     <xacro:arg name="k_velocity_value" default="20000.0" />
     <xacro:property name="k_velocity_value" value="$(arg k_velocity_value)" />
@@ -34,7 +35,7 @@
     <xacro:property name="hip_aa_frame_height" value="0.130"/>
     <xacro:property name="hip_aa_frame_width" value="0.1395"/>
-    <xacro:property name="hip_aa_mass" value="1.407"/>
+    <xacro:property name="hip_aa_mass" value="1.007"/>
     <!-- mass = Moving hip -->
-    <xacro:property name="hip_aa_mass_front" value="0"/>
+    <xacro:property name="hip_aa_mass_front" value="0.4"/>
     <!-- hip_aa_mass_front has been included in the hip_aa_mass -->
     <!-- Joint properties -->
@@ -298,5 +299,5 @@
         <inertial>
             <origin xyz="0 0 ${-ankle_plate_height/2}" rpy="0 0 0"/>
-            <mass value="${foot_mass}"/>
+            <mass value="${ankle_mass}"/>
             <inertia
                     ixx="${ankle_mass / 12.0 * (width*width + lower_leg_height*lower_leg_height)}" ixy="0.0" ixz="0.0"

Commit message: Remove the inertias of the fixed links.

File: march_description/urdf/march-iv.xacro (robot description, xacro)
@@ -26,6 +26,4 @@
     <xacro:property name="foot_mass" value="0.847"/>
     <!-- mass = Passive ankle + foot -->
-    <xacro:property name="ankle_mass" value="0"/>
-    <!-- ankle mass has been included in the foot mass -->
     <xacro:property name="ankle_plate_height" value="0.07"/>
     <xacro:property name="hip_height" value="0.420"/>
@@ -35,5 +33,5 @@
     <xacro:property name="hip_aa_frame_height" value="0.130"/>
     <xacro:property name="hip_aa_frame_width" value="0.1395"/>
-    <xacro:property name="hip_aa_mass" value="1.007"/>
+    <xacro:property name="hip_aa_mass" value="1.407"/>
     <!-- mass = Moving hip -->
     <xacro:property name="hip_aa_mass_front" value="0.4"/>
@@ -209,6 +207,14 @@
             <material name="blue"/>
         </visual>
-        <inertial>
+        <collision>
             <origin xyz="0 ${-hip_aa_frame_height/2} 0" rpy="0 0 0"/>
+            <geometry>
+                <box size="${width} ${hip_aa_frame_height} ${width}"/>
+            </geometry>
+        </collision>
+    </link>
+    <link name="hip_aa_frame_left_front">
+        <inertial>
+            <origin xyz="${-hip_aa_frame_width/2} 0 0" rpy="0 0 0"/>
             <mass value="${hip_aa_mass}"/>
             <inertia
@@ -218,20 +224,4 @@
         </inertial>
         <collision>
-            <origin xyz="0 ${-hip_aa_frame_height/2} 0" rpy="0 0 0"/>
-            <geometry>
-                <box size="${width} ${hip_aa_frame_height} ${width}"/>
-            </geometry>
-        </collision>
-    </link>
-    <link name="hip_aa_frame_left_front">
-        <inertial>
-            <origin xyz="${-hip_aa_frame_width/2} 0 0" rpy="0 0 0"/>
-            <mass value="${hip_aa_mass_front}"/>
-            <inertia
-                    ixx="${hip_aa_mass_front / 12.0 * (width*width + lower_leg_height*lower_leg_height)}" ixy="0.0" ixz="0.0"
-                    iyy="${hip_aa_mass_front / 12.0 * (lower_leg_height*lower_leg_height + width*width)}" iyz="0.0"
-                    izz="${hip_aa_mass_front / 12.0 * (width*width + width*width)}"/>
-        </inertial>
-        <collision>
             <origin xyz="${-hip_aa_frame_width/2} 0 0" rpy="0 0 0"/>
             <geometry>
@@ -297,12 +287,4 @@
             <material name="blue"/>
         </visual>
-        <inertial>
-            <origin xyz="0 0 ${-ankle_plate_height/2}" rpy="0 0 0"/>
-            <mass value="${ankle_mass}"/>
-            <inertia
-                    ixx="${ankle_mass / 12.0 * (width*width + lower_leg_height*lower_leg_height)}" ixy="0.0" ixz="0.0"
-                    iyy="${ankle_mass / 12.0 * (lower_leg_height*lower_leg_height + width*width)}" iyz="0.0"
-                    izz="${ankle_mass / 12.0 * (width*width + width*width)}"/>
-        </inertial>
         <collision>
             <origin xyz="0 0 ${-ankle_plate_height/2}" rpy="0 0 0"/>
@@ -338,6 +320,14 @@
             <material name="blue"/>
         </visual>
-        <inertial>
+        <collision>
             <origin xyz="0 ${hip_aa_frame_height/2} 0" rpy="0 0 0"/>
+            <geometry>
+                <box size="${width} ${hip_aa_frame_height} ${width}"/>
+            </geometry>
+        </collision>
+    </link>
+    <link name="hip_aa_frame_right_front">
+        <inertial>
+            <origin xyz="${-hip_aa_frame_width/2} 0 0" rpy="0 0 0"/>
             <mass value="${hip_aa_mass}"/>
             <inertia
@@ -347,20 +337,4 @@
         </inertial>
         <collision>
-            <origin xyz="0 ${hip_aa_frame_height/2} 0" rpy="0 0 0"/>
-            <geometry>
-                <box size="${width} ${hip_aa_frame_height} ${width}"/>
-            </geometry>
-        </collision>
-    </link>
-    <link name="hip_aa_frame_right_front">
-        <inertial>
-            <origin xyz="${-hip_aa_frame_width/2} 0 0" rpy="0 0 0"/>
-            <mass value="${hip_aa_mass_front}"/>
-            <inertia
-                    ixx="${hip_aa_mass_front / 12.0 * (width*width + lower_leg_height*lower_leg_height)}" ixy="0.0" ixz="0.0"
-                    iyy="${hip_aa_mass_front / 12.0 * (lower_leg_height*lower_leg_height + width*width)}" iyz="0.0"
-                    izz="${hip_aa_mass_front / 12.0 * (width*width + width*width)}"/>
-        </inertial>
-        <collision>
             <origin xyz="${-hip_aa_frame_width/2} 0 0" rpy="0 0 0"/>
             <geometry>
@@ -426,12 +400,4 @@
             <material name="blue"/>
         </visual>
-        <inertial>
-            <origin xyz="0 0 ${-ankle_plate_height/2}" rpy="0 0 0"/>
-            <mass value="${ankle_mass}"/>
-            <inertia
-                    ixx="${ankle_mass / 12.0 * (width*width + lower_leg_height*lower_leg_height)}" ixy="0.0" ixz="0.0"
-                    iyy="${ankle_mass / 12.0 * (lower_leg_height*lower_leg_height + width*width)}" iyz="0.0"
-                    izz="${ankle_mass / 12.0 * (width*width + width*width)}"/>
-        </inertial>
         <collision>
             <origin xyz="0 0 ${-ankle_plate_height/2}" rpy="0 0 0"/>
