Commit message: Add Center of Mass to URDF and fix lengths.

File: march_description/urdf/march-iv.xacro (robot description, xacro)
@@ -16,25 +16,44 @@
     <!-- Masses determined in https://confluence.projectmarch.nl:8443/display/41TECH/Weights+of+the+Exoskeleton -->
     <xacro:property name="width" value="0.05"/> <!-- Square dimensions (widthxwidth) of beams -->
-    <xacro:property name="upper_leg_height" value="${0.385}"/>
+    <xacro:property name="hip_base_height" value="0.160"/>
+    <xacro:property name="hip_base_mass" value="6.089"/>
+    <!-- mass = Hip base + HAA actuators -->
+    <xacro:property name="hip_aa_frame_height" value="0.170"/>
+    <xacro:property name="hip_aa_frame_width" value="0.1395"/>
+    <xacro:property name="hip_aa_mass" value="1.407"/>
+    <!-- mass = Moving hip -->
+    <xacro:property name="upper_leg_height" value="0.385"/>
     <xacro:property name="upper_leg_mass" value="7.238"/>
     <!-- mass = KFE joint + HFE joint + Upper leg -->
-    <xacro:property name="lower_leg_height" value="${0.385}"/>
+    <xacro:property name="lower_leg_height" value="0.385"/>
     <xacro:property name="lower_leg_mass" value="2.944"/>
     <!-- mass = Ankle actuator + Lower leg -->
+    <xacro:property name="ankle_plate_height" value="0.12"/>
     <xacro:property name="foot_height_forward" value="${0.184}"/>
     <xacro:property name="foot_height_backward" value="${0.059}"/>
     <xacro:property name="foot_mass" value="0.847"/>
     <!-- mass = Passive ankle + foot -->
-    <xacro:property name="ankle_plate_height" value="0.07"/>
-    <xacro:property name="hip_height" value="0.420"/>
-    <xacro:property name="hip_base_height" value="0.160"/>
-    <xacro:property name="hip_base_mass" value="6.089"/>
-    <!-- mass = Hip base + HAA actuators -->
-    <xacro:property name="hip_aa_frame_height" value="0.130"/>
-    <xacro:property name="hip_aa_frame_width" value="0.1395"/>
-    <xacro:property name="hip_aa_mass" value="1.407"/>
-    <!-- mass = Moving hip -->
-    <xacro:property name="hip_aa_mass_front" value="0.4"/>
-    <!-- hip_aa_mass_front has been included in the hip_aa_mass -->
+    <!-- Com of the parts -->
+    <!-- CoM has been determined in Catia, see https://confluence.projectmarch.nl:8443/display/51/URDF+description -->
+    <!-- The Catia locations were defined in a global coordinate system with the origin at the center of the
+         rotation axis of the two HFE joints. Here, the joints were all set at zero degrees. Hence, we need some
+         translations to transfer it to the reference frame of each of the parts. Not that in the Catia x axis is
+         the URDF y axis and the Catia y axis is the negative URDF x axis. The given CoM are for the right leg,
+         the y coordinate will be inverted for the left leg. -->
+    <xacro:property name="hip_base_com_x" value="${-hip_aa_frame_width + 0.124786}"/>
+    <xacro:property name="hip_base_com_y" value="0.00000911124"/>
+    <xacro:property name="hip_base_com_z" value="0.152163"/>
+    <xacro:property name="hip_aa_com_x" value="${-hip_aa_frame_width + 0.0669488}"/>
+    <xacro:property name="hip_aa_com_y" value="${-hip_base_height/2 - hip_aa_frame_height + 0.210566}"/>
+    <xacro:property name="hip_aa_com_z" value="-0.000250494"/>
+    <xacro:property name="upper_leg_com_x" value="-0.00219961"/>
+    <xacro:property name="upper_leg_com_y" value="${-hip_base_height/2 - hip_aa_frame_height + 0.221535}"/>
+    <xacro:property name="upper_leg_com_z" value="-0.184207"/>
+    <xacro:property name="lower_leg_com_x" value="-0.00434063"/>
+    <xacro:property name="lower_leg_com_y" value="${-hip_base_height/2 - hip_aa_frame_height + 0.184583}"/>
+    <xacro:property name="lower_leg_com_z" value="${upper_leg_height - 0.511661}"/>
+    <xacro:property name="foot_com_x" value="-0.0450791"/>
+    <xacro:property name="foot_com_y" value="${-hip_base_height/2 - hip_aa_frame_height + 0.147081}"/>
+    <xacro:property name="foot_com_z" value="${upper_leg_height + lower_leg_height + ankle_plate_height - 0.844751}"/>
     <!-- Joint properties -->
     <xacro:property name="hip_fe_rotation_lower_limit" value="${-20*pi/180}"/> <!-- rad -->
@@ -184,5 +203,5 @@
         </visual>
         <inertial>
-            <origin xyz="0 0 0" rpy="0 0 0"/>
+            <origin xyz="${hip_base_com_x} ${hip_base_com_y} ${hip_base_com_z}" rpy="0 0 0"/>
             <mass value="${hip_base_mass}"/>
             <inertia
@@ -219,5 +238,5 @@
     <link name="hip_aa_frame_left_front">
         <inertial>
-            <origin xyz="${-hip_aa_frame_width/2} 0 0" rpy="0 0 0"/>
+            <origin xyz="${hip_aa_com_x} ${-hip_aa_com_y} ${hip_aa_com_z}" rpy="0 0 0"/>
             <mass value="${hip_aa_mass}"/>
             <inertia
@@ -246,5 +265,5 @@
         </visual>
         <inertial>
-            <origin xyz="0 0 ${-upper_leg_height/2}" rpy="0 0 0"/>
+            <origin xyz="${upper_leg_com_x} ${-upper_leg_com_y} ${upper_leg_com_z}" rpy="0 0 0"/>
             <mass value="${upper_leg_mass}"/>
             <inertia
@@ -273,5 +292,5 @@
         </visual>
         <inertial>
-            <origin xyz="0 0 ${-lower_leg_height/2}" rpy="0 0 0"/>
+            <origin xyz="${lower_leg_com_x} ${-lower_leg_com_y} ${lower_leg_com_z}" rpy="0 0 0"/>
             <mass value="${lower_leg_mass}"/>
             <inertia
@@ -309,5 +328,5 @@
     <link name="foot_left">
         <inertial>
-            <origin xyz="${(-foot_height_forward+foot_height_backward)/2} 0 0" rpy="0 0 0"/>
+            <origin xyz="${foot_com_x} ${-foot_com_y} ${foot_com_z}" rpy="0 0 0"/>
             <mass value="${foot_mass}"/>
             <inertia
@@ -344,5 +363,5 @@
     <link name="hip_aa_frame_right_front">
         <inertial>
-            <origin xyz="${-hip_aa_frame_width/2} 0 0" rpy="0 0 0"/>
+            <origin xyz="${hip_aa_com_x} ${hip_aa_com_y} ${hip_aa_com_z}" rpy="0 0 0"/>
             <mass value="${hip_aa_mass}"/>
             <inertia
@@ -371,5 +390,5 @@
         </visual>
         <inertial>
-            <origin xyz="0 0 ${-upper_leg_height/2}" rpy="0 0 0"/>
+            <origin xyz="${upper_leg_com_x} ${upper_leg_com_y} ${upper_leg_com_z}" rpy="0 0 0"/>
             <mass value="${upper_leg_mass}"/>
             <inertia
@@ -398,5 +417,5 @@
         </visual>
         <inertial>
-            <origin xyz="0 0 ${-lower_leg_height/2}" rpy="0 0 0"/>
+            <origin xyz="${lower_leg_com_x} ${lower_leg_com_y} ${lower_leg_com_z}" rpy="0 0 0"/>
             <mass value="${lower_leg_mass}"/>
             <inertia
@@ -434,5 +453,5 @@
     <link name="foot_right">
         <inertial>
-            <origin xyz="${(-foot_height_forward+foot_height_backward)/2} 0 0" rpy="0 0 0"/>
+            <origin xyz="${foot_com_x} ${foot_com_y} ${foot_com_z}" rpy="0 0 0"/>
             <mass value="${foot_mass}"/>
             <inertia

Commit message: Fix axis of the inertias in the URDF.

File: march_description/urdf/march-iv.xacro (robot description, xacro)
@@ -38,5 +38,5 @@
     <!-- The Catia locations were defined in a global coordinate system with the origin at the center of the
          rotation axis of the two HFE joints. Here, the joints were all set at zero degrees. Hence, we need some
-         translations to transfer it to the reference frame of each of the parts. Not that in the Catia x axis is
+         translations to transfer it to the reference frame of each of the parts. Note that in the Catia x axis is
          the URDF y axis and the Catia y axis is the negative URDF x axis. The given CoM are for the right leg,
          the y coordinate will be inverted for the left leg. -->
@@ -56,4 +56,40 @@
     <xacro:property name="foot_com_y" value="${-hip_base_height/2 - hip_aa_frame_height + 0.147081}"/>
     <xacro:property name="foot_com_z" value="${upper_leg_height + lower_leg_height + ankle_plate_height - 0.844751}"/>
+    <!-- Inertia of the parts -->
+    <!-- Inertia's have been determined in Catia, see
+         https://confluence.projectmarch.nl:8443/display/51/URDF+description -->
+    <!-- The inertia's were defined around the CoM. Note that in the Catia x axis is the URDF y axis and the Catia y
+         axis is the negative URDF x axis, see confluence for the impact. The given inertia's are for the right leg,
+         Ixy and Iyz will be inverted for the left leg. -->
+    <xacro:property name="hip_base_Ixx" value="0.117325"/>
+    <xacro:property name="hip_base_Ixy" value="-0.0000239249"/>
+    <xacro:property name="hip_base_Ixz" value="0.0179732"/>
+    <xacro:property name="hip_base_Iyy" value="0.0745937"/>
+    <xacro:property name="hip_base_Iyz" value="-0.00000472801"/>
+    <xacro:property name="hip_base_Izz" value="0.0684134"/>
+    <xacro:property name="hip_aa_Ixx" value="0.00841686"/>
+    <xacro:property name="hip_aa_Ixy" value="0.00655578"/>
+    <xacro:property name="hip_aa_Ixz" value="0.0000910634"/>
+    <xacro:property name="hip_aa_Iyy" value="0.0165504"/>
+    <xacro:property name="hip_aa_Iyz" value="0.0000996411"/>
+    <xacro:property name="hip_aa_Izz" value="0.0229261"/>
+    <xacro:property name="upper_leg_Ixx" value="0.119187"/>
+    <xacro:property name="upper_leg_Ixy" value="-0.0000363676"/>
+    <xacro:property name="upper_leg_Ixz" value="-0.0000393791"/>
+    <xacro:property name="upper_leg_Iyy" value="0.11867"/>
+    <xacro:property name="upper_leg_Iyz" value="-0.0125652"/>
+    <xacro:property name="upper_leg_Izz" value="0.00881972"/>
+    <xacro:property name="lower_leg_Ixx" value="0.0725438"/>
+    <xacro:property name="lower_leg_Ixy" value="-0.0264923"/>
+    <xacro:property name="lower_leg_Ixz" value="0.00934723"/>
+    <xacro:property name="lower_leg_Iyy" value="0.108683"/>
+    <xacro:property name="lower_leg_Iyz" value="0.00109811"/>
+    <xacro:property name="lower_leg_Izz" value="0.0715361" />
+    <xacro:property name="foot_Ixx" value="0.00414758"/>
+    <xacro:property name="foot_Ixy" value="-0.00185339"/>
+    <xacro:property name="foot_Ixz" value="-0.00254464"/>
+    <xacro:property name="foot_Iyy" value="0.00855883"/>
+    <xacro:property name="foot_Iyz" value="-0.00166213"/>
+    <xacro:property name="foot_Izz" value="0.00715736" />
     <!-- Joint properties -->
     <xacro:property name="hip_fe_rotation_lower_limit" value="${-20*pi/180}"/> <!-- rad -->
@@ -206,10 +242,10 @@
             <mass value="${hip_base_mass}"/>
             <inertia
-                    ixx="0.0745937"
-                    ixy="0.0000239249"
-                    ixz="-0.00000472801"
-                    iyy="0.117325"
-                    iyz="-0.0179732"
-                    izz="0.0684134" />
+                    ixx="hip_base_Ixx"
+                    ixy="hip_base_Ixy"
+                    ixz="hip_base_Ixz"
+                    iyy="hip_base_Iyy"
+                    iyz="hip_base_Iyz"
+                    izz="hip_base_Izz" />
         </inertial>
         <collision>
@@ -241,10 +277,10 @@
             <mass value="${hip_aa_mass}"/>
             <inertia
-                    ixx="0.0165504"
-                    ixy="0.00655578"
-                    ixz="-0.0000996411"
-                    iyy="0.00841686"
-                    iyz="-0.0000910634"
-                    izz="0.0229261" />
+                    ixx="hip_aa_Ixx"
+                    ixy="-hip_aa_Ixy"
+                    ixz="hip_aa_Ixz"
+                    iyy="hip_aa_Iyy"
+                    iyz="-hip_aa_Iyz"
+                    izz="hip_aa_Izz" />
         </inertial>
         <collision>
@@ -268,10 +304,10 @@
             <mass value="${upper_leg_mass}"/>
             <inertia
-                    ixx="0.11867"
-                    ixy="-0.0000363676"
-                    ixz="0.0125652"
-                    iyy="0.119187"
-                    iyz="0.0000393791"
-                    izz="0.00881972" />
+                    ixx="upper_leg_Ixx"
+                    ixy="-upper_leg_Ixy"
+                    ixz="upper_leg_Ixz"
+                    iyy="upper_leg_Iyy"
+                    iyz="-upper_leg_Iyz"
+                    izz="upper_leg_Izz" />
         </inertial>
         <collision>
@@ -295,10 +331,10 @@
             <mass value="${lower_leg_mass}"/>
             <inertia
-                    ixx="0.108683"
-                    ixy="-0.0264923"
-                    ixz="-0.00109811"
-                    iyy="0.0725438"
-                    iyz="-0.00934723"
-                    izz="0.0715361" />
+                    ixx="lower_leg_Ixx"
+                    ixy="-lower_leg_Ixy"
+                    ixz="lower_leg_Ixz"
+                    iyy="lower_leg_Iyy"
+                    iyz="-lower_leg_Iyz"
+                    izz="lower_leg_Izz" />
         </inertial>
         <collision>
@@ -331,10 +367,10 @@
             <mass value="${foot_mass}"/>
             <inertia
-                    ixx="0.00855883"
-                    ixy="-0.00185339"
-                    ixz="0.00166213"
-                    iyy="0.00855883"
-                    iyz="0.00254464"
-                    izz="0.00715736" />
+                    ixx="foot_Ixx"
+                    ixy="-foot_Ixy"
+                    ixz="foot_Ixz"
+                    iyy="foot_Iyy"
+                    iyz="-foot_Iyz"
+                    izz="foot_Izz" />
         </inertial>
         <collision>
@@ -366,10 +402,10 @@
             <mass value="${hip_aa_mass}"/>
             <inertia
-                    ixx="0.0165504"
-                    ixy="-0.00655578"
-                    ixz="0.0000996411"
-                    iyy="0.00841686"
-                    iyz="-0.0000910634"
-                    izz="0.0229261" />
+                    ixx="hip_aa_Ixx"
+                    ixy="hip_aa_Ixy"
+                    ixz="hip_aa_Ixz"
+                    iyy="hip_aa_Iyy"
+                    iyz="hip_aa_Iyz"
+                    izz="hip_aa_Izz" />
         </inertial>
         <collision>
@@ -393,10 +429,10 @@
             <mass value="${upper_leg_mass}"/>
             <inertia
-                    ixx="0.11867"
-                    ixy="0.0000363676"
-                    ixz="-0.0125652"
-                    iyy="0.119187"
-                    iyz="0.0000393791"
-                    izz="0.00881972" />
+                    ixx="upper_leg_Ixx"
+                    ixy="upper_leg_Ixy"
+                    ixz="upper_leg_Ixz"
+                    iyy="upper_leg_Iyy"
+                    iyz="upper_leg_Iyz"
+                    izz="upper_leg_Izz" />
         </inertial>
         <collision>
@@ -420,10 +456,10 @@
             <mass value="${lower_leg_mass}"/>
             <inertia
-                    ixx="0.108683"
-                    ixy="0.0264923"
-                    ixz="0.00109811"
-                    iyy="0.0725438"
-                    iyz="-0.00934723"
-                    izz="0.0715361" />
+                    ixx="lower_leg_Ixx"
+                    ixy="lower_leg_Ixy"
+                    ixz="lower_leg_Ixz"
+                    iyy="lower_leg_Iyy"
+                    iyz="lower_leg_Iyz"
+                    izz="lower_leg_Izz" />
         </inertial>
         <collision>
@@ -456,10 +492,10 @@
             <mass value="${foot_mass}"/>
             <inertia
-                    ixx="0.00855883"
-                    ixy="0.00185339"
-                    ixz="-0.00166213"
-                    iyy="0.00855883"
-                    iyz="0.00254464"
-                    izz="0.00715736" />
+                    ixx="foot_Ixx"
+                    ixy="foot_Ixy"
+                    ixz="foot_Ixz"
+                    iyy="foot_Iyy"
+                    iyz="foot_Iyz"
+                    izz="foot_Izz" />
         </inertial>
         <collision>
