Commit message: Change order in URDF; first define parts, then joints.

File: march_description/urdf/march-iv.xacro (robot description, xacro)
@@ -128,4 +128,282 @@
     <!-- Used for fixing robot to Gazebo 'base_link' -->
     <link name="${parent_name}"/>
+    <!-- Parts -->
+    <!-- Hip-->
+    <link name="hip_base">
+        <visual>
+            <origin xyz="0 0 0" rpy="0 0 ${-pi/2}"/>
+            <geometry>
+                <mesh filename="package://march_description/urdf/stl-files/HipBase.stl" scale="1.15 1.15 1.15"/>
+            </geometry>
+            <material name="blue"/>
+        </visual>
+        <inertial>
+            <origin xyz="${hip_base_com_x} ${hip_base_com_y} ${hip_base_com_z}" rpy="0 0 0"/>
+            <mass value="${hip_base_mass}"/>
+            <inertia
+                    ixx="${hip_base_Ixx}"
+                    ixy="${hip_base_Ixy}"
+                    ixz="${hip_base_Ixz}"
+                    iyy="${hip_base_Iyy}"
+                    iyz="${hip_base_Iyz}"
+                    izz="${hip_base_Izz}" />
+        </inertial>
+        <collision>
+            <origin xyz="0 0 0" rpy="0 0 0"/>
+            <geometry>
+                <box size="${width} ${hip_base_height} ${width}"/>
+            </geometry>
+        </collision>
+    </link>
+    <!-- Left Moving Hip-->
+    <link name="hip_aa_frame_left_side">
+        <visual>
+            <origin xyz="0 0 0" rpy="0 0 ${-pi/2}"/>
+            <geometry>
+                <mesh filename="package://march_description/urdf/stl-files/HipLeft.stl" scale="1.15 1.15 1.15"/>
+            </geometry>
+            <material name="blue"/>
+        </visual>
+        <collision>
+            <origin xyz="0 ${-hip_aa_frame_height/2} 0" rpy="0 0 0"/>
+            <geometry>
+                <box size="${width} ${hip_aa_frame_height} ${width}"/>
+            </geometry>
+        </collision>
+    </link>
+    <link name="hip_aa_frame_left_front">
+        <inertial>
+            <origin xyz="${hip_aa_com_x} ${-hip_aa_com_y} ${hip_aa_com_z}" rpy="0 0 0"/>
+            <mass value="${hip_aa_mass}"/>
+            <inertia
+                    ixx="${hip_aa_Ixx}"
+                    ixy="${-hip_aa_Ixy}"
+                    ixz="${hip_aa_Ixz}"
+                    iyy="${hip_aa_Iyy}"
+                    iyz="${-hip_aa_Iyz}"
+                    izz="${hip_aa_Izz}" />
+        </inertial>
+        <collision>
+            <origin xyz="${-hip_aa_frame_width/2} 0 0" rpy="0 0 0"/>
+            <geometry>
+                <box size="${hip_aa_frame_width} ${width} ${width}"/>
+            </geometry>
+        </collision>
+    </link>
+    <!-- Upper Leg Left-->
+    <link name="upper_leg_left">
+        <visual>
+            <origin xyz="0 0 0" rpy="0 0 ${-pi/2}"/>
+            <geometry>
+                <mesh filename="package://march_description/urdf/stl-files/UpperLegLeft.stl" scale="1.15 1.15 1.15"/>
+            </geometry>
+            <material name="blue"/>
+        </visual>
+        <inertial>
+            <origin xyz="${upper_leg_com_x} ${-upper_leg_com_y} ${upper_leg_com_z}" rpy="0 0 0"/>
+            <mass value="${upper_leg_mass}"/>
+            <inertia
+                    ixx="${upper_leg_Ixx}"
+                    ixy="${-upper_leg_Ixy}"
+                    ixz="${upper_leg_Ixz}"
+                    iyy="${upper_leg_Iyy}"
+                    iyz="${-upper_leg_Iyz}"
+                    izz="${upper_leg_Izz}" />
+        </inertial>
+        <collision>
+            <origin xyz="0 0 ${-upper_leg_height/2}" rpy="0 0 0"/>
+            <geometry>
+                <box size="${width} ${width} ${upper_leg_height}"/>
+            </geometry>
+        </collision>
+    </link>
+    <!-- Lower Leg Left -->
+    <link name="lower_leg_left">
+        <visual>
+            <origin xyz="0 0 0" rpy="0 0 ${-pi/2}"/>
+            <geometry>
+                <mesh filename="package://march_description/urdf/stl-files/LowerLegLeft.stl" scale="1.15 1.15 1.15"/>
+            </geometry>
+            <material name="blue"/>
+        </visual>
+        <inertial>
+            <origin xyz="${lower_leg_com_x} ${-lower_leg_com_y} ${lower_leg_com_z}" rpy="0 0 0"/>
+            <mass value="${lower_leg_mass}"/>
+            <inertia
+                    ixx="${lower_leg_Ixx}"
+                    ixy="${-lower_leg_Ixy}"
+                    ixz="${lower_leg_Ixz}"
+                    iyy="${lower_leg_Iyy}"
+                    iyz="${-lower_leg_Iyz}"
+                    izz="${lower_leg_Izz}" />
+        </inertial>
+        <collision>
+            <origin xyz="0 0 ${-lower_leg_height/2}" rpy="0 0 0"/>
+            <geometry>
+                <box size="${width} ${width} ${lower_leg_height}"/>
+            </geometry>
+        </collision>
+    </link>
+    <!-- Ankle plate Left -->
+    <link name="ankle_plate_left">
+        <visual>
+            <origin xyz="0 0 0" rpy="0 0 ${-pi/2}"/>
+            <geometry>
+                <mesh filename="package://march_description/urdf/stl-files/FootLeft.stl" scale="1.15 1.15 1.15"/>
+            </geometry>
+            <material name="blue"/>
+        </visual>
+        <collision>
+            <origin xyz="0 0 ${-ankle_plate_height/2}" rpy="0 0 0"/>
+            <geometry>
+                <box size="${width} ${width} ${ankle_plate_height}"/>
+            </geometry>
+        </collision>
+    </link>
+    <!-- Foot Left -->
+    <link name="foot_left">
+        <inertial>
+            <origin xyz="${foot_com_x} ${-foot_com_y} ${foot_com_z}" rpy="0 0 0"/>
+            <mass value="${foot_mass}"/>
+            <inertia
+                    ixx="${foot_Ixx}"
+                    ixy="${-foot_Ixy}"
+                    ixz="${foot_Ixz}"
+                    iyy="${foot_Iyy}"
+                    iyz="${-foot_Iyz}"
+                    izz="${foot_Izz}" />
+        </inertial>
+        <collision>
+            <origin xyz="${(-foot_height_forward+foot_height_backward)/2} 0 0" rpy="0 0 0"/>
+            <geometry>
+                <box size="${foot_height_forward+foot_height_backward} ${width} ${width}"/>
+            </geometry>
+        </collision>
+    </link>
+    <!-- Right Moving Hip-->
+    <link name="hip_aa_frame_right_side">
+        <visual>
+            <origin xyz="0 0 0" rpy="0 0 ${-pi/2}"/>
+            <geometry>
+                <mesh filename="package://march_description/urdf/stl-files/HipRight.stl" scale="1.15 1.15 1.15"/>
+            </geometry>
+            <material name="blue"/>
+        </visual>
+        <collision>
+            <origin xyz="0 ${hip_aa_frame_height/2} 0" rpy="0 0 0"/>
+            <geometry>
+                <box size="${width} ${hip_aa_frame_height} ${width}"/>
+            </geometry>
+        </collision>
+    </link>
+    <link name="hip_aa_frame_right_front">
+        <inertial>
+            <origin xyz="${hip_aa_com_x} ${hip_aa_com_y} ${hip_aa_com_z}" rpy="0 0 0"/>
+            <mass value="${hip_aa_mass}"/>
+            <inertia
+                    ixx="${hip_aa_Ixx}"
+                    ixy="${hip_aa_Ixy}"
+                    ixz="${hip_aa_Ixz}"
+                    iyy="${hip_aa_Iyy}"
+                    iyz="${hip_aa_Iyz}"
+                    izz="${hip_aa_Izz}" />
+        </inertial>
+        <collision>
+            <origin xyz="${-hip_aa_frame_width/2} 0 0" rpy="0 0 0"/>
+            <geometry>
+                <box size="${hip_aa_frame_width} ${width} ${width}"/>
+            </geometry>
+        </collision>
+    </link>
+    <!-- Upper Leg Right-->
+    <link name="upper_leg_right">
+        <visual>
+            <origin xyz="0 0 0" rpy="0 0 ${-pi/2}"/>
+            <geometry>
+                <mesh filename="package://march_description/urdf/stl-files/UpperLegRight.stl" scale="1.15 1.15 1.15"/>
+            </geometry>
+            <material name="blue"/>
+        </visual>
+        <inertial>
+            <origin xyz="${upper_leg_com_x} ${upper_leg_com_y} ${upper_leg_com_z}" rpy="0 0 0"/>
+            <mass value="${upper_leg_mass}"/>
+            <inertia
+                    ixx="${upper_leg_Ixx}"
+                    ixy="${upper_leg_Ixy}"
+                    ixz="${upper_leg_Ixz}"
+                    iyy="${upper_leg_Iyy}"
+                    iyz="${upper_leg_Iyz}"
+                    izz="${upper_leg_Izz}" />
+        </inertial>
+        <collision>
+            <origin xyz="0 0 ${-upper_leg_height/2}" rpy="0 0 0"/>
+            <geometry>
+                <box size="${width} ${width} ${upper_leg_height}"/>
+            </geometry>
+        </collision>
+    </link>
+    <!-- Lower Leg Right -->
+    <link name="lower_leg_right">
+        <visual>
+            <origin xyz="0 0 0" rpy="0 0 ${-pi/2}"/>
+            <geometry>
+                <mesh filename="package://march_description/urdf/stl-files/LowerLegRight.stl" scale="1.15 1.15 1.15"/>
+            </geometry>
+            <material name="blue"/>
+        </visual>
+        <inertial>
+            <origin xyz="${lower_leg_com_x} ${lower_leg_com_y} ${lower_leg_com_z}" rpy="0 0 0"/>
+            <mass value="${lower_leg_mass}"/>
+            <inertia
+                    ixx="${lower_leg_Ixx}"
+                    ixy="${lower_leg_Ixy}"
+                    ixz="${lower_leg_Ixz}"
+                    iyy="${lower_leg_Iyy}"
+                    iyz="${lower_leg_Iyz}"
+                    izz="${lower_leg_Izz}" />
+        </inertial>
+        <collision>
+            <origin xyz="0 0 ${-lower_leg_height/2}" rpy="0 0 0"/>
+            <geometry>
+                <box size="${width} ${width} ${lower_leg_height}"/>
+            </geometry>
+        </collision>
+    </link>
+    <!-- Ankle Plate Right -->
+    <link name="ankle_plate_right">
+        <visual>
+            <origin xyz="0 0 0" rpy="0 0 ${-pi/2}"/>
+            <geometry>
+                <mesh filename="package://march_description/urdf/stl-files/FootRight.stl" scale="1.15 1.15 1.15"/>
+            </geometry>
+            <material name="blue"/>
+        </visual>
+        <collision>
+            <origin xyz="0 0 ${-ankle_plate_height/2}" rpy="0 0 0"/>
+            <geometry>
+                <box size="${width} ${width} ${ankle_plate_height}"/>
+            </geometry>
+        </collision>
+    </link>
+    <!-- Foot Right -->
+    <link name="foot_right">
+        <inertial>
+            <origin xyz="${foot_com_x} ${foot_com_y} ${foot_com_z}" rpy="0 0 0"/>
+            <mass value="${foot_mass}"/>
+            <inertia
+                    ixx="${foot_Ixx}"
+                    ixy="${foot_Ixy}"
+                    ixz="${foot_Ixz}"
+                    iyy="${foot_Iyy}"
+                    iyz="${foot_Iyz}"
+                    izz="${foot_Izz}" />
+        </inertial>
+        <collision>
+            <origin xyz="${(-foot_height_forward+foot_height_backward)/2} 0 0" rpy="0 0 0"/>
+            <geometry>
+                <box size="${foot_height_forward+foot_height_backward} ${width} ${width}"/>
+            </geometry>
+        </collision>
+    </link>
     <!-- Joints -->
     <joint name="hip" type="fixed">
@@ -218,292 +496,4 @@
         <origin xyz="0 0 ${-ankle_plate_height}" rpy="0 0 0"/>
     </joint>
-    <!-- give colors to some links in gazebo -->
-    <gazebo reference="hip_base">
-        <material>Gazebo/Blue</material>
-    </gazebo>
-    <gazebo reference="foot_left">
-        <material>Gazebo/Blue</material>
-    </gazebo>
-    <gazebo reference="foot_right">
-        <material>Gazebo/Blue</material>
-    </gazebo>
-    <!-- Parts -->
-    <!-- Hip-->
-    <link name="hip_base">
-        <visual>
-            <origin xyz="0 0 0" rpy="0 0 ${-pi/2}"/>
-            <geometry>
-                <mesh filename="package://march_description/urdf/stl-files/HipBase.stl" scale="1.15 1.15 1.15"/>
-            </geometry>
-            <material name="blue"/>
-        </visual>
-        <inertial>
-            <origin xyz="${hip_base_com_x} ${hip_base_com_y} ${hip_base_com_z}" rpy="0 0 0"/>
-            <mass value="${hip_base_mass}"/>
-            <inertia
-                    ixx="${hip_base_Ixx}"
-                    ixy="${hip_base_Ixy}"
-                    ixz="${hip_base_Ixz}"
-                    iyy="${hip_base_Iyy}"
-                    iyz="${hip_base_Iyz}"
-                    izz="${hip_base_Izz}" />
-        </inertial>
-        <collision>
-            <origin xyz="0 0 0" rpy="0 0 0"/>
-            <geometry>
-                <box size="${width} ${hip_base_height} ${width}"/>
-            </geometry>
-        </collision>
-    </link>
-    <!-- Left Moving Hip-->
-    <link name="hip_aa_frame_left_side">
-        <visual>
-            <origin xyz="0 0 0" rpy="0 0 ${-pi/2}"/>
-            <geometry>
-                <mesh filename="package://march_description/urdf/stl-files/HipLeft.stl" scale="1.15 1.15 1.15"/>
-            </geometry>
-            <material name="blue"/>
-        </visual>
-        <collision>
-            <origin xyz="0 ${-hip_aa_frame_height/2} 0" rpy="0 0 0"/>
-            <geometry>
-                <box size="${width} ${hip_aa_frame_height} ${width}"/>
-            </geometry>
-        </collision>
-    </link>
-    <link name="hip_aa_frame_left_front">
-        <inertial>
-            <origin xyz="${hip_aa_com_x} ${-hip_aa_com_y} ${hip_aa_com_z}" rpy="0 0 0"/>
-            <mass value="${hip_aa_mass}"/>
-            <inertia
-                    ixx="${hip_aa_Ixx}"
-                    ixy="${-hip_aa_Ixy}"
-                    ixz="${hip_aa_Ixz}"
-                    iyy="${hip_aa_Iyy}"
-                    iyz="${-hip_aa_Iyz}"
-                    izz="${hip_aa_Izz}" />
-        </inertial>
-        <collision>
-            <origin xyz="${-hip_aa_frame_width/2} 0 0" rpy="0 0 0"/>
-            <geometry>
-                <box size="${hip_aa_frame_width} ${width} ${width}"/>
-            </geometry>
-        </collision>
-    </link>
-    <!-- Upper Leg Left-->
-    <link name="upper_leg_left">
-        <visual>
-            <origin xyz="0 0 0" rpy="0 0 ${-pi/2}"/>
-            <geometry>
-                <mesh filename="package://march_description/urdf/stl-files/UpperLegLeft.stl" scale="1.15 1.15 1.15"/>
-            </geometry>
-            <material name="blue"/>
-        </visual>
-        <inertial>
-            <origin xyz="${upper_leg_com_x} ${-upper_leg_com_y} ${upper_leg_com_z}" rpy="0 0 0"/>
-            <mass value="${upper_leg_mass}"/>
-            <inertia
-                    ixx="${upper_leg_Ixx}"
-                    ixy="${-upper_leg_Ixy}"
-                    ixz="${upper_leg_Ixz}"
-                    iyy="${upper_leg_Iyy}"
-                    iyz="${-upper_leg_Iyz}"
-                    izz="${upper_leg_Izz}" />
-        </inertial>
-        <collision>
-            <origin xyz="0 0 ${-upper_leg_height/2}" rpy="0 0 0"/>
-            <geometry>
-                <box size="${width} ${width} ${upper_leg_height}"/>
-            </geometry>
-        </collision>
-    </link>
-    <!-- Lower Leg Left -->
-    <link name="lower_leg_left">
-        <visual>
-            <origin xyz="0 0 0" rpy="0 0 ${-pi/2}"/>
-            <geometry>
-                <mesh filename="package://march_description/urdf/stl-files/LowerLegLeft.stl" scale="1.15 1.15 1.15"/>
-            </geometry>
-            <material name="blue"/>
-        </visual>
-        <inertial>
-            <origin xyz="${lower_leg_com_x} ${-lower_leg_com_y} ${lower_leg_com_z}" rpy="0 0 0"/>
-            <mass value="${lower_leg_mass}"/>
-            <inertia
-                    ixx="${lower_leg_Ixx}"
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
Commit message: initial commit, working for velocities, bad printing

File: march_description/urdf/march-iv.xacro (robot description, xacro)
@@ -131,5 +131,5 @@
     <!-- Hip-->
     <link name="hip_base">
-        <visual>
+        <vcolisual>
             <origin xyz="0 0 0" rpy="0 0 ${-pi/2}"/>
             <geometry>
@@ -137,5 +137,5 @@
             </geometry>
             <material name="blue"/>
-        </visual>
+        </vcolisual>
         <inertial>
             <origin xyz="${hip_base_com_x} ${hip_base_com_y} ${hip_base_com_z}" rpy="0 0 0"/>

Commit message: Reverted some accidental chagnes

File: march_description/urdf/march-iv.xacro (robot description, xacro)
@@ -131,5 +131,5 @@
     <!-- Hip-->
     <link name="hip_base">
-        <vcolisual>
+        <visual>
             <origin xyz="0 0 0" rpy="0 0 ${-pi/2}"/>
             <geometry>
@@ -137,5 +137,5 @@
             </geometry>
             <material name="blue"/>
-        </vcolisual>
+        </visual>
         <inertial>
             <origin xyz="${hip_base_com_x} ${hip_base_com_y} ${hip_base_com_z}" rpy="0 0 0"/>
