Commit message: added package for moveit configuration

File: march_description/urdf/march4.xacro (robot description, xacro)
@@ -6,6 +6,6 @@
     <!-- Value set to: 'base_link' makes the robot stand on the ground also set launch parameter fixed to false and set
     the hover_height to 0.0-->
-    <xacro:property name="parent_name" value="world"/>
-    <xacro:property name="hover_height" value="0.3"/>
+    <xacro:property name="parent_name" value="base_link"/>
+    <xacro:property name="hover_height" value="0.0"/>
     <xacro:arg name="max_effort_rotary" default="20475" /> <!-- = 25 A -->
     <xacro:arg name="max_effort_linear" default="22932.0" />  <!-- = 28 A -->

Commit message: Feature/gazebo com controller (#435)
* Make test plugin

* Make test model plugin

* Initial structure com_controller plugin

* Fix linter errors

* Better step size

* Clean up controller code and change subgait to message

* Add launch argument for ground gaiting in simulation

* Remove verdwaalde file

* Fix merge conflict

* Processing Olav's excellent comments :)

File: march_description/urdf/march4.xacro (robot description, xacro)
@@ -6,6 +6,15 @@
     <!-- Value set to: 'base_link' makes the robot stand on the ground also set launch parameter fixed to false and set
     the hover_height to 0.0-->
-    <xacro:property name="parent_name" value="world"/>
-    <xacro:property name="hover_height" value="0.3"/>
+    <xacro:unless value="$(arg ground_gait)">
+        <xacro:property name="parent_name" value="world"/>
+        <xacro:property name="hover_height" value="0.3"/>
+    </xacro:unless>
+    <xacro:if value="$(arg ground_gait)">
+        <xacro:property name="parent_name" value="base_link"/>
+        <xacro:property name="hover_height" value="0.0"/>
+        <gazebo>
+            <plugin name="com_controller" filename="libmarch_gazebo_plugins.so"/>
+        </gazebo>
+    </xacro:if>
     <xacro:arg name="max_effort_rotary" default="20475" /> <!-- = 25 A -->
     <xacro:arg name="max_effort_linear" default="22932.0" />  <!-- = 28 A -->

Commit message: Increase friction

File: march_description/urdf/march4.xacro (robot description, xacro)
@@ -60,6 +60,6 @@
     <xacro:property name="foot_height_backward" value="${0.059}"/>
     <xacro:property name="foot_mass" value="0.847"/>
-    <xacro:property name="foot_mu1" value="0.9"/>
-    <xacro:property name="foot_mu2" value="0.9"/>
+    <xacro:property name="foot_mu1" value="1"/>
+    <xacro:property name="foot_mu2" value="1"/>
     <!-- Minimum allowable depth before contact correction impulse is applied. -->
     <xacro:property name="foot_min_depth" value="0.0005"/>
@@ -315,4 +315,5 @@
         <mu2>${foot_mu2}</mu2>
         <minDepth>${foot_min_depth}</minDepth>
+        <fdir1>1 0 0</fdir1>
     </gazebo>
     <!-- Right Moving Hip-->
@@ -445,4 +446,5 @@
         <mu2>${foot_mu2}</mu2>
         <minDepth>${foot_min_depth}</minDepth>
+        <fdir1>1 0 0</fdir1>
     </gazebo>
     <!-- Joints -->

Commit message: Change stl file names

File: march_description/urdf/march4.xacro (robot description, xacro)
@@ -44,20 +44,20 @@
     <xacro:property name="width" value="0.05"/> <!-- Square dimensions (widthxwidth) of beams -->
     <xacro:property name="hip_base_height" value="0.160"/>
-    <xacro:property name="hip_base_mass" value="6.089"/>
+    <xacro:property name="hip_base_mass" value="8.686"/>
     <!-- mass = Hip base + HAA actuators -->
     <xacro:property name="hip_aa_frame_height" value="0.170"/>
     <xacro:property name="hip_aa_frame_width" value="0.1395"/>
-    <xacro:property name="hip_aa_mass" value="1.407"/>
+    <xacro:property name="hip_aa_mass" value="2.917"/>
     <!-- mass = Moving hip -->
     <xacro:property name="upper_leg_height" value="0.385"/>
-    <xacro:property name="upper_leg_mass" value="7.238"/>
+    <xacro:property name="upper_leg_mass" value="5.022"/>
     <!-- mass = KFE joint + HFE joint + Upper leg -->
     <xacro:property name="lower_leg_height" value="0.385"/>
-    <xacro:property name="lower_leg_mass" value="2.944"/>
+    <xacro:property name="lower_leg_mass" value="4.459"/>
     <!-- mass = Ankle actuator + Lower leg -->
     <xacro:property name="ankle_plate_height" value="0.12"/>
     <xacro:property name="foot_height_forward" value="${0.184}"/>
     <xacro:property name="foot_height_backward" value="${0.059}"/>
-    <xacro:property name="foot_mass" value="0.847"/>
+    <xacro:property name="foot_mass" value="1.821"/>
     <xacro:property name="foot_mu1" value="1"/>
     <xacro:property name="foot_mu2" value="1"/>
@@ -191,5 +191,5 @@
             <origin xyz="0 0 0" rpy="0 0 ${-pi/2}"/>
             <geometry>
-                <mesh filename="package://march_description/urdf/stl-files/HipLeft.stl" scale="1.15 1.15 1.15"/>
+                <mesh filename="package://march_description/urdf/stl-files/LeftHAA.stl" scale="1.15 1.15 1.15"/>
             </geometry>
             <material name="blue"/>
@@ -226,5 +226,5 @@
             <origin xyz="0 0 0" rpy="0 0 ${-pi/2}"/>
             <geometry>
-                <mesh filename="package://march_description/urdf/stl-files/UpperLegLeft.stl" scale="1.15 1.15 1.15"/>
+                <mesh filename="package://march_description/urdf/stl-files/UpperLeftLeg.stl" scale="1.15 1.15 1.15"/>
             </geometry>
             <material name="blue"/>
@@ -253,5 +253,5 @@
             <origin xyz="0 0 0" rpy="0 0 ${-pi/2}"/>
             <geometry>
-                <mesh filename="package://march_description/urdf/stl-files/LowerLegLeft.stl" scale="1.15 1.15 1.15"/>
+                <mesh filename="package://march_description/urdf/stl-files/LowerLeftLeg.stl" scale="1.15 1.15 1.15"/>
             </geometry>
             <material name="blue"/>
@@ -280,5 +280,5 @@
             <origin xyz="0 0 0" rpy="0 0 ${-pi/2}"/>
             <geometry>
-                <mesh filename="package://march_description/urdf/stl-files/FootLeft.stl" scale="1.15 1.15 1.15"/>
+                <mesh filename="package://march_description/urdf/stl-files/LeftFoot.stl" scale="1.15 1.15 1.15"/>
             </geometry>
             <material name="blue"/>
@@ -322,5 +322,5 @@
             <origin xyz="0 0 0" rpy="0 0 ${-pi/2}"/>
             <geometry>
-                <mesh filename="package://march_description/urdf/stl-files/HipRight.stl" scale="1.15 1.15 1.15"/>
+                <mesh filename="package://march_description/urdf/stl-files/RightHAA.stl" scale="1.15 1.15 1.15"/>
             </geometry>
             <material name="blue"/>
@@ -357,5 +357,5 @@
             <origin xyz="0 0 0" rpy="0 0 ${-pi/2}"/>
             <geometry>
-                <mesh filename="package://march_description/urdf/stl-files/UpperLegRight.stl" scale="1.15 1.15 1.15"/>
+                <mesh filename="package://march_description/urdf/stl-files/UpperRightLeg.stl" scale="1.15 1.15 1.15"/>
             </geometry>
             <material name="blue"/>
@@ -384,5 +384,5 @@
             <origin xyz="0 0 0" rpy="0 0 ${-pi/2}"/>
             <geometry>
-                <mesh filename="package://march_description/urdf/stl-files/LowerLegRight.stl" scale="1.15 1.15 1.15"/>
+                <mesh filename="package://march_description/urdf/stl-files/LowerRightLeg.stl" scale="1.15 1.15 1.15"/>
             </geometry>
             <material name="blue"/>
@@ -411,5 +411,5 @@
             <origin xyz="0 0 0" rpy="0 0 ${-pi/2}"/>
             <geometry>
-                <mesh filename="package://march_description/urdf/stl-files/FootRight.stl" scale="1.15 1.15 1.15"/>
+                <mesh filename="package://march_description/urdf/stl-files/RightFoot.stl" scale="1.15 1.15 1.15"/>
             </geometry>
             <material name="blue"/>

Commit message: Update masses, inertia and CoM in URDF

File: march_description/urdf/march4.xacro (robot description, xacro)
@@ -44,20 +44,20 @@
     <xacro:property name="width" value="0.05"/> <!-- Square dimensions (widthxwidth) of beams -->
     <xacro:property name="hip_base_height" value="0.160"/>
-    <xacro:property name="hip_base_mass" value="8.686"/>
+    <xacro:property name="hip_base_mass" value="8.677"/>
     <!-- mass = Hip base + HAA actuators -->
     <xacro:property name="hip_aa_frame_height" value="0.170"/>
     <xacro:property name="hip_aa_frame_width" value="0.1395"/>
-    <xacro:property name="hip_aa_mass" value="2.917"/>
+    <xacro:property name="hip_aa_mass" value="3.186"/>
     <!-- mass = Moving hip -->
     <xacro:property name="upper_leg_height" value="0.385"/>
-    <xacro:property name="upper_leg_mass" value="5.022"/>
+    <xacro:property name="upper_leg_mass" value="4.995"/>
     <!-- mass = KFE joint + HFE joint + Upper leg -->
     <xacro:property name="lower_leg_height" value="0.385"/>
-    <xacro:property name="lower_leg_mass" value="4.459"/>
+    <xacro:property name="lower_leg_mass" value="4.455"/>
     <!-- mass = Ankle actuator + Lower leg -->
     <xacro:property name="ankle_plate_height" value="0.12"/>
     <xacro:property name="foot_height_forward" value="${0.184}"/>
     <xacro:property name="foot_height_backward" value="${0.059}"/>
-    <xacro:property name="foot_mass" value="1.821"/>
+    <xacro:property name="foot_mass" value="1.552"/>
     <xacro:property name="foot_mu1" value="1"/>
     <xacro:property name="foot_mu2" value="1"/>
@@ -72,19 +72,19 @@
          the URDF y axis and the Catia y axis is the negative URDF x axis. The given CoM are for the right leg,
          the y coordinate will be inverted for the left leg. -->
-    <xacro:property name="hip_base_com_x" value="${-hip_aa_frame_width + 0.124786}"/>
-    <xacro:property name="hip_base_com_y" value="0.00000911124"/>
-    <xacro:property name="hip_base_com_z" value="0.152163"/>
-    <xacro:property name="hip_aa_com_x" value="${-hip_aa_frame_width + 0.0669488}"/>
-    <xacro:property name="hip_aa_com_y" value="${-hip_base_height/2 - hip_aa_frame_height + 0.210566}"/>
-    <xacro:property name="hip_aa_com_z" value="-0.000250494"/>
-    <xacro:property name="upper_leg_com_x" value="-0.00219961"/>
-    <xacro:property name="upper_leg_com_y" value="${-hip_base_height/2 - hip_aa_frame_height + 0.221535}"/>
-    <xacro:property name="upper_leg_com_z" value="-0.184207"/>
-    <xacro:property name="lower_leg_com_x" value="-0.00434063"/>
-    <xacro:property name="lower_leg_com_y" value="${-hip_base_height/2 - hip_aa_frame_height + 0.184583}"/>
-    <xacro:property name="lower_leg_com_z" value="${upper_leg_height - 0.511661}"/>
-    <xacro:property name="foot_com_x" value="-0.0450791"/>
-    <xacro:property name="foot_com_y" value="${-hip_base_height/2 - hip_aa_frame_height + 0.147081}"/>
-    <xacro:property name="foot_com_z" value="${upper_leg_height + lower_leg_height + ankle_plate_height - 0.844751}"/>
+    <xacro:property name="hip_base_com_x" value="${-hip_aa_frame_width + 0.147398}"/>
+    <xacro:property name="hip_base_com_y" value="0.0000096"/>
+    <xacro:property name="hip_base_com_z" value="0.162659"/>
+    <xacro:property name="hip_aa_com_x" value="${-hip_aa_frame_width + 0.108336}"/>
+    <xacro:property name="hip_aa_com_y" value="${-hip_base_height/2 - hip_aa_frame_height + 0.196537}"/>
+    <xacro:property name="hip_aa_com_z" value="0.02943"/>
+    <xacro:property name="upper_leg_com_x" value="0.000827"/>
+    <xacro:property name="upper_leg_com_y" value="${-hip_base_height/2 - hip_aa_frame_height + 0.214247}"/>
+    <xacro:property name="upper_leg_com_z" value="-0.191575"/>
+    <xacro:property name="lower_leg_com_x" value="-0.00321"/>
+    <xacro:property name="lower_leg_com_y" value="${-hip_base_height/2 - hip_aa_frame_height + 0.184081}"/>
+    <xacro:property name="lower_leg_com_z" value="${upper_leg_height - 0.527082}"/>
+    <xacro:property name="foot_com_x" value="-0.020736"/>
+    <xacro:property name="foot_com_y" value="${-hip_base_height/2 - hip_aa_frame_height + 0.169177}"/>
+    <xacro:property name="foot_com_z" value="${upper_leg_height + lower_leg_height + ankle_plate_height - 0.648891}"/>
     <!-- Inertia of the parts -->
     <!-- Inertia's have been determined in Catia, see
@@ -93,34 +93,34 @@
          axis is the negative URDF x axis, see confluence for the impact. The given inertia's are for the right leg,
          Ixy and Iyz will be inverted for the left leg. -->
-    <xacro:property name="hip_base_Ixx" value="0.117325"/>
-    <xacro:property name="hip_base_Ixy" value="-0.0000239249"/>
-    <xacro:property name="hip_base_Ixz" value="0.0179732"/>
-    <xacro:property name="hip_base_Iyy" value="0.0745937"/>
-    <xacro:property name="hip_base_Iyz" value="-0.00000472801"/>
-    <xacro:property name="hip_base_Izz" value="0.0684134"/>
-    <xacro:property name="hip_aa_Ixx" value="0.00841686"/>
-    <xacro:property name="hip_aa_Ixy" value="0.00655578"/>
-    <xacro:property name="hip_aa_Ixz" value="0.0000910634"/>
-    <xacro:property name="hip_aa_Iyy" value="0.0165504"/>
-    <xacro:property name="hip_aa_Iyz" value="0.0000996411"/>
-    <xacro:property name="hip_aa_Izz" value="0.0229261"/>
-    <xacro:property name="upper_leg_Ixx" value="0.119187"/>
-    <xacro:property name="upper_leg_Ixy" value="-0.0000363676"/>
-    <xacro:property name="upper_leg_Ixz" value="-0.0000393791"/>
-    <xacro:property name="upper_leg_Iyy" value="0.11867"/>
-    <xacro:property name="upper_leg_Iyz" value="-0.0125652"/>
-    <xacro:property name="upper_leg_Izz" value="0.00881972"/>
-    <xacro:property name="lower_leg_Ixx" value="0.0725438"/>
-    <xacro:property name="lower_leg_Ixy" value="-0.0264923"/>
-    <xacro:property name="lower_leg_Ixz" value="0.00934723"/>
-    <xacro:property name="lower_leg_Iyy" value="0.108683"/>
-    <xacro:property name="lower_leg_Iyz" value="0.00109811"/>
-    <xacro:property name="lower_leg_Izz" value="0.0715361" />
-    <xacro:property name="foot_Ixx" value="0.00414758"/>
-    <xacro:property name="foot_Ixy" value="-0.00185339"/>
-    <xacro:property name="foot_Ixz" value="-0.00254464"/>
-    <xacro:property name="foot_Iyy" value="0.00855883"/>
-    <xacro:property name="foot_Iyz" value="-0.00166213"/>
-    <xacro:property name="foot_Izz" value="0.00715736" />
+    <xacro:property name="hip_base_Ixx" value="0.141"/>
+    <xacro:property name="hip_base_Ixy" value="0.0000335"/>
+    <xacro:property name="hip_base_Ixz" value="-0.007"/>
+    <xacro:property name="hip_base_Iyy" value="0.087"/>
+    <xacro:property name="hip_base_Iyz" value="0.0005089"/>
+    <xacro:property name="hip_base_Izz" value="0.089"/>
+    <xacro:property name="hip_aa_Ixx" value="0.02"/>
+    <xacro:property name="hip_aa_Ixy" value="0.009"/>
+    <xacro:property name="hip_aa_Ixz" value="0.005"/>
+    <xacro:property name="hip_aa_Iyy" value="0.031"/>
+    <xacro:property name="hip_aa_Iyz" value="-0.004"/>
+    <xacro:property name="hip_aa_Izz" value="0.03"/>
+    <xacro:property name="upper_leg_Ixx" value="0.127"/>
+    <xacro:property name="upper_leg_Ixy" value="0.0001291"/>
+    <xacro:property name="upper_leg_Ixz" value="-0.0002056"/>
+    <xacro:property name="upper_leg_Iyy" value="0.122"/>
+    <xacro:property name="upper_leg_Iyz" value="0.016"/>
+    <xacro:property name="upper_leg_Izz" value="0.015"/>
+    <xacro:property name="lower_leg_Ixx" value="0.075"/>
+    <xacro:property name="lower_leg_Ixy" value="-0.027"/>
+    <xacro:property name="lower_leg_Ixz" value="0.008"/>
+    <xacro:property name="lower_leg_Iyy" value="0.11"/>
+    <xacro:property name="lower_leg_Iyz" value="-0.002"/>
+    <xacro:property name="lower_leg_Izz" value="0.071" />
+    <xacro:property name="foot_Ixx" value="0.01"/>
+    <xacro:property name="foot_Ixy" value="-0.002"/>
+    <xacro:property name="foot_Ixz" value="0.005"/>
+    <xacro:property name="foot_Iyy" value="0.014"/>
+    <xacro:property name="foot_Iyz" value="0.002"/>
+    <xacro:property name="foot_Izz" value="0.007" />
     <!-- Joint properties -->
     <xacro:property name="hip_fe_rotation_lower_limit" value="${-20*pi/180}"/> <!-- rad -->

Commit message: Revert name change

File: march_description/urdf/march4.xacro (robot description, xacro)
@@ -191,5 +191,5 @@
             <origin xyz="0 0 0" rpy="0 0 ${-pi/2}"/>
             <geometry>
-                <mesh filename="package://march_description/urdf/stl-files/LeftHAA.stl" scale="1.15 1.15 1.15"/>
+                <mesh filename="package://march_description/urdf/stl-files/HipLeft.stl" scale="1.15 1.15 1.15"/>
             </geometry>
             <material name="blue"/>
@@ -226,5 +226,5 @@
             <origin xyz="0 0 0" rpy="0 0 ${-pi/2}"/>
             <geometry>
-                <mesh filename="package://march_description/urdf/stl-files/UpperLeftLeg.stl" scale="1.15 1.15 1.15"/>
+                <mesh filename="package://march_description/urdf/stl-files/UpperLegLeft.stl" scale="1.15 1.15 1.15"/>
             </geometry>
             <material name="blue"/>
@@ -253,5 +253,5 @@
             <origin xyz="0 0 0" rpy="0 0 ${-pi/2}"/>
             <geometry>
-                <mesh filename="package://march_description/urdf/stl-files/LowerLeftLeg.stl" scale="1.15 1.15 1.15"/>
+                <mesh filename="package://march_description/urdf/stl-files/LowerLegLeft.stl" scale="1.15 1.15 1.15"/>
             </geometry>
             <material name="blue"/>
@@ -280,5 +280,5 @@
             <origin xyz="0 0 0" rpy="0 0 ${-pi/2}"/>
             <geometry>
-                <mesh filename="package://march_description/urdf/stl-files/LeftFoot.stl" scale="1.15 1.15 1.15"/>
+                <mesh filename="package://march_description/urdf/stl-files/FootLeft.stl" scale="1.15 1.15 1.15"/>
             </geometry>
             <material name="blue"/>
@@ -322,5 +322,5 @@
             <origin xyz="0 0 0" rpy="0 0 ${-pi/2}"/>
             <geometry>
-                <mesh filename="package://march_description/urdf/stl-files/RightHAA.stl" scale="1.15 1.15 1.15"/>
+                <mesh filename="package://march_description/urdf/stl-files/HipRight.stl" scale="1.15 1.15 1.15"/>
             </geometry>
             <material name="blue"/>
@@ -357,5 +357,5 @@
             <origin xyz="0 0 0" rpy="0 0 ${-pi/2}"/>
             <geometry>
-                <mesh filename="package://march_description/urdf/stl-files/UpperRightLeg.stl" scale="1.15 1.15 1.15"/>
+                <mesh filename="package://march_description/urdf/stl-files/UpperLegRight.stl" scale="1.15 1.15 1.15"/>
             </geometry>
             <material name="blue"/>
@@ -384,5 +384,5 @@
             <origin xyz="0 0 0" rpy="0 0 ${-pi/2}"/>
             <geometry>
-                <mesh filename="package://march_description/urdf/stl-files/LowerRightLeg.stl" scale="1.15 1.15 1.15"/>
+                <mesh filename="package://march_description/urdf/stl-files/LowerLegRight.stl" scale="1.15 1.15 1.15"/>
             </geometry>
             <material name="blue"/>
@@ -411,5 +411,5 @@
             <origin xyz="0 0 0" rpy="0 0 ${-pi/2}"/>
             <geometry>
-                <mesh filename="package://march_description/urdf/stl-files/RightFoot.stl" scale="1.15 1.15 1.15"/>
+                <mesh filename="package://march_description/urdf/stl-files/FootRight.stl" scale="1.15 1.15 1.15"/>
             </geometry>
             <material name="blue"/>

Commit message: Rename files

File: march_description/urdf/march4.xacro (robot description, xacro)
@@ -191,5 +191,5 @@
             <origin xyz="0 0 0" rpy="0 0 ${-pi/2}"/>
             <geometry>
-                <mesh filename="package://march_description/urdf/stl-files/HipLeft.stl" scale="1.15 1.15 1.15"/>
+                <mesh filename="package://march_description/urdf/stl-files/LeftHAA.stl" scale="1.15 1.15 1.15"/>
             </geometry>
             <material name="blue"/>
@@ -226,5 +226,5 @@
             <origin xyz="0 0 0" rpy="0 0 ${-pi/2}"/>
             <geometry>
-                <mesh filename="package://march_description/urdf/stl-files/UpperLegLeft.stl" scale="1.15 1.15 1.15"/>
+                <mesh filename="package://march_description/urdf/stl-files/UpperLeftLeg.stl" scale="1.15 1.15 1.15"/>
             </geometry>
             <material name="blue"/>
@@ -253,5 +253,5 @@
             <origin xyz="0 0 0" rpy="0 0 ${-pi/2}"/>
             <geometry>
-                <mesh filename="package://march_description/urdf/stl-files/LowerLegLeft.stl" scale="1.15 1.15 1.15"/>
+                <mesh filename="package://march_description/urdf/stl-files/LowerLeftLeg.stl" scale="1.15 1.15 1.15"/>
             </geometry>
             <material name="blue"/>
@@ -280,5 +280,5 @@
             <origin xyz="0 0 0" rpy="0 0 ${-pi/2}"/>
             <geometry>
-                <mesh filename="package://march_description/urdf/stl-files/FootLeft.stl" scale="1.15 1.15 1.15"/>
+                <mesh filename="package://march_description/urdf/stl-files/LeftFoot.stl" scale="1.15 1.15 1.15"/>
             </geometry>
             <material name="blue"/>
@@ -322,5 +322,5 @@
             <origin xyz="0 0 0" rpy="0 0 ${-pi/2}"/>
             <geometry>
-                <mesh filename="package://march_description/urdf/stl-files/HipRight.stl" scale="1.15 1.15 1.15"/>
+                <mesh filename="package://march_description/urdf/stl-files/RightHAA.stl" scale="1.15 1.15 1.15"/>
             </geometry>
             <material name="blue"/>
@@ -357,5 +357,5 @@
             <origin xyz="0 0 0" rpy="0 0 ${-pi/2}"/>
             <geometry>
-                <mesh filename="package://march_description/urdf/stl-files/UpperLegRight.stl" scale="1.15 1.15 1.15"/>
+                <mesh filename="package://march_description/urdf/stl-files/UpperRightLeg.stl" scale="1.15 1.15 1.15"/>
             </geometry>
             <material name="blue"/>
@@ -384,5 +384,5 @@
             <origin xyz="0 0 0" rpy="0 0 ${-pi/2}"/>
             <geometry>
-                <mesh filename="package://march_description/urdf/stl-files/LowerLegRight.stl" scale="1.15 1.15 1.15"/>
+                <mesh filename="package://march_description/urdf/stl-files/LowerRightLeg.stl" scale="1.15 1.15 1.15"/>
             </geometry>
             <material name="blue"/>
@@ -411,5 +411,5 @@
             <origin xyz="0 0 0" rpy="0 0 ${-pi/2}"/>
             <geometry>
-                <mesh filename="package://march_description/urdf/stl-files/FootRight.stl" scale="1.15 1.15 1.15"/>
+                <mesh filename="package://march_description/urdf/stl-files/RightFoot.stl" scale="1.15 1.15 1.15"/>
             </geometry>
             <material name="blue"/>
