Commit message: Update stl files

File: march_description/urdf/march4.xacro (robot description, xacro)
@@ -161,5 +161,5 @@
             <origin xyz="0 0 0" rpy="0 0 ${-pi/2}"/>
             <geometry>
-                <mesh filename="package://march_description/urdf/stl-files/HipBase.stl" scale="1.15 1.15 1.15"/>
+                <mesh filename="package://march_description/urdf/stl-files/HipBase.stl" scale="1150 1150 1150"/>
             </geometry>
             <material name="blue"/>
@@ -191,5 +191,5 @@
             <origin xyz="0 0 0" rpy="0 0 ${-pi/2}"/>
             <geometry>
-                <mesh filename="package://march_description/urdf/stl-files/LeftHAA.stl" scale="1.15 1.15 1.15"/>
+                <mesh filename="package://march_description/urdf/stl-files/LeftHAA.stl" scale="1150 1150 1150"/>
             </geometry>
             <material name="blue"/>
@@ -226,5 +226,5 @@
             <origin xyz="0 0 0" rpy="0 0 ${-pi/2}"/>
             <geometry>
-                <mesh filename="package://march_description/urdf/stl-files/UpperLeftLeg.stl" scale="1.15 1.15 1.15"/>
+                <mesh filename="package://march_description/urdf/stl-files/UpperLegLeft.stl" scale="1150 1150 1150"/>
             </geometry>
             <material name="blue"/>
@@ -253,5 +253,5 @@
             <origin xyz="0 0 0" rpy="0 0 ${-pi/2}"/>
             <geometry>
-                <mesh filename="package://march_description/urdf/stl-files/LowerLeftLeg.stl" scale="1.15 1.15 1.15"/>
+                <mesh filename="package://march_description/urdf/stl-files/LowerLegLeft.stl" scale="1150 1150 1150"/>
             </geometry>
             <material name="blue"/>
@@ -280,5 +280,5 @@
             <origin xyz="0 0 0" rpy="0 0 ${-pi/2}"/>
             <geometry>
-                <mesh filename="package://march_description/urdf/stl-files/LeftFoot.stl" scale="1.15 1.15 1.15"/>
+                <mesh filename="package://march_description/urdf/stl-files/LeftFoot.stl" scale="1150 1150 1150"/>
             </geometry>
             <material name="blue"/>
@@ -322,5 +322,5 @@
             <origin xyz="0 0 0" rpy="0 0 ${-pi/2}"/>
             <geometry>
-                <mesh filename="package://march_description/urdf/stl-files/RightHAA.stl" scale="1.15 1.15 1.15"/>
+                <mesh filename="package://march_description/urdf/stl-files/RightHAA.stl" scale="1150 1150 1150"/>
             </geometry>
             <material name="blue"/>
@@ -357,5 +357,5 @@
             <origin xyz="0 0 0" rpy="0 0 ${-pi/2}"/>
             <geometry>
-                <mesh filename="package://march_description/urdf/stl-files/UpperRightLeg.stl" scale="1.15 1.15 1.15"/>
+                <mesh filename="package://march_description/urdf/stl-files/UpperLegRight.stl" scale="1150 1150 1150"/>
             </geometry>
             <material name="blue"/>
@@ -384,5 +384,5 @@
             <origin xyz="0 0 0" rpy="0 0 ${-pi/2}"/>
             <geometry>
-                <mesh filename="package://march_description/urdf/stl-files/LowerRightLeg.stl" scale="1.15 1.15 1.15"/>
+                <mesh filename="package://march_description/urdf/stl-files/LowerLegRight.stl" scale="1150 1150 1150"/>
             </geometry>
             <material name="blue"/>
@@ -411,5 +411,5 @@
             <origin xyz="0 0 0" rpy="0 0 ${-pi/2}"/>
             <geometry>
-                <mesh filename="package://march_description/urdf/stl-files/RightFoot.stl" scale="1.15 1.15 1.15"/>
+                <mesh filename="package://march_description/urdf/stl-files/RightFoot.stl" scale="1150 1150 1150"/>
             </geometry>
             <material name="blue"/>

Commit message: Fix scale of visualisation

File: march_description/urdf/march4.xacro (robot description, xacro)
@@ -161,5 +161,5 @@
             <origin xyz="0 0 0" rpy="0 0 ${-pi/2}"/>
             <geometry>
-                <mesh filename="package://march_description/urdf/stl-files/HipBase.stl" scale="1150 1150 1150"/>
+                <mesh filename="package://march_description/urdf/stl-files/HipBase.stl" scale="0.00115 0.00115 0.00115"/>
             </geometry>
             <material name="blue"/>
@@ -189,7 +189,7 @@
     <link name="hip_aa_frame_left_side">
         <visual>
-            <origin xyz="0 0 0" rpy="0 0 ${-pi/2}"/>
-            <geometry>
-                <mesh filename="package://march_description/urdf/stl-files/LeftHAA.stl" scale="1150 1150 1150"/>
+            <origin xyz="0.2 0 0" rpy="0 0 ${-pi/2}"/>
+            <geometry>
+                <mesh filename="package://march_description/urdf/stl-files/LeftHAA.stl" scale="0.00115 0.00115 0.00115"/>
             </geometry>
             <material name="blue"/>
@@ -226,5 +226,5 @@
             <origin xyz="0 0 0" rpy="0 0 ${-pi/2}"/>
             <geometry>
-                <mesh filename="package://march_description/urdf/stl-files/UpperLegLeft.stl" scale="1150 1150 1150"/>
+                <mesh filename="package://march_description/urdf/stl-files/UpperLegLeft.stl" scale="0.00115 0.00115 0.00115"/>
             </geometry>
             <material name="blue"/>
@@ -253,5 +253,5 @@
             <origin xyz="0 0 0" rpy="0 0 ${-pi/2}"/>
             <geometry>
-                <mesh filename="package://march_description/urdf/stl-files/LowerLegLeft.stl" scale="1150 1150 1150"/>
+                <mesh filename="package://march_description/urdf/stl-files/LowerLegLeft.stl" scale="0.00115 0.00115 0.00115"/>
             </geometry>
             <material name="blue"/>
@@ -280,5 +280,5 @@
             <origin xyz="0 0 0" rpy="0 0 ${-pi/2}"/>
             <geometry>
-                <mesh filename="package://march_description/urdf/stl-files/LeftFoot.stl" scale="1150 1150 1150"/>
+                <mesh filename="package://march_description/urdf/stl-files/LeftFoot.stl" scale="0.00115 0.00115 0.00115"/>
             </geometry>
             <material name="blue"/>
@@ -320,7 +320,7 @@
     <link name="hip_aa_frame_right_side">
         <visual>
-            <origin xyz="0 0 0" rpy="0 0 ${-pi/2}"/>
-            <geometry>
-                <mesh filename="package://march_description/urdf/stl-files/RightHAA.stl" scale="1150 1150 1150"/>
+            <origin xyz="-0.2 0 0" rpy="0 0 ${pi/2}"/>
+            <geometry>
+                <mesh filename="package://march_description/urdf/stl-files/RightHAA.stl" scale="0.00115 0.00115 0.00115"/>
             </geometry>
             <material name="blue"/>
@@ -357,5 +357,5 @@
             <origin xyz="0 0 0" rpy="0 0 ${-pi/2}"/>
             <geometry>
-                <mesh filename="package://march_description/urdf/stl-files/UpperLegRight.stl" scale="1150 1150 1150"/>
+                <mesh filename="package://march_description/urdf/stl-files/UpperLegRight.stl" scale="0.00115 0.00115 0.00115"/>
             </geometry>
             <material name="blue"/>
@@ -384,5 +384,5 @@
             <origin xyz="0 0 0" rpy="0 0 ${-pi/2}"/>
             <geometry>
-                <mesh filename="package://march_description/urdf/stl-files/LowerLegRight.stl" scale="1150 1150 1150"/>
+                <mesh filename="package://march_description/urdf/stl-files/LowerLegRight.stl" scale="0.00115 0.00115 0.00115"/>
             </geometry>
             <material name="blue"/>
@@ -411,5 +411,5 @@
             <origin xyz="0 0 0" rpy="0 0 ${-pi/2}"/>
             <geometry>
-                <mesh filename="package://march_description/urdf/stl-files/RightFoot.stl" scale="1150 1150 1150"/>
+                <mesh filename="package://march_description/urdf/stl-files/RightFoot.stl" scale="0.00115 0.00115 0.00115"/>
             </geometry>
             <material name="blue"/>

Commit message: Update stl files and

File: march_description/urdf/march4.xacro (robot description, xacro)
@@ -159,7 +159,7 @@
     <link name="hip_base">
         <visual>
-            <origin xyz="0 0 0" rpy="0 0 ${-pi/2}"/>
-            <geometry>
-                <mesh filename="package://march_description/urdf/stl-files/HipBase.stl" scale="0.00115 0.00115 0.00115"/>
+            <origin xyz="${-hip_aa_frame_width} 0 0" rpy="0 0 ${pi}"/>
+            <geometry>
+                <mesh filename="package://march_description/urdf/stl-files/HipBase.stl" scale="1.15 1.15 1.15"/>
             </geometry>
             <material name="blue"/>
@@ -189,7 +189,7 @@
     <link name="hip_aa_frame_left_side">
         <visual>
-            <origin xyz="0.2 0 0" rpy="0 0 ${-pi/2}"/>
-            <geometry>
-                <mesh filename="package://march_description/urdf/stl-files/LeftHAA.stl" scale="0.00115 0.00115 0.00115"/>
+            <origin xyz="${-hip_aa_frame_width} ${hip_base_height/2} 0" rpy="0 0 ${pi}"/>
+            <geometry>
+                <mesh filename="package://march_description/urdf/stl-files/LeftHAA.stl" scale="1.15 1.15 1.15"/>
             </geometry>
             <material name="blue"/>
@@ -224,7 +224,7 @@
     <link name="upper_leg_left">
         <visual>
-            <origin xyz="0 0 0" rpy="0 0 ${-pi/2}"/>
-            <geometry>
-                <mesh filename="package://march_description/urdf/stl-files/UpperLegLeft.stl" scale="0.00115 0.00115 0.00115"/>
+            <origin xyz="0 ${hip_base_height/2 + hip_aa_frame_height} 0" rpy="0 0 ${pi}"/>
+            <geometry>
+                <mesh filename="package://march_description/urdf/stl-files/UpperLeftLeg.stl" scale="1.15 1.15 1.15"/>
             </geometry>
             <material name="blue"/>
@@ -251,7 +251,7 @@
     <link name="lower_leg_left">
         <visual>
-            <origin xyz="0 0 0" rpy="0 0 ${-pi/2}"/>
-            <geometry>
-                <mesh filename="package://march_description/urdf/stl-files/LowerLegLeft.stl" scale="0.00115 0.00115 0.00115"/>
+            <origin xyz="0 ${hip_base_height/2 + hip_aa_frame_height} ${upper_leg_height}" rpy="0 0 ${pi}"/>
+            <geometry>
+                <mesh filename="package://march_description/urdf/stl-files/LowerLeftLeg.stl" scale="1.15 1.15 1.15"/>
             </geometry>
             <material name="blue"/>
@@ -278,7 +278,7 @@
     <link name="ankle_plate_left">
         <visual>
-            <origin xyz="0 0 0" rpy="0 0 ${-pi/2}"/>
-            <geometry>
-                <mesh filename="package://march_description/urdf/stl-files/LeftFoot.stl" scale="0.00115 0.00115 0.00115"/>
+            <origin xyz="0 ${hip_base_height/2 + hip_aa_frame_height} ${upper_leg_height + lower_leg_height}" rpy="0 0 ${pi}"/>
+            <geometry>
+                <mesh filename="package://march_description/urdf/stl-files/LeftFoot.stl" scale="1.15 1.15 1.15"/>
             </geometry>
             <material name="blue"/>
@@ -320,7 +320,7 @@
     <link name="hip_aa_frame_right_side">
         <visual>
-            <origin xyz="-0.2 0 0" rpy="0 0 ${pi/2}"/>
-            <geometry>
-                <mesh filename="package://march_description/urdf/stl-files/RightHAA.stl" scale="0.00115 0.00115 0.00115"/>
+            <origin xyz="${-hip_aa_frame_width} ${-hip_base_height/2} 0" rpy="0 0 ${pi}"/>
+            <geometry>
+                <mesh filename="package://march_description/urdf/stl-files/RightHAA.stl" scale="1.15 1.15 1.15"/>
             </geometry>
             <material name="blue"/>
@@ -355,7 +355,7 @@
     <link name="upper_leg_right">
         <visual>
-            <origin xyz="0 0 0" rpy="0 0 ${-pi/2}"/>
-            <geometry>
-                <mesh filename="package://march_description/urdf/stl-files/UpperLegRight.stl" scale="0.00115 0.00115 0.00115"/>
+            <origin xyz="0 ${-hip_base_height/2 - hip_aa_frame_height} 0" rpy="0 0 ${pi}"/>
+            <geometry>
+                <mesh filename="package://march_description/urdf/stl-files/UpperRightLeg.stl" scale="1.15 1.15 1.15"/>
             </geometry>
             <material name="blue"/>
@@ -382,7 +382,7 @@
     <link name="lower_leg_right">
         <visual>
-            <origin xyz="0 0 0" rpy="0 0 ${-pi/2}"/>
-            <geometry>
-                <mesh filename="package://march_description/urdf/stl-files/LowerLegRight.stl" scale="0.00115 0.00115 0.00115"/>
+            <origin xyz="0 ${-hip_base_height/2 - hip_aa_frame_height} ${upper_leg_height}" rpy="0 0 ${pi}"/>
+            <geometry>
+                <mesh filename="package://march_description/urdf/stl-files/LowerRightLeg.stl" scale="1.15 1.15 1.15"/>
             </geometry>
             <material name="blue"/>
@@ -409,7 +409,7 @@
     <link name="ankle_plate_right">
         <visual>
-            <origin xyz="0 0 0" rpy="0 0 ${-pi/2}"/>
-            <geometry>
-                <mesh filename="package://march_description/urdf/stl-files/RightFoot.stl" scale="0.00115 0.00115 0.00115"/>
+            <origin xyz="0 ${-hip_base_height/2 - hip_aa_frame_height} ${upper_leg_height + lower_leg_height}" rpy="0 0 ${pi}"/>
+            <geometry>
+                <mesh filename="package://march_description/urdf/stl-files/RightFoot.stl" scale="1.15 1.15 1.15"/>
             </geometry>
             <material name="blue"/>

Commit message: Fix scaling and enlarge shoe

File: march_description/urdf/march4.xacro (robot description, xacro)
@@ -87,4 +87,5 @@
     <xacro:property name="foot_com_y" value="${-hip_base_height/2 - hip_aa_frame_height + 0.169177}"/>
     <xacro:property name="foot_com_z" value="${upper_leg_height + lower_leg_height + ankle_plate_height - 0.648891}"/>
+    <xacro:property name="foot_scale" value="1.35"/>
     <!-- Inertia of the parts -->
     <!-- Inertia's have been determined in Catia, see
@@ -161,5 +162,5 @@
             <origin xyz="${-hip_aa_frame_width} 0 0" rpy="0 0 ${pi}"/>
             <geometry>
-                <mesh filename="package://march_description/urdf/stl-files/HipBase.stl" scale="1.15 1.15 1.15"/>
+                <mesh filename="package://march_description/urdf/stl-files/HipBase.stl" scale="1 1 1"/>
             </geometry>
             <material name="blue"/>
@@ -191,5 +192,5 @@
             <origin xyz="${-hip_aa_frame_width} ${hip_base_height/2} 0" rpy="0 0 ${pi}"/>
             <geometry>
-                <mesh filename="package://march_description/urdf/stl-files/LeftHAA.stl" scale="1.15 1.15 1.15"/>
+                <mesh filename="package://march_description/urdf/stl-files/LeftHAA.stl" scale="1 1 1"/>
             </geometry>
             <material name="blue"/>
@@ -226,5 +227,5 @@
             <origin xyz="0 ${hip_base_height/2 + hip_aa_frame_height} 0" rpy="0 0 ${pi}"/>
             <geometry>
-                <mesh filename="package://march_description/urdf/stl-files/UpperLeftLeg.stl" scale="1.15 1.15 1.15"/>
+                <mesh filename="package://march_description/urdf/stl-files/UpperLeftLeg.stl" scale="1 1 1"/>
             </geometry>
             <material name="blue"/>
@@ -253,5 +254,5 @@
             <origin xyz="0 ${hip_base_height/2 + hip_aa_frame_height} ${upper_leg_height}" rpy="0 0 ${pi}"/>
             <geometry>
-                <mesh filename="package://march_description/urdf/stl-files/LowerLeftLeg.stl" scale="1.15 1.15 1.15"/>
+                <mesh filename="package://march_description/urdf/stl-files/LowerLeftLeg.stl" scale="1 1 1"/>
             </geometry>
             <material name="blue"/>
@@ -278,7 +279,7 @@
     <link name="ankle_plate_left">
         <visual>
-            <origin xyz="0 ${hip_base_height/2 + hip_aa_frame_height} ${upper_leg_height + lower_leg_height}" rpy="0 0 ${pi}"/>
-            <geometry>
-                <mesh filename="package://march_description/urdf/stl-files/LeftFoot.stl" scale="1.15 1.15 1.15"/>
+            <origin xyz="0 ${hip_base_height/2 + hip_aa_frame_height} ${foot_scale * (upper_leg_height + lower_leg_height)}" rpy="0 0 ${pi}"/>
+            <geometry>
+                <mesh filename="package://march_description/urdf/stl-files/LeftFoot.stl" scale="1 1 ${foot_scale}"/>
             </geometry>
             <material name="blue"/>
@@ -322,5 +323,5 @@
             <origin xyz="${-hip_aa_frame_width} ${-hip_base_height/2} 0" rpy="0 0 ${pi}"/>
             <geometry>
-                <mesh filename="package://march_description/urdf/stl-files/RightHAA.stl" scale="1.15 1.15 1.15"/>
+                <mesh filename="package://march_description/urdf/stl-files/RightHAA.stl" scale="1 1 1"/>
             </geometry>
             <material name="blue"/>
@@ -357,5 +358,5 @@
             <origin xyz="0 ${-hip_base_height/2 - hip_aa_frame_height} 0" rpy="0 0 ${pi}"/>
             <geometry>
-                <mesh filename="package://march_description/urdf/stl-files/UpperRightLeg.stl" scale="1.15 1.15 1.15"/>
+                <mesh filename="package://march_description/urdf/stl-files/UpperRightLeg.stl" scale="1 1 1"/>
             </geometry>
             <material name="blue"/>
@@ -384,5 +385,5 @@
             <origin xyz="0 ${-hip_base_height/2 - hip_aa_frame_height} ${upper_leg_height}" rpy="0 0 ${pi}"/>
             <geometry>
-                <mesh filename="package://march_description/urdf/stl-files/LowerRightLeg.stl" scale="1.15 1.15 1.15"/>
+                <mesh filename="package://march_description/urdf/stl-files/LowerRightLeg.stl" scale="1 1 1"/>
             </geometry>
             <material name="blue"/>
@@ -409,7 +410,7 @@
     <link name="ankle_plate_right">
         <visual>
-            <origin xyz="0 ${-hip_base_height/2 - hip_aa_frame_height} ${upper_leg_height + lower_leg_height}" rpy="0 0 ${pi}"/>
-            <geometry>
-                <mesh filename="package://march_description/urdf/stl-files/RightFoot.stl" scale="1.15 1.15 1.15"/>
+            <origin xyz="0 ${-hip_base_height/2 - hip_aa_frame_height} ${foot_scale * (upper_leg_height + lower_leg_height)}" rpy="0 0 ${pi}"/>
+            <geometry>
+                <mesh filename="package://march_description/urdf/stl-files/RightFoot.stl" scale="1 1 ${foot_scale}"/>
             </geometry>
             <material name="blue"/>

Commit message: break up some long lines

File: march_description/urdf/march4.xacro (robot description, xacro)
@@ -279,5 +279,8 @@
     <link name="ankle_plate_left">
         <visual>
-            <origin xyz="0 ${hip_base_height/2 + hip_aa_frame_height} ${foot_scale * (upper_leg_height + lower_leg_height)}" rpy="0 0 ${pi}"/>
+            <origin
+                xyz="0 ${hip_base_height/2 + hip_aa_frame_height} ${foot_scale * (upper_leg_height + lower_leg_height)}"
+                rpy="0 0 ${pi}"
+            />
             <geometry>
                 <mesh filename="package://march_description/urdf/stl-files/LeftFoot.stl" scale="1 1 ${foot_scale}"/>
@@ -410,5 +413,8 @@
     <link name="ankle_plate_right">
         <visual>
-            <origin xyz="0 ${-hip_base_height/2 - hip_aa_frame_height} ${foot_scale * (upper_leg_height + lower_leg_height)}" rpy="0 0 ${pi}"/>
+            <origin
+                xyz="0 ${-hip_base_height/2 - hip_aa_frame_height} ${foot_scale * (upper_leg_height + lower_leg_height)}"
+                rpy="0 0 ${pi}"/>
+            />
             <geometry>
                 <mesh filename="package://march_description/urdf/stl-files/RightFoot.stl" scale="1 1 ${foot_scale}"/>
