Commit message: Add two_odrive_joints robot #2

File: march_description/urdf/two_odrive_joints.xacro (robot description, xacro)
@@ -623,49 +623,4 @@
     </joint>
     <!-- ROS Control plugin for Gazebo -->
-    <transmission name="left_hip_aa">
-        <type>transmission_interface/SimpleTransmission</type>
-        <joint name="left_hip_aa">
-            <hardwareInterface>hardware_interface/EffortJointInterface</hardwareInterface>
-        </joint>
-        <actuator name="left_hip_aa_motor">
-            <mechanicalReduction>200</mechanicalReduction>
-        </actuator>
-    </transmission>
-    <transmission name="left_hip_fe">
-        <type>transmission_interface/SimpleTransmission</type>
-        <joint name="left_hip_fe">
-            <hardwareInterface>hardware_interface/EffortJointInterface</hardwareInterface>
-        </joint>
-        <actuator name="left_hip_fe_motor">
-            <mechanicalReduction>101</mechanicalReduction>
-        </actuator>
-    </transmission>
-    <transmission name="left_knee">
-        <type>transmission_interface/SimpleTransmission</type>
-        <joint name="left_knee">
-            <hardwareInterface>hardware_interface/EffortJointInterface</hardwareInterface>
-        </joint>
-        <actuator name="left_knee_motor">
-            <mechanicalReduction>101</mechanicalReduction>
-        </actuator>
-    </transmission>
-    <transmission name="left_ankle">
-        <type>transmission_interface/SimpleTransmission</type>
-        <joint name="left_ankle">
-            <hardwareInterface>hardware_interface/EffortJointInterface</hardwareInterface>
-        </joint>
-        <actuator name="left_ankle_motor">
-            <mechanicalReduction>200</mechanicalReduction>
-        </actuator>
-    </transmission>
-    <transmission name="right_hip_aa">
-        <type>transmission_interface/SimpleTransmission</type>
-        <joint name="right_hip_aa">
-            <hardwareInterface>hardware_interface/EffortJointInterface</hardwareInterface>
-        </joint>
-        <actuator name="right_hip_aa_motor">
-            <mechanicalReduction>200</mechanicalReduction>
-        </actuator>
-    </transmission>
     <transmission name="right_hip_fe">
         <type>transmission_interface/SimpleTransmission</type>
@@ -686,12 +641,3 @@
         </actuator>
     </transmission>
-    <transmission name="right_ankle">
-        <type>transmission_interface/SimpleTransmission</type>
-        <joint name="right_ankle">
-            <hardwareInterface>hardware_interface/EffortJointInterface</hardwareInterface>
-        </joint>
-        <actuator name="right_ankle_motor">
-            <mechanicalReduction>200</mechanicalReduction>
-        </actuator>
-    </transmission>
 </robot>

Commit message: Remove one joint

File: march_description/urdf/two_odrive_joints.xacro (robot description, xacro)
@@ -575,5 +575,5 @@
         <origin xyz="0 ${hip_aa_frame_height} 0" rpy="0 0 0"/>
     </joint>
-    <joint name="right_hip_fe" type="revolute">
+    <joint name="right_hip_fe" type="fixed">
         <parent link="hip_aa_frame_right_front"/>
         <child link="upper_leg_right"/>

Commit message: Added all the configurations to launch two motors

File: march_description/urdf/two_odrive_joints.xacro (robot description, xacro)
@@ -575,5 +575,5 @@
         <origin xyz="0 ${hip_aa_frame_height} 0" rpy="0 0 0"/>
     </joint>
-    <joint name="right_hip_fe" type="fixed">
+    <joint name="right_hip_fe" type="revolute">
         <parent link="hip_aa_frame_right_front"/>
         <child link="upper_leg_right"/>
